File: EC1834_201.1.sch (KiCad schematic (older format))
At the start: 0 parts

Commit message: Added more ICs Added README
Parts:
- added D10, D16, D39: DL000D, symbol RFT_Digitalschaltkreise:DL000D
- added D100, D115, D116, d101: U2764, symbol robotron_ec1834:U2764
- added D111, D112, D44: DS8286D-D111, symbol robotron_ec1834:DS8286D-D111
- added D13, D67: DL074, symbol robotron_ec1834:DL074
- added D30, D31: DL374, symbol robotron_ec1834:DL374
- added D34, D59, D82, D87: DL004D, symbol RFT_Digitalschaltkreise:DL004D
- added D37, D62: DL032D, symbol RFT_Digitalschaltkreise:DL032D
- added D47: DL008D, symbol robotron_ec1834:DL008D
- added D5: DL030D, symbol RFT_Digitalschaltkreise:DL030D
- added D52, D58, D60: 74HC74, symbol robotron_ec1834:74HC74
- added D53: KR580WI53, Package_DIP:DIP-24_W15.24mm, symbol robotron_ec1834:KR580WI53
- added D54: 8255A, Package_DIP:DIP-40_W15.24mm, symbol robotron_ec1834:8255A
- added D55: UC8821, EC1834-Board:EMR-64_W22.86mm, symbol robotron_ec1834:UC8821
- added D56: 2716, Package_DIP:DIP-24_W15.24mm, symbol robotron_ec1834:2716
- added D57, D69, D70, D72, D88: DL008D, symbol RFT_Digitalschaltkreise:DL008D
- added D63: DL010D-D63, symbol robotron_ec1834:DL010D-D63
- added D65, D66: DS8205, symbol robotron_ec1834:DS8205
- added D68: 74S51, symbol robotron_ec1834:74S51
- added D71: DL002D, symbol RFT_Digitalschaltkreise:DL002D
- added D85, D86: KR531KP11, symbol robotron_ec1834:KR531KP11
- added D90: KR531LI1, symbol robotron_ec1834:KR531LI1
