File: EC1834_201.1.sch (KiCad schematic (older format))
At the start: 42 parts

Commit message: Switch to Kicad 6
Parts:
- added R11: 1k, Resistor_THT:R_Array_SIP6, symbol Device:R_Network05_Split
- added R12: 4k7, Resistor_THT:R_Array_SIP10, symbol Device:R_Network09_Split
- added R14, R15, R16: 30, Resistor_THT:R_Array_SIP8, symbol Device:R_Pack04_SIP_Split
- added R17: 4k7, symbol Device:R
- added R18, R30, R31: 30, symbol Device:R
- added R22: 130, symbol Device:R
- added R23: 4k7, Resistor_THT:R_Array_SIP10, symbol Device:R_Network09
- added R24, R25, R32, R33, R4: 1k, symbol Device:R
- added R40, R41: 4k7, Resistor_THT:R_Array_SIP9, symbol Device:R_Network08
- added R52: 3k9, Resistor_THT:R_Array_SIP8, symbol Device:R_Network07_Split
- added SW1: SW_DIP_x08, symbol Switch:SW_DIP_x08
- renumbered d101 to D101
Connections:
- no-connect marks 0 -> 1
Other:
- moved on the sheet: D70A, D70B
