File: EC1834_201.3.sch (KiCad schematic (older format))
At the start: 65 parts

Commit message: Added more ICs Added README
Connections:
- net MDPEA: now also D90.5 (B2); no longer D90.10 (B3)
- net MEMR: now also D90.4 (A2); no longer D90.9 (A3)
- net at D113.4 (D8): now also D90.6 (Y2); no longer D90.8 (Y3)
Changed lines of the file:
@@
 $Descr A3 11693 16535 portrait
 encoding utf-8
-Sheet 4 4
+Sheet 4 5
 Title "EC1834 201.3 RAM"
 Date "2022-09-05"
@@
 $Comp
 L robotron_ec1834:KR531LI1 D90
-U 3 1 6322F280
+U 2 1 6322F280
 P 6150 14500
 F 0 "D90" H 6150 14550 50  0000 C CNN
@@
 F 2 "" H 6150 14500 50  0001 C CNN
 F 3 "https://www-user.tu-chemnitz.de/~heha/basteln/Konsumg%C3%BCter/DDR-Halbleiter/dl008.gif" H 6150 14500 50  0001 C CNN
-	3    6150 14500
+	2    6150 14500
 	1    0    0    1
 $EndComp
