File: EC1834_201.2.sch (KiCad schematic (older format))
At the start: 56 parts

Commit message: Added more ICs Added README
Parts:
- D88: value KR531LI1 -> DL008D
Changed lines of the file:
@@
 $Descr A2 23386 16535
 encoding utf-8
-Sheet 2 4
+Sheet 2 5
 Title ""
 Date ""
@@
 P 2100 3650
 F 0 "D88" H 2100 3967 50  0000 C CNN
-F 1 "KR531LI1" H 2100 3876 50  0000 C CNN
+F 1 "DL008D" H 2100 3876 50  0000 C CNN
 F 2 "" H 2100 3650 50  0001 C CNN
 F 3 "https://www-user.tu-chemnitz.de/~heha/basteln/Konsumg%C3%BCter/DDR-Halbleiter/dl008.gif" H 2100 3650 50  0001 C CNN
@@
 P 12250 7250
 F 0 "D88" H 12250 7567 50  0000 C CNN
-F 1 "KR531LI1" H 12250 7476 50  0000 C CNN
+F 1 "DL008D" H 12250 7476 50  0000 C CNN
 F 2 "" H 12250 7250 50  0001 C CNN
 F 3 "https://www-user.tu-chemnitz.de/~heha/basteln/Konsumg%C3%BCter/DDR-Halbleiter/dl008.gif" H 12250 7250 50  0001 C CNN

Commit message: Switch to Kicad 6
Parts:
- removed D21: DS8286D-D21, symbol robotron_ec1834:DS8286D-D21
- added D21: DS8286D-D111, symbol robotron_ec1834:DS8286D-D111
- added R1, R2: 4k7, symbol Device:R
- added R10, R12: 4k7, Resistor_THT:R_Array_SIP10, symbol Device:R_Network09_Split
- added R11: 1k, Resistor_THT:R_Array_SIP6, symbol Device:R_Network05_Split
- added R13: 4,7k, symbol Device:R
- added R19: 18k, symbol Device:R
- added R20: 180k, symbol Device:R
- added R21: 100k, symbol Device:R
- added R3, R7, R8: 30, symbol Device:R
- added R5, R6: 511, symbol Device:R
- added R50, R51: 100, symbol Device:R
- added R52: 3k9, Resistor_THT:R_Array_SIP8, symbol Device:R_Network07_Split
- added R9: 30, Resistor_THT:R_Array_SIP8, symbol Device:R_Pack04_SIP_Split
- added WD1: WD1, symbol Jumper:SolderJumper_2_Bridged
- added WD2: WD2, symbol Jumper:SolderJumper_2_Bridged
- added WD3: WD3, symbol Jumper:SolderJumper_2_Bridged
Connections:
- net labels added: CEN, D0, D1, D10, D11, D12, D13, D14, D15, D2, D3, D4, D5, D6, D7, D8, D9, DEN, MEMR, ~CLK
- wire segments 0 -> 131
- no-connect marks 0 -> 3
Other:
- moved on the sheet: D11B, D12A, D12B, D12C, D12D, D13A, D14C, D15A, D16A, D22A, D23A, D24A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
