File: EC1834_201.1.kicad_sch (KiCad schematic)
At the start: 62 parts, among them SW1 SW_DIP_x08

Commit message: Improved schematics and docs
Connections:
- net D1: now reaches D111.18 (B1)
- net D0: now reaches D111.19 (B0)
- net +5V: now reaches R11.1 (R1.1)
Changed lines of the file:
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@@
     (rev "1")
   )
+  (junction (at 350.52 33.02) (diameter 0) (color 0 0 0 0)
+  )
   (no_connect (at 297.18 336.55))
+  (bus_entry (at 138.43 106.68) (size 2.54 2.54)
+    (stroke (width 0) (type default) (color 0 0 0 0))
+  )
+  (bus_entry (at 350.52 49.53) (size -2.54 2.54)
+    (stroke (width 0) (type default) (color 0 0 0 0))
+  )
+  (bus_entry (at 350.52 54.61) (size -2.54 2.54)
+    (stroke (width 0) (type default) (color 0 0 0 0))
+  )
+  (bus_entry (at 350.52 44.45) (size -2.54 2.54)
+    (stroke (width 0) (type default) (color 0 0 0 0))
+  )
+  (bus_entry (at 350.52 39.37) (size -2.54 2.54)
+    (stroke (width 0) (type default) (color 0 0 0 0))
+  )
+  (bus_entry (at 138.43 104.14) (size 2.54 2.54)
+    (stroke (width 0) (type default) (color 0 0 0 0))
+  )
+  (bus (pts (xy 350.52 33.02) (xy 433.07 33.02))
+    (stroke (width 0) (type default) (color 0 0 0 0))
+  )
+  (bus (pts (xy 350.52 49.53) (xy 350.52 54.61))
+    (stroke (width 0) (type default) (color 0 0 0 0))
+  )
+  (bus (pts (xy 24.13 92.71) (xy 24.13 97.79))
+    (stroke (width 0) (type default) (color 0 0 0 0))
+  )
+  (bus (pts (xy 340.36 33.02) (xy 350.52 33.02))
+    (stroke (width 0) (type default) (color 0 0 0 0))
+  )
+  (bus (pts (xy 350.52 44.45) (xy 350.52 49.53))
+    (stroke (width 0) (type default) (color 0 0 0 0))
+  )
+  (bus (pts (xy 350.52 39.37) (xy 350.52 44.45))
+    (stroke (width 0) (type default) (color 0 0 0 0))
+  )
+  (bus (pts (xy 350.52 33.02) (xy 350.52 39.37))
+    (stroke (width 0) (type default) (color 0 0 0 0))
+  )
+  (wire (pts (xy 337.82 41.91) (xy 347.98 41.91))
+    (stroke (width 0) (type default) (color 0 0 0 0))
+  )
+  (wire (pts (xy 337.82 57.15) (xy 347.98 57.15))
+    (stroke (width 0) (type default) (color 0 0 0 0))
+  )
+  (wire (pts (xy 140.97 109.22) (xy 147.32 109.22))
+    (stroke (width 0) (type default) (color 0 0 0 0))
+  )
+  (bus (pts (xy 350.52 54.61) (xy 350.52 104.14))
+    (stroke (width 0) (type default) (color 0 0 0 0))
+  )
+  (bus (pts (xy 138.43 97.79) (xy 138.43 104.14))
+    (stroke (width 0) (type default) (color 0 0 0 0))
+  )
+  (wire (pts (xy 140.97 106.68) (xy 147.32 106.68))
+    (stroke (width 0) (type default) (color 0 0 0 0))
+  )
+  (wire (pts (xy 337.82 52.07) (xy 347.98 52.07))
+    (stroke (width 0) (type default) (color 0 0 0 0))
+  )
+  (wire (pts (xy 337.82 46.99) (xy 347.98 46.99))
+    (stroke (width 0) (type default) (color 0 0 0 0))
+  )
+  (bus (pts (xy 138.43 104.14) (xy 138.43 106.68))
+    (stroke (width 0) (type default) (color 0 0 0 0))
+  )
+  (bus (pts (xy 24.13 97.79) (xy 138.43 97.79))
+    (stroke (width 0) (type default) (color 0 0 0 0))
+  )
+  (bus (pts (xy 433.07 33.02) (xy 433.07 38.1))
+    (stroke (width 0) (type default) (color 0 0 0 0))
+  )
+  (bus (pts (xy 138.43 106.68) (xy 138.43 172.72))
+    (stroke (width 0) (type default) (color 0 0 0 0))
+  )
+  (wire (pts (xy 31.75 121.92) (xy 35.56 121.92))
+    (stroke (width 0) (type default) (color 0 0 0 0))
+  )
+  (label "2" (at 345.44 41.91 0)
+    (effects (font (size 1.27 1.27)) (justify left bottom))
+  )
+  (label "D0" (at 142.24 106.68 0)
+    (effects (font (size 1.27 1.27)) (justify left bottom))
+  )
+  (label "0" (at 345.44 57.15 0)
+    (effects (font (size 1.27 1.27)) (justify left bottom))
+  )
+  (label "D[0..15]" (at 40.64 97.79 0)
+    (effects (font (size 1.27 1.27)) (justify left bottom))
+  )
+  (label "D1" (at 142.24 109.22 0)
+    (effects (font (size 1.27 1.27)) (justify left bottom))
+  )
+  (label "3" (at 345.44 52.07 0)
+    (effects (font (size 1.27 1.27)) (justify left bottom))
+  )
+  (label "1" (at 345.44 46.99 0)
+    (effects (font (size 1.27 1.27)) (justify left bottom))
+  )
+  (global_label "{[0..8], ~{RAS0}, ~{RAS1}, ~{CASL}, ~{CASH}}" (shape input) (at 433.07 33.02 0) (fields_autoplaced)
+    (effects (font (size 1.27 1.27)) (justify left))
+    (property "Intersheet References" "${INTERSHEET_REFS}" (id 0) (at 467.749 32.9406 0)
+      (effects (font (size 1.27 1.27)) (justify left) hide)
+    )
+  )
+  (global_label "D[0..15]" (shape input) (at 24.13 96.52 0) (fields_autoplaced)
+    (effects (font (size 1.27 1.27)) (justify left))
+    (property "Intersheet References" "${INTERSHEET_REFS}" (id 0) (at 34.2556 96.4406 0)
+      (effects (font (size 1.27 1.27)) (justify left) hide)
+    )
+  )
+  (hierarchical_label "D[0..15]" (shape input) (at 24.13 93.98 0)
+    (effects (font (size 1.27 1.27)) (justify left))
+  )
+  (hierarchical_label "{[0..8], ~{RAS0}, ~{RAS1}, ~{CASL}, ~{CASH}}" (shape input) (at 433.07 38.1 0)
+    (effects (font (size 1.27 1.27)) (justify left))
+  )
   (symbol (lib_id "robotron_ec1834:U2764") (at 67.31 62.23 0) (unit 1)
     (in_bom yes) (on_board yes)
@@
   (symbol (lib_id "Device:R_Pack04_SIP_Split") (at 323.85 46.99 90) (unit 1)
     (in_bom yes) (on_board yes)
-    (property "Reference" "R15" (id 0) (at 331.47 48.26 90))
+    (property "Reference" "R15" (id 0) (at 341.63 48.26 90))
     (property "Value" "30" (id 1) (at 323.85 46.99 90))
     (property "Footprint" "Resistor_THT:R_Array_SIP8" (id 2) (at 323.85 49.022 90)
@@
   (symbol (lib_id "Device:R_Pack04_SIP_Split") (at 323.85 41.91 90) (unit 2)
     (in_bom yes) (on_board yes)
-    (property "Reference" "R15" (id 0) (at 331.47 43.18 90))
+    (property "Reference" "R15" (id 0) (at 341.63 43.18 90))
     (property "Value" "30" (id 1) (at 323.85 41.91 90))
     (property "Footprint" "Resistor_THT:R_Array_SIP8" (id 2) (at 323.85 43.942 90)
@@
   (symbol (lib_id "Device:R_Pack04_SIP_Split") (at 323.85 57.15 270) (mirror x) (unit 3)
     (in_bom yes) (on_board yes)
-    (property "Reference" "R15" (id 0) (at 331.47 58.42 90))
+    (property "Reference" "R15" (id 0) (at 341.63 58.42 90))
     (property "Value" "30" (id 1) (at 323.85 57.15 90))
     (property "Footprint" "Resistor_THT:R_Array_SIP8" (id 2) (at 323.85 59.182 90)
@@
   (symbol (lib_id "Device:R_Pack04_SIP_Split") (at 323.85 52.07 90) (unit 4)
     (in_bom yes) (on_board yes)
-    (property "Reference" "R15" (id 0) (at 331.47 53.34 90))
+    (property "Reference" "R15" (id 0) (at 341.63 53.34 90))
     (property "Value" "30" (id 1) (at 323.85 52.07 90))
     (property "Footprint" "Resistor_THT:R_Array_SIP8" (id 2) (at 323.85 54.102 90)
@@
     (pin "2")
   )
+  (symbol (lib_id "power:+5V") (at 31.75 121.92 0) (unit 1)
+    (in_bom yes) (on_board yes) (fields_autoplaced)
+    (property "Reference" "#PWR?" (id 0) (at 31.75 125.73 0)
+      (effects (font (size 1.27 1.27)) hide)
+    )
+    (property "Value" "+5V" (id 1) (at 31.75 118.3442 0))
+    (property "Footprint" "" (id 2) (at 31.75 121.92 0)
+      (effects (font (size 1.27 1.27)) hide)
+    )
+    (property "Datasheet" "" (id 3) (at 31.75 121.92 0)
+      (effects (font (size 1.27 1.27)) hide)
+    )
+    (pin "1")
+  )
 )

Commit message: Improved schematics
Parts:
- removed unit 1 of R12
- removed R22: 130, symbol Device:R
- removed R30, R31: 30, symbol Device:R
- removed R32, R33, R4: 1k, symbol Device:R
- added C7, K?: 680pF, Capacitor_THT:C_Disc_D4.3mm_W1.9mm_P5.00mm, symbol Device:C
- R17, R18, R24, R25: footprint (none) -> Resistor_THT:R_Axial_DIN0309_L9.0mm_D3.2mm_P12.70mm_Horizontal
- SW1: footprint (none) -> Button_Switch_THT:SW_DIP_SPSTx08_Slide_9.78x22.5mm_W7.62mm_P2.54mm
Changed lines of the file:
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@@
     (property "Reference" "SW1" (id 0) (at 262.89 309.4482 0))
     (property "Value" "SW_DIP_x08" (id 1) (at 262.89 311.7596 0))
-    (property "Footprint" "" (id 2) (at 262.89 326.39 0)
+    (property "Footprint" "Button_Switch_THT:SW_DIP_SPSTx08_Slide_9.78x22.5mm_W7.62mm_P2.54mm" (id 2) (at 262.89 326.39 0)
       (effects (font (size 1.27 1.27)) hide)
     )
@@
     (pin "10")
   )
-  (symbol (lib_id "Device:R_Network09_Split") (at 491.49 280.67 90) (unit 1)
-    (in_bom yes) (on_board yes)
-    (property "Reference" "R12" (id 0) (at 491.49 274.955 90))
-    (property "Value" "4k7" (id 1) (at 491.49 277.2664 90))
-    (property "Footprint" "Resistor_THT:R_Array_SIP10" (id 2) (at 491.49 282.702 90)
-      (effects (font (size 1.27 1.27)) hide)
-    )
-    (property "Datasheet" "http://www.vishay.com/docs/31509/csc.pdf" (id 3) (at 491.49 280.67 0)
-      (effects (font (size 1.27 1.27)) hide)
-    )
-    (pin "1")
-    (pin "2")
-    (pin "3")
-    (pin "4")
-    (pin "5")
-    (pin "6")
-    (pin "7")
-    (pin "8")
-    (pin "9")
-    (pin "10")
-  )
   (symbol (lib_id "Device:R_Network09_Split") (at 220.98 220.98 90) (unit 4)
     (in_bom yes) (on_board yes)
@@
     (property "Reference" "R17" (id 0) (at 93.98 168.7322 90))
     (property "Value" "4k7" (id 1) (at 93.98 171.0436 90))
-    (property "Footprint" "" (id 2) (at 93.98 172.212 90)
+    (property "Footprint" "Resistor_THT:R_Axial_DIN0309_L9.0mm_D3.2mm_P12.70mm_Horizontal" (id 2) (at 93.98 172.212 90)
       (effects (font (size 1.27 1.27)) hide)
     )
@@
     (property "Reference" "R18" (id 0) (at 342.9 182.7022 90))
     (property "Value" "30" (id 1) (at 342.9 185.0136 90))
-    (property "Footprint" "" (id 2) (at 342.9 186.182 90)
+    (property "Footprint" "Resistor_THT:R_Axial_DIN0309_L9.0mm_D3.2mm_P12.70mm_Horizontal" (id 2) (at 342.9 186.182 90)
       (effects (font (size 1.27 1.27)) hide)
     )
@@
     (property "Reference" "R24" (id 0) (at 256.54 373.38 90))
     (property "Value" "1k" (id 1) (at 259.08 368.3 90))
-    (property "Footprint" "" (id 2) (at 260.858 368.3 90)
+    (property "Footprint" "Resistor_THT:R_Axial_DIN0309_L9.0mm_D3.2mm_P12.70mm_Horizontal" (id 2) (at 260.858 368.3 90)
       (effects (font (size 1.27 1.27)) hide)
     )
@@
     (property "Reference" "R25" (id 0) (at 250.19 373.38 90))
     (property "Value" "1k" (id 1) (at 252.73 368.3 90))
-    (property "Footprint" "" (id 2) (at 254.508 368.3 90)
+    (property "Footprint" "Resistor_THT:R_Axial_DIN0309_L9.0mm_D3.2mm_P12.70mm_Horizontal" (id 2) (at 254.508 368.3 90)
       (effects (font (size 1.27 1.27)) hide)
     )
@@
     (pin "8")
   )
-  (symbol (lib_id "Device:R") (at 455.93 273.05 90) (unit 1)
-    (in_bom yes) (on_board yes)
-    (property "Reference" "R22" (id 0) (at 455.93 270.51 90))
-    (property "Value" "130" (id 1) (at 455.93 273.05 90))
-    (property "Footprint" "" (id 2) (at 455.93 274.828 90)
-      (effects (font (size 1.27 1.27)) hide)
-    )
-    (property "Datasheet" "~" (id 3) (at 455.93 273.05 0)
-      (effects (font (size 1.27 1.27)) hide)
-    )
-    (pin "1")
-    (pin "2")
-  )
-  (symbol (lib_id "Device:R") (at 468.63 266.7 0) (unit 1)
-    (in_bom yes) (on_board yes)
-    (property "Reference" "R32" (id 0) (at 471.17 266.7 90))
-    (property "Value" "1k" (id 1) (at 468.63 266.7 90))
-    (property "Footprint" "" (id 2) (at 466.852 266.7 90)
-      (effects (font (size 1.27 1.27)) hide)
-    )
-    (property "Datasheet" "~" (id 3) (at 468.63 266.7 0)
-      (effects (font (size 1.27 1.27)) hide)
-    )
-    (pin "1")
-    (pin "2")
-  )
-  (symbol (lib_id "Device:R") (at 459.74 292.1 0) (unit 1)
-    (in_bom yes) (on_board yes)
-    (property "Reference" "R30" (id 0) (at 462.28 292.1 90))
-    (property "Value" "30" (id 1) (at 459.74 292.1 90))
-    (property "Footprint" "" (id 2) (at 457.962 292.1 90)
-      (effects (font (size 1.27 1.27)) hide)
-    )
-    (property "Datasheet" "~" (id 3) (at 459.74 292.1 0)
-      (effects (font (size 1.27 1.27)) hide)
-    )
-    (pin "1")
-    (pin "2")
-  )
-  (symbol (lib_id "Device:R") (at 468.63 316.23 0) (unit 1)
-    (in_bom yes) (on_board yes)
-    (property "Reference" "R31" (id 0) (at 471.17 316.23 90))
-    (property "Value" "30" (id 1) (at 468.63 316.23 90))
-    (property "Footprint" "" (id 2) (at 466.852 316.23 90)
-      (effects (font (size 1.27 1.27)) hide)
-    )
-    (property "Datasheet" "~" (id 3) (at 468.63 316.23 0)
-      (effects (font (size 1.27 1.27)) hide)
-    )
-    (pin "1")
-    (pin "2")
-  )
-  (symbol (lib_id "Device:R") (at 476.25 323.85 0) (unit 1)
-    (in_bom yes) (on_board yes)
-    (property "Reference" "R33" (id 0) (at 478.79 323.85 90))
-    (property "Value" "1k" (id 1) (at 476.25 323.85 90))
-    (property "Footprint" "" (id 2) (at 474.472 323.85 90)
-      (effects (font (size 1.27 1.27)) hide)
-    )
-    (property "Datasheet" "~" (id 3) (at 476.25 323.85 0)
-      (effects (font (size 1.27 1.27)) hide)
-    )
-    (pin "1")
-    (pin "2")
-  )
-  (symbol (lib_id "Device:R") (at 491.49 266.7 90) (unit 1)
-    (in_bom yes) (on_board yes)
-    (property "Reference" "R4" (id 0) (at 491.49 264.16 90))
-    (property "Value" "1k" (id 1) (at 491.49 266.7 90))
-    (property "Footprint" "" (id 2) (at 491.49 268.478 90)
-      (effects (font (size 1.27 1.27)) hide)
-    )
-    (property "Datasheet" "~" (id 3) (at 491.49 266.7 0)
+  (symbol (lib_id "Device:C") (at 234.95 368.3 0) (unit 1)
+    (in_bom yes) (on_board yes)
+    (property "Reference" "C7" (id 0) (at 229.87 365.76 0)
+      (effects (font (size 1.27 1.27)) (justify left))
+    )
+    (property "Value" "680pF" (id 1) (at 238.76 370.84 90)
+      (effects (font (size 1.27 1.27)) (justify left))
+    )
+    (property "Footprint" "Capacitor_THT:C_Disc_D4.3mm_W1.9mm_P5.00mm" (id 2) (at 235.9152 372.11 0)
+      (effects (font (size 1.27 1.27)) hide)
+    )
+    (property "Datasheet" "~" (id 3) (at 234.95 368.3 0)
+      (effects (font (size 1.27 1.27)) hide)
+    )
+    (pin "1")
+    (pin "2")
+  )
+  (symbol (lib_id "Device:C") (at 243.84 368.3 0) (unit 1)
+    (in_bom yes) (on_board yes)
+    (property "Reference" "K?" (id 0) (at 238.76 373.38 0)
+      (effects (font (size 1.27 1.27)) (justify left))
+    )
+    (property "Value" "680pF" (id 1) (at 247.65 370.84 90)
+      (effects (font (size 1.27 1.27)) (justify left))
+    )
+    (property "Footprint" "Capacitor_THT:C_Disc_D4.3mm_W1.9mm_P5.00mm" (id 2) (at 244.8052 372.11 0)
+      (effects (font (size 1.27 1.27)) hide)
+    )
+    (property "Datasheet" "~" (id 3) (at 243.84 368.3 0)
       (effects (font (size 1.27 1.27)) hide)
     )
@@
   (symbol (lib_id "power:+5V") (at 31.75 121.92 0) (unit 1)
     (in_bom yes) (on_board yes) (fields_autoplaced)
-    (property "Reference" "#PWR?" (id 0) (at 31.75 125.73 0)
-      (effects (font (size 1.27 1.27)) hide)
-    )
+    (property "Reference" "#PWR0118" (id 0) (at 31.75 125.73 0)
+      (effects (font (size 1.27 1.27)) hide)
+    )

Commit message: Almsot completed page 1
Parts:
- gave numbers to parts that had none: 1
Changed lines of the file:
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@@
   (symbol (lib_id "Device:C") (at 243.84 368.3 0) (unit 1)
     (in_bom yes) (on_board yes)
-    (property "Reference" "K?" (id 0) (at 238.76 373.38 0)
+    (property "Reference" "C8" (id 0) (at 238.76 373.38 0)
       (effects (font (size 1.27 1.27)) (justify left))
     )

Commit message: Corrected schema names added bus signals
Parts:
- removed C7, C8: 680pF, Capacitor_THT:C_Disc_D4.3mm_W1.9mm_P5.00mm, symbol Device:C
- removed D10, D16, D39: DL000D, symbol RFT_Digitalschaltkreise:DL000D
- removed D100, D101, D115, D116: U2764, symbol robotron_ec1834:U2764
- removed D111, D112, D44: DS8286D-D111, symbol robotron_ec1834:DS8286D-D111
- removed D13, D67: DL074, symbol robotron_ec1834:DL074
- removed D30, D31: DL374, symbol robotron_ec1834:DL374
- removed D34, D59, D82, D87: DL004D, symbol RFT_Digitalschaltkreise:DL004D
- removed D37, D62: DL032D, symbol RFT_Digitalschaltkreise:DL032D
- removed D47: DL008D, symbol robotron_ec1834:DL008D
- removed D5: DL030D, symbol RFT_Digitalschaltkreise:DL030D
- removed D52, D58, D60: 74HC74, symbol robotron_ec1834:74HC74
- removed D53: KR580WI53, Package_DIP:DIP-24_W15.24mm, symbol robotron_ec1834:KR580WI53
- removed D54: 8255A, Package_DIP:DIP-40_W15.24mm, symbol robotron_ec1834:8255A
- removed D55: UC8821, EC1834-Board:EMR-64_W22.86mm, symbol robotron_ec1834:UC8821
- removed D56: 2716, Package_DIP:DIP-24_W15.24mm, symbol robotron_ec1834:2716
- removed D57, D69, D70, D72, D88: DL008D, symbol RFT_Digitalschaltkreise:DL008D
- removed D63: DL010D-D63, symbol robotron_ec1834:DL010D-D63
- removed D65, D66: DS8205, symbol robotron_ec1834:DS8205
- removed D68: 74S51, symbol robotron_ec1834:74S51
- removed D71: DL002D, symbol RFT_Digitalschaltkreise:DL002D
- removed D85, D86: KR531KP11, symbol robotron_ec1834:KR531KP11
- removed D90: KR531LI1, symbol robotron_ec1834:KR531LI1
- removed R11: 1k, Resistor_THT:R_Array_SIP6, symbol Device:R_Network05_Split
- removed R12: 4k7, Resistor_THT:R_Array_SIP10, symbol Device:R_Network09_Split
- removed R14, R15, R16: 30, Resistor_THT:R_Array_SIP8, symbol Device:R_Pack04_SIP_Split
- removed R17: 4k7, Resistor_THT:R_Axial_DIN0309_L9.0mm_D3.2mm_P12.70mm_Horizontal, symbol Device:R
- removed R18: 30, Resistor_THT:R_Axial_DIN0309_L9.0mm_D3.2mm_P12.70mm_Horizontal, symbol Device:R
- removed R23: 4k7, Resistor_THT:R_Array_SIP10, symbol Device:R_Network09
- removed R24, R25: 1k, Resistor_THT:R_Axial_DIN0309_L9.0mm_D3.2mm_P12.70mm_Horizontal, symbol Device:R
- removed R40, R41: 4k7, Resistor_THT:R_Array_SIP9, symbol Device:R_Network08
- removed R52: 3k9, Resistor_THT:R_Array_SIP8, symbol Device:R_Network07_Split
- removed SW1: SW_DIP_x08, Button_Switch_THT:SW_DIP_SPSTx08_Slide_9.78x22.5mm_W7.62mm_P2.54mm, symbol Switch:SW_DIP_x08
- added Br4: Br4, Resistor_THT:R_Axial_DIN0204_L3.6mm_D1.6mm_P5.08mm_Horizontal, symbol Jumper:SolderJumper_2_Bridged
- added C10: 10pF, Capacitor_THT:C_Disc_D4.3mm_W1.9mm_P5.00mm, symbol Device:C
- added C5: 47µF, Capacitor_THT:CP_Radial_D12.5mm_P5.00mm, symbol Device:C
- added C6: 10nF, Capacitor_THT:C_Disc_D4.3mm_W1.9mm_P5.00mm, symbol Device:C
- added D1: K1810WM87, Package_DIP:DIP-40_W15.24mm, symbol robotron_ec1834:K1810WM87
- added D10, D16, D32, D39: DL000D, symbol RFT_Digitalschaltkreise:DL000D
- added D11, D3: DL020D, symbol RFT_Digitalschaltkreise:DL020D
- added D12, D40, D47, D88: DL008D, symbol RFT_Digitalschaltkreise:DL008D
- added D126, D13, D15, D38, D51, D67: DL074, symbol robotron_ec1834:DL074
- added D14: DL010D, symbol RFT_Digitalschaltkreise:DL010D
- added D2, D25, D26, D45: DS8282, symbol robotron_ec1834:DS8282
- added D20: K1810WM86, Package_DIP:DIP-40_W15.24mm, symbol robotron_ec1834:K1810WM86
- added D21: DS8286D-D111, symbol robotron_ec1834:DS8286D-D111
- added D22, D83, D84: DS8286D, symbol robotron_ec1834:DS8286D
- added D23, D64: DS8286D-D23, symbol robotron_ec1834:DS8286D-D23
- added D24: DL374, symbol robotron_ec1834:DL374
- added D27: DS8286D-D27, symbol robotron_ec1834:DS8286D-D27
- added D28, D29, D6: DL295, symbol robotron_ec1834:DL295
- added D33, D71: DL002D, symbol RFT_Digitalschaltkreise:DL002D
- added D34, D59, D8, D87: DL004D, symbol RFT_Digitalschaltkreise:DL004D
- added D35, D36: DL175, symbol robotron_ec1834:DL175
- added D37, D62, D7: DL032D, symbol RFT_Digitalschaltkreise:DL032D
- added D4: KR1810WG88, Package_DIP:DIP-20_W7.62mm, symbol robotron_ec1834:KR1810WG88
- added D42: A302D, Package_DIP:DIP-4_W7.62mm, symbol robotron_ec1834:A302D
- added D43: 8284, Package_DIP:DIP-18_W7.62mm, symbol robotron_ec1834:8284
- added D46, D61: DS8216, symbol robotron_ec1834:DS8216
- added D48, D49: KR580WN59A, Package_DIP:DIP-28_W15.24mm, symbol robotron_ec1834:KR580WN59A
- added D50: KR580IK57, Package_DIP:DIP-40_W15.24mm, symbol robotron_ec1834:KR580IK57
- added D63: DL010D-D63, symbol robotron_ec1834:DL010D-D63
- added D89, D9: DS8205, symbol robotron_ec1834:DS8205
- added E1, E2, E5: SolderJumper_2_Bridged, symbol Connector_Generic:Conn_02x01
- added PS1, PS2: Conn_01x03, symbol Connector_Generic:Conn_01x03
- added R1, R2: 4k7, Resistor_THT:R_Axial_DIN0309_L9.0mm_D3.2mm_P12.70mm_Horizontal, symbol Device:R
- added R10, R12: 4k7, Resistor_THT:R_Array_SIP10, symbol Device:R_Network09_Split
- added R11: 1k, Resistor_THT:R_Array_SIP6, symbol Device:R_Network05_Split
- added R13: 4,7k, Resistor_THT:R_Axial_DIN0309_L9.0mm_D3.2mm_P12.70mm_Horizontal, symbol Device:R
- added R19: 18k, Resistor_THT:R_Axial_DIN0309_L9.0mm_D3.2mm_P12.70mm_Horizontal, symbol Device:R
- added R20: 180k, Resistor_THT:R_Axial_DIN0309_L9.0mm_D3.2mm_P12.70mm_Horizontal, symbol Device:R
- added R21: 100k, Resistor_THT:R_Axial_DIN0309_L9.0mm_D3.2mm_P12.70mm_Horizontal, symbol Device:R
- added R3, R7, R8: 30, Resistor_THT:R_Axial_DIN0309_L9.0mm_D3.2mm_P12.70mm_Horizontal, symbol Device:R
- added R5, R6: 511, Resistor_THT:R_Axial_DIN0309_L9.0mm_D3.2mm_P12.70mm_Horizontal, symbol Device:R
- added R50, R51: 100, Resistor_THT:R_Axial_DIN0309_L9.0mm_D3.2mm_P12.70mm_Horizontal, symbol Device:R
- added R52: 3k9, Resistor_THT:R_Array_SIP8, symbol Device:R_Network07_Split
- added R9: 30, Resistor_THT:R_Array_SIP8, symbol Device:R_Pack04_SIP_Split
- added V1: 14745,6KHz, Crystal:Crystal_HC18-U_Horizontal, symbol Device:Crystal
- added V2: SAY30, symbol Device:D
- added W2, W3: Conn_01x01, symbol Connector_Generic:Conn_01x01
- added WD1: WD1, symbol Jumper:SolderJumper_2_Bridged
- added WD2: WD2, symbol Jumper:SolderJumper_2_Bridged
- added WD3: WD3, symbol Jumper:SolderJumper_2_Bridged
- added X6: Conn_02x01, symbol Connector_Generic:Conn_02x01
Connections:
- net +5V: now also D1.40 (VCC), D11.12 (C2), D126.1 (R), D13.4 (S), D15.1 (R), D15.10 (S), D15.13 (R), D15.4 (S), D20.40 (VCC), D28.06 (V), D29.06 (V), D38.1 (R), D42.1, D43.18 (VCC), D47.9 (A3), D51.10 (S), D6.06 (V), R1.1, R10.1 (R1.1), R13.2, R19.2, R2.2, R52.1 (R1.1)
- net 1: now also D50.37 (A4), D64.5 (A4)
- net 2: now also D50.38 (A5), D64.6 (A5)
- net 3: now also D50.39 (A6), D64.7 (A6)
- net D0: now also D22.19 (B0), D23.12 (B7), D24.13 (D4)
- net D1: now also D22.18 (B1), D23.13 (B6), D24.8 (D3)
- new net: D16.3 (Y1), D22.11 (T)
- new net: D22.9 (OE), R12.7 (R6.2), WD3.2 (B)
- new net: D12.8 (Y3), D38.4 (S)
- new net: D12.9 (A3), D36.14
- new net: D34.4 (Y2), D38.3 (C)
- new net: D15.2 (D), D38.6
- new net: D15.5, D36.4 (D1)
- new net: D12.3 (Y1), D36.1 (R), D36.1 (R), D36.1 (R), D36.1 (R)
- new net: D36.2, D39.9 (A3)
- new net: D36.5 (D2), D39.11 (Y4)
- new net: D36.6, D39.12 (A4)
- new net: D15.12 (D), D24.11 (C), D32.9 (A3), D36.12 (D3), D36.7
- new net: D11.9 (A2), D36.10, D36.13 (D4)
- new net: D32.10 (B3), D36.11
- new net: D13.2 (D), D36.15
- new net: D13.3 (C), D59.10 (Y5)
- new net: D12.1 (A1), D13.6
- new net: D11.8 (Y2), WD2.2 (B)
- new net: D12.4 (A2), D32.8 (Y3)
- new net: D39.13 (B4), D39.8 (Y3)
- new net: D89.07 (O7), W3.1 (Pin_1)
- new net: D1.23 (BUSY), D20.23 (TEST), R2.1
- new net: D4.5 (ALE), R8.2
- new net: D43.1 (CSYN), PS2.1 (Pin_1), R51.2
- new net: C6.2, D42.4, D43.11 (RES), R19.1, X6.2 (Pin_2)
- new net: D43.12 (OSC), E5.1 (Pin_1)
- new net: D43.13 (F/C), E2.2 (Pin_2)
- new net: D43.14 (EFI), PS2.3 (Pin_3), W2.1 (Pin_1)
- new net: D43.15 (ASYN), E1.2 (Pin_2)
- new net: D43.16 (X2), R5.2, V1.1
- new net: C10.1, D43.17 (X1), R6.1
- new net: D43.2 (PC), R7.2
- new net: D126.2 (D), D14.12 (Y1), D43.3 (AEN1)
- new net: D126.6, D43.4 (RDY1)
- new net: D43.8 (CLK), R3.2
- new net: C5.2, D42.2, R20.1, R21.2, V2.2 (A)
- new net: D46.04 (DI0), D7.10 (B3), D7.11 (Y4)
- new net: D23.9 (OE), D7.8 (Y3)
- new net: D24.1 (OE), R12.8 (R7.2), WD2.1 (A)
- new net: D33.4 (Y2), D6.08 (CS)
- new net: D6.09 (C), D8.6 (Y3)
- new net: D28.08 (CS), D33.10 (Y3)
- new net: D28.09 (C), D8.8 (Y4)
- new net: D29.08 (CS), D33.13 (Y4)
- new net: D29.09 (C), D8.10 (Y5)
- new net: D33.5 (A2), D40.3 (Y1)
- new net: D8.5 (A3), D9.07 (O7)
- new net: D8.9 (A4), D9.10 (O5)
- new net: D8.11 (A5), D9.09 (O6)
- new net: D35.6, D40.9 (A3)
- new net: D45.9 (OE), D61.01 (CS), D62.3 (Y1), D64.9 (OE)
- new net: D45.11 (STN), D50.8 (ADSTB)
- new net: D35.4 (D1), D37.3 (Y1)
- new net: D35.10, D35.13 (D4)
- new net: D35.11, D47.2 (B1), D67.13 (R)
- new net: D35.12 (D3), D67.9
- new net: D37.2 (B1), D38.9, D51.2 (D)
- new net: D34.2 (Y1), D38.12 (D)
- new net: D3.8 (Y2), D34.1 (A1)
- new net: D47.10 (B3), D50.36 (TC)
- new net: D49.16 (SP), R12.10 (R9.2)
- new net: D14.9 (A3), D33.1 (Y1)
- new net: D14.11 (C3), D32.2 (B1), D40.5 (B2), D88.8 (Y3)
- new net: D14.10 (B3), D32.6 (Y2), D40.4 (A2), D59.11 (A5)
- new net: D16.2 (B1), D16.6 (Y2)
- new net: D16.1 (A1), D32.11 (Y4)
- new net: D32.3 (Y1), D40.12 (A4)
- new net: D47.11 (Y4), D63.5 (C2)
- new net: D40.6 (Y2), D7.1 (A1)
- new net: D63.4 (B2), D7.3 (Y1)
- new net: D14.8 (Y3), D34.3 (A2)
- new net: D7.4 (A2), D7.9 (A3), D8.4 (Y2)
- new net: D7.12 (A4), D88.11 (Y4)
- new net: D15.9, D7.13 (B4)
- new net: D40.11 (Y4), D63.3 (A2)
- new net: D63.6 (Y2), WD3.1 (A)
- new net: E2.1 (Pin_1), PS2.2 (Pin_2), R50.2
- new net: C10.2, V1.2
- new net +12V: R20.2, V2.1 (K)
- new net 4: D50.40 (A7), D64.8 (A7)
- new net 5PW1: D1.33 (~{GT1}), D20.31 (~{GT0}), D43.7 (AEN2), E1.1 (Pin_1)
- new net 5PW2: D64.11 (T), D83.11 (T), D84.11 (T), D9.06 (E3)
- new net A0: D2.18 (DO1), D40.13 (B4), D46.03 (DB0), D64.19 (B0)
- new net A1: D26.19 (DO0), D64.18 (B1), D83.2 (A1)
- new net A10: D25.17 (DO2), D45.17 (DO2), D84.3 (A2)
- new net A11: D25.16 (DO3), D45.16 (DO3), D84.4 (A3)
- new net A12: D25.15 (DO4), D45.15 (DO4), D84.5 (A4)
- new net A13: D25.14 (DO5), D45.14 (DO5), D83.1 (A0)
- new net A14: D25.13 (DO6), D45.13 (DO6)
- new net A15: D25.12 (DO7), D45.12 (DO7)
- new net A16: D2.15 (DO4), D28.13 (F0), D29.13 (F0), D6.13 (F0)
- new net A17: D2.14 (DO5), D28.12 (F1), D29.12 (F1), D6.12 (F1)
- new net A18: D2.13 (DO6), D28.11 (F2), D29.11 (F2), D6.11 (F2)
- new net A19: D2.16 (DO3), D28.10 (F3), D29.10 (F3), D6.10 (F3)
- new net A2: D26.18 (DO1), D64.17 (B2), D83.3 (A2)
- new net A3: D26.17 (DO2), D64.16 (B3), D83.4 (A3)
- new net A4: D26.16 (DO3), D64.15 (B4), D83.5 (A4)
- new net A5: D26.15 (DO4), D64.14 (B5), D83.6 (A5)
- new net A6: D26.14 (DO5), D64.13 (B6), D83.7 (A6)
- new net A7: D26.13 (DO6), D64.12 (B7), D83.8 (A7)
- new net A8: D25.19 (DO0), D45.19 (DO0), D84.1 (A0)
- new net A9: D25.18 (DO1), D45.18 (DO1), D84.2 (A1)
- new net AD0: D1.16 (AD0), D2.2 (DI1), D20.16 (AD0), D23.8 (A7), D24.12 (Q4), D26.8 (DI7)
- new net AD1: D1.15 (AD1), D20.15 (AD1), D23.7 (A6), D24.9 (Q3), D26.1 (DI0)
- new net AD10: D1.6 (AD10), D20.6 (AD10), D21.3 (A2), D25.3 (DI2)
- new net AD11: D1.5 (AD11), D20.5 (AD11), D21.4 (A3), D25.4 (DI3)
- new net AD12: D1.4 (AD12), D20.4 (AD12), D21.5 (A4), D25.5 (DI4)
- new net AD13: D1.3 (AD13), D20.3 (AD13), D21.6 (A5), D25.6 (DI5)
- new net AD14: D1.2 (AD14), D20.2 (AD14), D21.7 (A6), D25.7 (DI6)
- new net AD15: D1.39 (AD15), D20.39 (AD15), D21.8 (A7), D25.8 (DI7)
- new net AD16: D1.38 (A16), D2.5 (DI4), D20.38 (A16)
- new net AD17: D1.37 (A17), D2.6 (DI5), D20.37 (A17)
- new net AD18: D1.36 (A18), D2.7 (DI6), D20.36 (A18)
- new net AD19: D1.35 (A19), D2.4 (DI3), D20.35 (A19)
- new net AD2: D1.14 (AD2), D20.14 (AD2), D23.6 (A5), D24.6 (Q2), D26.2 (DI1)
- new net AD3: D1.13 (AD3), D20.13 (AD3), D23.5 (A4), D24.15 (Q5), D26.3 (DI2)
- new net AD4: D1.12 (AD4), D20.12 (AD4), D23.4 (A3), D24.16 (Q6), D26.4 (DI3)
- new net AD5: D1.11 (AD5), D20.11 (AD5), D23.3 (A2), D24.5 (Q1), D26.5 (DI4)
- new net AD6: D1.10 (AD6), D20.10 (AD6), D23.2 (A1), D24.2 (Q0), D26.6 (DI5)
- new net AD7: D1.9 (AD7), D20.9 (AD7), D23.1 (A0), D24.19 (Q7), D26.7 (DI6)
- new net AD8: D1.8 (AD8), D20.8 (AD8), D21.1 (A0), D25.1 (DI0)
- new net AD9: D1.7 (AD9), D20.7 (AD9), D21.2 (A1), D25.2 (DI1)
- new net AEN: D84.14 (B5)
- new net AENBRD: D12.13 (B4), D27.11 (T), D32.1 (A1), D35.2, D35.5 (D2), D39.1 (A1), D46.01 (CS), D83.9 (OE), WD1.2 (B)
- new net AENBRDW: D2.9 (OE), D25.9 (OE), D26.9 (OE), D4.6 (AEN), R10.10 (R9.2), WD1.1 (A)
- new net AENDMA: D37.1 (A1), D39.2 (B1), D50.9 (AEN)
- new net AENI: D12.11 (Y4), D32.12 (A4), D84.6 (A5)
- new net ALE: D2.11 (STN), D25.11 (STN), D26.11 (STN), R8.1
- new net BHE: D47.12 (A4)
- new net BS-/WAIT: D14.2 (B1), D38.5
- new net CAS0: D48.12 (CAS0), D49.12 (CAS0)
- new net CAS1: D48.13 (CAS1), D49.13 (CAS1)
- new net CAS2: D48.15 (CAS2), D49.15 (CAS2)
- new net CEN: D12.6 (Y2), D4.15 (CEN)
- new net CLK: D35.9 (C), D35.9 (C), D35.9 (C), D35.9 (C), D38.11 (C), D84.13 (B6)
- new net CLK86: D1.19 (CLK), D126.3 (C), D20.19 (CLK), D4.2 (CLK), D84.7 (A6), D87.13 (A6), R3.1
- new net D10: D21.17 (B2), D22.3 (A2)
- new net D11: D21.16 (B3), D22.4 (A3)
- new net D12: D21.15 (B4), D22.5 (A4)
- new net D13: D21.14 (B5), D22.6 (A5)
- new net D14: D21.13 (B6), D22.7 (A6)
- new net D15: D21.12 (B7), D22.8 (A7)
- new net D2: D22.17 (B2), D23.14 (B5), D24.7 (D2)
- new net D3: D22.16 (B3), D23.15 (B4), D24.14 (D5)
- new net D4: D22.15 (B4), D23.16 (B3), D24.17 (D6)
- new net D5: D22.14 (B5), D23.17 (B2), D24.4 (D1)
- new net D6: D22.13 (B6), D23.18 (B1), D24.3 (D0)
- new net D7: D22.12 (B7), D23.19 (B0), D24.18 (D7)
- new net D8: D21.19 (B0), D22.1 (A0)
- new net D9: D21.18 (B1), D22.2 (A1)
- new net DACK0: D51.12 (D), D8.12 (Y6)
- new net DEN: D11.13 (D2), D4.16 (DEN), D8.3 (A2)
- new net DRQ0: D50.19 (DRQ0)
- new net DRQ1: D50.18 (DRQ1)
- new net DRQ2: D50.17 (DRQ2)
- new net DRQ3: D50.16 (DRQ3)
- new net DT-/R: D16.4 (A2), D21.11 (T), D23.11 (T), D4.4 (DT/~{R})
- new net GND: C5.1, C6.1, D1.1 (GND), D1.20 (GND), D20.1 (GND), D20.20 (GND), D20.33 (MAX), D28.01 (A0), D29.01 (A0), D38.2 (D), D4.1 (IOB), D42.3, D43.6 (RDY2), D46.07 (DI1), D46.09 (DI2), D46.12 (DI3), D46.15 (DIEN), D48.16 (SP), D6.01 (A0), D61.04 (DI0), D61.07 (DI1), D61.09 (DI2), D61.15 (DIEN), D84.9 (OE), D9.04 (E1), D9.05 (E2), R21.1, R5.1, R50.1, R51.1, R6.2, X6.1 (Pin_1)
- new net HOLDA: D50.7 (HLDA), D51.4 (S), D51.5, D51.6
- new net HRQDMA: D38.13 (R), D50.10 (HRQ)
- new net IED: D38.10 (S), D38.8, D40.10 (B3)
- new net INT: D20.18 (INTR), D49.17 (INT)
- new net IOCHRDY: D14.1 (A1), D67.10 (S), R13.1
- new net IORW: D10.3 (Y1), D67.11 (C), D7.2 (B1)
- new net IRQ0: D49.18 (IR0)
- new net IRQ1: D49.19 (IR1)
- new net IRQ10: D48.20 (IR2)
- new net IRQ11: D48.21 (IR3)
- new net IRQ12: D48.22 (IR4)
- new net IRQ14: D48.24 (IR6)
- new net IRQ15: D48.25 (IR7)
- new net IRQ2: Br4.1 (A), Br4.2 (B), D48.17 (INT), D48.19 (IR1), D49.20 (IR2)
- new net IRQ3: D49.21 (IR3)
- new net IRQ4: D49.22 (IR4)
- new net IRQ5: D49.23 (IR5)
- new net IRQ6: D49.24 (IR6)
- new net IRQ7: D49.25 (IR7)
- new net IRQ8: D48.18 (IR0), D51.9
- new net MASTER: D27.9 (OE), D33.12 (B4), D33.6 (B2), D33.9 (B3), D62.2 (B1), D8.2 (Y1)
- new net MEMR: D11.10 (B2)
- new net NMI: D20.17 (NMI)
- new net NPNPI: D1.32 (INT), D48.23 (IR5)
- new net OSC1: E5.2 (Pin_2)
- new net PB3: D51.13 (R)
- new net PCLK: D50.12 (CLK), D51.3 (C), R7.1
- new net QS0: D1.25 (QS0), D20.25 (QS0)
- new net QS1: D1.24 (QS1), D20.24 (QS1)
- new net RDY-/WAIT: D14.13 (C1), D47.1 (A1), D67.8
- new net RDYTODMA: D47.3 (Y1)
- new net READY: D1.22 (READY), D20.22 (READY), D43.5 (READY)
- new net RESET: D1.21 (RESET), D20.21 (RESET), D34.11 (A5), D43.10 (RESET), D50.13 (RESET)
- new net RESETDRV: D59.2 (Y1)
- new net TC: D47.8 (Y3), D51.11 (C)
- new net TDYTODMA: D50.6 (RDY)
- new net VA0: D26.12 (DO7), D33.3 (B1), D88.12 (A4)
- new net WRTDMAPGREG: D71.10 (Y3), D9.03 (A2)
- new net XA0: D48.27 (A0), D49.27 (A0), D50.32 (A0), D64.1 (A0), D9.01 (A0)
- new net XA1: D50.33 (A1), D64.2 (A1), D83.18 (B1), D9.02 (A1)
- new net XA10: D84.17 (B2)
- new net XA11: D84.16 (B3)
- new net XA12: D84.15 (B4)
- new net XA13: D83.19 (B0)
- new net XA2: D50.34 (A2), D64.3 (A2), D83.17 (B2)
- new net XA3: D50.35 (A3), D64.4 (A3), D83.16 (B3)
- new net XA4: D83.15 (B4)
- new net XA5: D83.14 (B5), D89.01 (A0)
- new net XA6: D83.13 (B6), D89.02 (A1)
- new net XA7: D83.12 (B7), D89.03 (A2)
- new net XA8: D84.19 (B0), D89.04 (E1)
- new net XA9: D84.18 (B1), D89.05 (E2)
- new net XD0: D28.02 (A1), D29.02 (A1), D45.1 (DI0), D48.11 (D0), D49.11 (D0), D50.30 (DB0), D6.02 (A1)
- new net XD1: D28.03 (A2), D29.03 (A2), D45.2 (DI1), D48.10 (D1), D49.10 (D1), D50.29 (DB1), D6.03 (A2)
- new net XD2: D28.04 (A3), D29.04 (A3), D45.3 (DI2), D48.9 (D2), D49.9 (D2), D50.28 (DB2), D6.04 (A3)
- new net XD3: D28.05 (A4), D29.05 (A4), D45.4 (DI3), D48.8 (D3), D49.8 (D3), D50.27 (DB3), D6.05 (A4)
- new net XD4: D45.5 (DI4), D48.7 (D4), D49.7 (D4), D50.26 (DB4)
- new net XD5: D45.6 (DI5), D48.6 (D5), D49.6 (D5), D50.23 (DB5)
- new net XD6: D45.7 (DI6), D48.5 (D6), D49.5 (D6), D50.22 (DB6)
- new net XD7: D45.8 (DI7), D48.4 (D7), D49.4 (D7), D50.21 (DB7)
- new net ~{A0}: D61.12 (DI3)
- new net ~{AEN}: D12.5 (B2), D16.5 (B2), D35.3, D67.12 (D), D89.06 (E3)
- new net ~{BHE}: D1.34 (BHE), D2.12 (DO7), D2.8 (DI7), D20.34 (BHE), D33.2 (A1), D61.13 (DB3), D7.5 (B2)
- new net ~{CIOR}: D27.14 (B5), D4.13 (IORC), R10.7 (R6.2), R9.6 (R3.2)
- new net ~{CIOW}: D27.12 (B7), D4.12 (AIOWC), R10.9 (R8.2), R9.8 (R4.2)
- new net ~{CLK}: D13.1 (R), D15.11 (C), D15.3 (C), D36.9 (C), D36.9 (C), D36.9 (C), D36.9 (C), D87.12 (Y6)
- new net ~{CMEMR}: D27.18 (B1), D4.7 (MRDC), R10.3 (R2.2), R9.2 (R1.2)
- new net ~{CMEMW}: D27.16 (B3), D4.8 (AMWC), R10.5 (R4.2), R9.4 (R2.2)
- new net ~{CS86H}: D21.9 (OE), D7.6 (Y2)
- new net ~{DACK0BRD}: D50.25 (DACK0), D8.13 (A6), D84.8 (A7)
- new net ~{DACK0}: D40.2 (B1), D84.12 (B7)
- new net ~{DACK1}: D40.1 (A1), D50.24 (DACK1)
- new net ~{DACK2}: D33.8 (A3), D50.14 (DACK2)
- new net ~{DACK3}: D33.11 (A4), D50.15 (DACK3)
- new net ~{DMAAEN}: D39.3 (Y1), D62.1 (A1)
- new net ~{DMACS}: D50.11 (CS), D89.15 (O0)
- new net ~{DMAWAIT}: D126.4 (S), D40.8 (Y3)
- new net ~{F4}: D35.14, D39.10 (B3)
- new net ~{GT1}: D1.31 (~{GT0}), D20.30 (~{GT1}), R1.2
- new net ~{INTA}: D4.14 (~{INTA}), D48.26 (INTA), D49.26 (INTA), D88.13 (B4), R52.2 (R1.2)
- new net ~{INTRCS1}: D49.1 (CS), D89.14 (O1)
- new net ~{INTRCS2}: D48.1 (CS), D89.09 (O6)
- new net ~{IOR}: R9.5 (R3.1)
- new net ~{IOW}: R9.7 (R4.1)
- new net ~{LOCK}: D20.29 (~{LOCK}), D3.13 (D2)
- new net ~{MASTER}: D12.12 (A4), D47.13 (B4), D8.1 (A1), R11.4 (R3.2)
- new net ~{MEMADRSEL}: D88.10 (B3)
- new net ~{MEMCS16}: D88.9 (A3), R11.5 (R4.2)
- new net ~{MEMR}: D32.4 (A2), R9.1 (R1.1)
- new net ~{MEMW}: D32.5 (B2), R9.3 (R2.1)
- new net ~{NMIADRCS}: D71.9 (B3), D89.11 (O4)
- new net ~{NMIREGCS}: D89.10 (O5)
- new net ~{PPICS}: D89.12 (O3)
- new net ~{RESETDRV}: D12.10 (B3), D12.2 (B1), D34.10 (Y5), D35.1 (R), D35.1 (R), D35.1 (R), D35.1 (R), D59.1 (A1), R12.3 (R2.2)
- new net ~{S0}: D1.26 (S0), D20.26 (S0), D3.9 (A2), D4.19 (S0), PS1.1 (Pin_1)
- new net ~{S1}: D1.27 (S1), D20.27 (S1), D3.10 (B2), D4.3 (S1), PS1.2 (Pin_2)
- new net ~{S2}: D1.28 (S2), D20.28 (S2), D3.12 (C2), D4.18 (S2), PS1.3 (Pin_3)
- new net ~{TIMERCS}: D89.13 (O2)
- new net ~{XIOR}: D10.1 (A1), D27.15 (B4), D27.6 (A5), D48.3 (RD), D49.3 (RD), R10.6 (R5.2)
- new net ~{XIOW}: D10.2 (B1), D27.13 (B6), D27.8 (A7), D48.2 (WR), D49.2 (WR), D71.8 (A3), R10.8 (R7.2)
- new net ~{XMEMR}: D27.2 (A1), D50.3 (MEMR), R10.2 (R1.2)
- new net ~{XMEMW}: D27.4 (A3), D32.13 (B4), D50.4 (MEMW), R10.4 (R3.2)
- new net ~{YIOR}: D27.5 (A4), D50.1 (IOR), R12.6 (R5.2), R12.9 (R8.2)
- new net ~{YIOW}: D27.7 (A6), D50.2 (IOW)
- no-connect marks 1 -> 40
Other:
- note added: "5P"
- note added: "Bei der Verwend. d. K1810GF84 entfällt E1"
- note added: "D64A PIN Pos abweichend von Zeichnung 1.13.120030.0/04"
- note added: "WDx - Drahtbrücken"
- note added: "X1 Bus Connector auf Seite "BUS""
- title: EC1834_201.2 -> (none)
