File: EC1834_201.1.kicad_sch (KiCad schematic)
At the start: 91 parts, among them X6 Conn_02x01

Commit message: corrected page names progress on page 2 added 1834 bus symbol
Parts:
- PS1: symbol Connector_Generic:Conn_01x03 -> Connector_Generic:Conn_01x05
Connections:
- new net PS1:4: PS1.4 (Pin_4)
- no-connect marks 40 -> 41
Other:
- note added: "D5 p11 Koord C1 / Blatt 201.2"
Changed lines of the file:
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@@
   (junction (at 257.81 384.81) (diameter 0) (color 0 0 0 0)
   )
+  (junction (at 562.61 347.98) (diameter 0) (color 0 0 0 0)
+  )
   (junction (at 426.72 226.06) (diameter 0) (color 0 0 0 0)
   )
@@
   (no_connect (at 368.3 160.02))
   (no_connect (at 304.8 207.01))
+  (no_connect (at 421.64 260.35))
   (no_connect (at 502.92 138.43))
   (no_connect (at 502.92 133.35))
@@
     (stroke (width 0) (type default) (color 0 0 0 0))
   )
+  (bus (pts (xy 577.85 347.98) (xy 577.85 346.71))
+    (stroke (width 0) (type default) (color 0 0 0 0))
+  )
   (wire (pts (xy 386.08 336.55) (xy 455.93 336.55))
     (stroke (width 0) (type default) (color 0 0 0 0))
@@
     (stroke (width 2) (type default) (color 0 0 0 0))
   )
+  (wire (pts (xy 419.1 261.62) (xy 434.34 261.62))
+    (stroke (width 0) (type default) (color 0 0 0 0))
+  )
   (wire (pts (xy 393.7 213.36) (xy 361.95 213.36))
     (stroke (width 0) (type default) (color 0 0 0 0))
@@
     (stroke (width 2) (type default) (color 0 0 0 0))
   )
+  (bus (pts (xy 562.61 347.98) (xy 577.85 347.98))
+    (stroke (width 0) (type default) (color 0 0 0 0))
+  )
   (wire (pts (xy 265.43 261.62) (xy 322.58 261.62))
     (stroke (width 0) (type default) (color 0 0 0 0))
@@
     (stroke (width 0.5) (type default) (color 0 0 0 0))
   )
+  (wire (pts (xy 419.1 260.35) (xy 419.1 261.62))
+    (stroke (width 0) (type default) (color 0 0 0 0))
+  )
   (bus (pts (xy 78.74 347.98) (xy 78.74 350.52))
     (stroke (width 2) (type default) (color 0 0 0 0))
@@
     (effects (font (size 1.27 1.27)) (justify left bottom))
   )
+  (text "D5 p11\nKoord C1 / Blatt 201.2" (at 429.26 260.35 0)
+    (effects (font (size 1.27 1.27)) (justify left bottom))
+  )
   (text "5P" (at 156.21 123.19 0)
     (effects (font (size 1.27 1.27)) (justify left bottom))
@@
     )
   )
+  (hierarchical_label "XA[0..19]" (shape input) (at 562.61 363.22 0)
+    (effects (font (size 1.27 1.27)) (justify left))
+  )
   (hierarchical_label "D[0..15]" (shape input) (at 542.29 22.86 0)
     (effects (font (size 1.27 1.27)) (justify left))
   )
+  (hierarchical_label "XD[0..15]" (shape input) (at 562.61 372.11 0)
+    (effects (font (size 1.27 1.27)) (justify left))
+  )
+  (hierarchical_label "{AENBRD ~{AEN} MEMR PB3 ~{IOCHCK} BHE DRQ0 ~{DACK0BRD} DACK0 ~{DACK0} ~{INTA} ~{IOR} ~{IOW} ~{XIOR} ~{XIOW} ~{XMEMR} ~{MEMR} ~{MEMW} ~{NMIADRCS} ~{TIMERCS} ~{PPICS} ~{NIMREGCS} IRQ0 IRQ1 OSC OSC1 PCLK CLK86 ~{MEMADRSEL} NMI NPNPI RESET ~{RESETDRV}}" (shape input)
+    (at 577.85 346.71 90)
+    (effects (font (size 1.27 1.27)) (justify left))
+  )
   (hierarchical_label "{A[0..19] VA0 ~{BHE}}" (shape input) (at 542.29 27.94 0)
     (effects (font (size 1.27 1.27)) (justify left))
   )
+  (hierarchical_label "PS1:4" (shape input) (at 434.34 261.62 0)
+    (effects (font (size 1.27 1.27)) (justify left))
+  )
   (symbol (lib_id "robotron_ec1834:DS8286D") (at 213.36 57.15 0) (unit 1)
     (in_bom yes) (on_board yes)
@@
     (pin "1")
   )
-  (symbol (lib_id "Connector_Generic:Conn_01x03") (at 414.02 255.27 90) (unit 1)
+  (symbol (lib_id "Connector_Generic:Conn_01x05") (at 416.56 255.27 90) (unit 1)
     (in_bom yes) (on_board yes) (fields_autoplaced)
-    (property "Reference" "PS1" (id 0) (at 418.592 254.4353 90)
+    (property "Reference" "PS1" (id 0) (at 421.132 254.4353 90)
       (effects (font (size 1.27 1.27)) (justify right))
     )
-    (property "Value" "Conn_01x03" (id 1) (at 418.592 256.9722 90)
+    (property "Value" "Conn_01x03" (id 1) (at 421.132 256.9722 90)
       (effects (font (size 1.27 1.27)) (justify right) hide)
     )
-    (property "Footprint" "" (id 2) (at 414.02 255.27 0)
+    (property "Footprint" "" (id 2) (at 416.56 255.27 0)
       (effects (font (size 1.27 1.27)) hide)
     )
-    (property "Datasheet" "~" (id 3) (at 414.02 255.27 0)
+    (property "Datasheet" "~" (id 3) (at 416.56 255.27 0)
       (effects (font (size 1.27 1.27)) hide)
     )
@@
     (pin "2")
     (pin "3")
+    (pin "4")
+    (pin "5")
   )
   (symbol (lib_id "power:+5V") (at 477.52 314.96 90) (unit 1)
