File: EC1834_201.1.kicad_sch (KiCad schematic)
At the start: 91 parts, among them X6 Conn_02x01

Commit message: Page 1 & 2 connected Hierarchival connections created and tested
Connections:
- net HOLDA: no longer D51.4 (S), D51.6
- net HRQDMA: now also D51.1 (R)
- new net: D51.4 (S), D51.6
Changed lines of the file:
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@@
 (kicad_sch (version 20211123) (generator eeschema)
   (paper "A2")
-  (junction (at 186.69 190.5) (diameter 0) (color 0 0 0 0)
-  )
   (junction (at 111.76 152.4) (diameter 0) (color 0 0 0 0)
   )
@@
   (junction (at 257.81 207.01) (diameter 0) (color 0 0 0 0)
   )
+  (junction (at 132.08 203.2) (diameter 0) (color 0 0 0 0)
+  )
   (junction (at 356.87 232.41) (diameter 0) (color 0 0 0 0)
   )
@@
     (stroke (width 0) (type default) (color 0 0 0 0))
   )
-  (wire (pts (xy 388.62 223.52) (xy 393.7 223.52))
-    (stroke (width 0) (type default) (color 0 0 0 0))
-  )
   (bus (pts (xy 467.36 73.66) (xy 467.36 76.2))
     (stroke (width 0.5) (type default) (color 0 0 0 0))
@@
     (stroke (width 0) (type default) (color 0 0 0 0))
   )
+  (wire (pts (xy 168.91 191.77) (xy 168.91 203.2))
+    (stroke (width 0) (type default) (color 0 0 0 0))
+  )
   (wire (pts (xy 219.71 317.5) (xy 224.79 317.5))
     (stroke (width 0) (type default) (color 0 0 0 0))
@@
     (stroke (width 0) (type default) (color 0 0 0 0))
   )
+  (wire (pts (xy 132.08 203.2) (xy 132.08 217.17))
+    (stroke (width 0) (type default) (color 0 0 0 0))
+  )
   (wire (pts (xy 431.8 287.02) (xy 455.93 287.02))
     (stroke (width 0) (type default) (color 0 0 0 0))
@@
     (stroke (width 0) (type default) (color 0 0 0 0))
   )
-  (wire (pts (xy 248.92 290.83) (xy 242.57 290.83))
-    (stroke (width 0) (type default) (color 0 0 0 0))
-  )
   (wire (pts (xy 469.9 93.98) (xy 480.06 93.98))
     (stroke (width 0) (type default) (color 0 0 0 0))
@@
     (stroke (width 0) (type default) (color 0 0 0 0))
   )
-  (wire (pts (xy 474.98 280.67) (xy 480.06 280.67))
-    (stroke (width 0) (type default) (color 0 0 0 0))
-  )
-  (wire (pts (xy 186.69 185.42) (xy 186.69 190.5))
+  (wire (pts (xy 186.69 185.42) (xy 186.69 223.52))
     (stroke (width 0) (type default) (color 0 0 0 0))
   )
@@
     (stroke (width 0) (type default) (color 0 0 0 0))
   )
-  (wire (pts (xy 474.98 207.01) (xy 480.06 207.01))
-    (stroke (width 0) (type default) (color 0 0 0 0))
-  )
   (bus (pts (xy 458.47 323.85) (xy 458.47 336.55))
     (stroke (width 2) (type default) (color 0 0 0 0))
@@
     (stroke (width 0) (type default) (color 0 0 0 0))
   )
-  (wire (pts (xy 132.08 193.04) (xy 132.08 217.17))
+  (wire (pts (xy 132.08 193.04) (xy 132.08 203.2))
     (stroke (width 0) (type default) (color 0 0 0 0))
   )
@@
     (stroke (width 0) (type default) (color 0 0 0 0))
   )
-  (wire (pts (xy 316.23 196.85) (xy 322.58 196.85))
-    (stroke (width 0) (type default) (color 0 0 0 0))
-  )
   (bus (pts (xy 511.81 27.94) (xy 511.81 46.99))
     (stroke (width 0.5) (type default) (color 0 0 0 0))
@@
     (stroke (width 0) (type default) (color 0 0 0 0))
   )
-  (wire (pts (xy 226.06 354.33) (xy 226.06 359.41))
-    (stroke (width 0) (type default) (color 0 0 0 0))
-  )
   (wire (pts (xy 502.92 285.75) (xy 515.62 285.75))
     (stroke (width 0) (type default) (color 0 0 0 0))
@@
     (stroke (width 0) (type default) (color 0 0 0 0))
   )
+  (wire (pts (xy 168.91 203.2) (xy 132.08 203.2))
+    (stroke (width 0) (type default) (color 0 0 0 0))
+  )
   (wire (pts (xy 176.53 121.92) (xy 167.64 121.92))
     (stroke (width 0) (type default) (color 0 0 0 0))
@@
     (stroke (width 0.5) (type default) (color 0 0 0 0))
   )
-  (wire (pts (xy 186.69 190.5) (xy 186.69 223.52))
-    (stroke (width 0) (type default) (color 0 0 0 0))
-  )
   (bus (pts (xy 236.22 53.34) (xy 236.22 55.88))
     (stroke (width 0.5) (type default) (color 0 0 0 0))
@@
     (stroke (width 0) (type default) (color 0 0 0 0))
   )
-  (wire (pts (xy 369.57 210.82) (xy 375.92 210.82))
-    (stroke (width 0) (type default) (color 0 0 0 0))
-  )
   (wire (pts (xy 392.43 342.9) (xy 392.43 318.77))
     (stroke (width 0) (type default) (color 0 0 0 0))
@@
     (stroke (width 0) (type default) (color 0 0 0 0))
   )
+  (wire (pts (xy 171.45 191.77) (xy 168.91 191.77))
+    (stroke (width 0) (type default) (color 0 0 0 0))
+  )
   (bus (pts (xy 518.16 290.83) (xy 518.16 288.29))
     (stroke (width 0.5) (type default) (color 0 0 0 0))
@@
     (stroke (width 0) (type default) (color 0 0 0 0))
   )
-  (wire (pts (xy 316.23 264.16) (xy 322.58 264.16))
-    (stroke (width 0) (type default) (color 0 0 0 0))
-  )
   (bus (pts (xy 257.81 288.29) (xy 257.81 290.83))
     (stroke (width 0.5) (type default) (color 0 0 0 0))
@@
     (effects (font (size 1.27 1.27)) (justify left bottom))
   )
-  (label "5PW1" (at 474.98 280.67 0)
-    (effects (font (size 1.27 1.27)) (justify left bottom))
-  )
   (label "BS-{slash}WAIT" (at 313.69 212.09 0)
     (effects (font (size 1.27 1.27)) (justify left bottom))
@@
     (effects (font (size 1.27 1.27)) (justify left bottom))
   )
-  (label "5PW1" (at 388.62 223.52 0)
-    (effects (font (size 1.27 1.27)) (justify left bottom))
-  )
   (label "D9" (at 429.26 160.02 0)
     (effects (font (size 1.27 1.27)) (justify left bottom))
@@
     (effects (font (size 1.27 1.27)) (justify left bottom))
   )
-  (label "5PW2" (at 226.06 359.41 90)
-    (effects (font (size 1.27 1.27)) (justify left bottom))
-  )
   (label "XA3" (at 209.55 281.94 0)
     (effects (font (size 1.27 1.27)) (justify left bottom))
@@
     (effects (font (size 1.27 1.27)) (justify left bottom))
   )
-  (label "5PW1" (at 474.98 207.01 0)
-    (effects (font (size 1.27 1.27)) (justify left bottom))
-  )
   (label "A19" (at 502.92 140.97 0)
     (effects (font (size 1.27 1.27)) (justify left bottom))
@@
     (effects (font (size 1.27 1.27)) (justify left bottom))
   )
-  (label "5PW2" (at 316.23 196.85 0)
-    (effects (font (size 1.27 1.27)) (justify left bottom))
-  )
   (label "A13" (at 314.96 176.53 0)
     (effects (font (size 1.27 1.27)) (justify left bottom))
@@
     (effects (font (size 1.27 1.27)) (justify left bottom))
   )
-  (label "5PW2" (at 316.23 264.16 0)
-    (effects (font (size 1.27 1.27)) (justify left bottom))
-  )
   (label "~{MEMCS16}" (at 82.55 96.52 0)
     (effects (font (size 1.27 1.27)) (justify left bottom))
@@
     (effects (font (size 1.27 1.27)) (justify left bottom))
   )
-  (label "5PW1" (at 369.57 210.82 0)
-    (effects (font (size 1.27 1.27)) (justify left bottom))
-  )
   (label "~{XIOR}" (at 444.5 318.77 0)
     (effects (font (size 1.27 1.27)) (justify left bottom))
@@
     (effects (font (size 1.27 1.27)) (justify left bottom))
   )
-  (label "5PW2" (at 248.92 290.83 180)
-    (effects (font (size 1.27 1.27)) (justify right bottom))
-  )
   (label "{A[0..19] VA0 ~{BHE}}" (at 443.23 27.94 0)
     (effects (font (size 1.27 1.27)) (justify left bottom))
@@
     )
   )
+  (hierarchical_label "5PW1" (shape input) (at 480.06 280.67 180)
+    (effects (font (size 1.27 1.27)) (justify right))
+  )
+  (hierarchical_label "5PW1" (shape input) (at 393.7 223.52 180)
+    (effects (font (size 1.27 1.27)) (justify right))
+  )
   (hierarchical_label "XA[0..19]" (shape input) (at 562.61 363.22 0)
     (effects (font (size 1.27 1.27)) (justify left))
   )
+  (hierarchical_label "5PW2" (shape input) (at 226.06 354.33 180)
+    (effects (font (size 1.27 1.27)) (justify right))
+  )
   (hierarchical_label "D[0..15]" (shape input) (at 542.29 22.86 0)
     (effects (font (size 1.27 1.27)) (justify left))
   )
+  (hierarchical_label "5PW2" (shape input) (at 242.57 290.83 0)
+    (effects (font (size 1.27 1.27)) (justify left))
+  )
+  (hierarchical_label "5PW1" (shape input) (at 480.06 207.01 180)
+    (effects (font (size 1.27 1.27)) (justify right))
+  )
+  (hierarchical_label "5PW2" (shape input) (at 322.58 264.16 180)
+    (effects (font (size 1.27 1.27)) (justify right))
+  )
+  (hierarchical_label "5PW2" (shape input) (at 322.58 196.85 180)
+    (effects (font (size 1.27 1.27)) (justify right))
+  )
+  (hierarchical_label "5PW1" (shape input) (at 375.92 210.82 180)
+    (effects (font (size 1.27 1.27)) (justify right))
+  )
   (hierarchical_label "XD[0..15]" (shape input) (at 562.61 372.11 0)
     (effects (font (size 1.27 1.27)) (justify left))
@@
     (pin "20")
   )
-  (symbol (lib_id "robotron_ec1834:DL295") (at 332.74 353.06 0) (unit 1)
+  (symbol (lib_name "DL295_1") (lib_id "robotron_ec1834:DL295") (at 332.74 353.06 0) (unit 1)
     (in_bom yes) (on_board yes)
     (property "Reference" "D6" (id 0) (at 332.74 361.95 0))
@@
       (effects (font (size 1.27 1.27)) hide)
     )
-    (property "Datasheet" "http://www.ti.com/lit/gpn/sn74LS295" (id 3) (at 332.74 353.06 0)
+    (property "Datasheet" "http://www.ti.com/lit/gpn/sn74LS295" (id 3) (at 332.74 365.76 0)
       (effects (font (size 1.27 1.27)) hide)
     )
@@
     (pin "7")
   )
-  (symbol (lib_id "robotron_ec1834:DL295") (at 332.74 292.1 0) (unit 1)
+  (symbol (lib_name "DL295_2") (lib_id "robotron_ec1834:DL295") (at 332.74 292.1 0) (unit 1)
     (in_bom yes) (on_board yes)
     (property "Reference" "D29" (id 0) (at 332.74 300.99 0))
@@
       (effects (font (size 1.27 1.27)) hide)
     )
-    (property "Datasheet" "http://www.ti.com/lit/gpn/sn74LS295" (id 3) (at 332.74 292.1 0)
+    (property "Datasheet" "http://www.ti.com/lit/gpn/sn74LS295" (id 3) (at 332.74 304.8 0)
       (effects (font (size 1.27 1.27)) hide)
     )
@@
     (pin "28")
   )
-  (symbol (lib_id "robotron_ec1834:KR580WN59A") (at 134.62 323.85 0) (unit 1)
+  (symbol (lib_name "KR580WN59A_1") (lib_id "robotron_ec1834:KR580WN59A") (at 134.62 323.85 0) (unit 1)
     (in_bom yes) (on_board yes)
     (property "Reference" "D49" (id 0) (at 134.62 295.275 0))
@@
       (effects (font (size 1.27 1.27) italic) hide)
     )
-    (property "Datasheet" "http://pdos.csail.mit.edu/6.828/2005/readings/hardware/8259A.pdf" (id 3) (at 134.62 323.85 0)
+    (property "Datasheet" "http://pdos.csail.mit.edu/6.828/2005/readings/hardware/8259A.pdf" (id 3) (at 133.35 335.28 0)
       (effects (font (size 1.27 1.27)) hide)
     )

Commit message: Completed BUS Final checks required
Parts:
- D10, D11, D12, D126, D13, D14, D15, D16, D28, D29, D3, D32, D33, D34, D37, D38, D39, D40, D47, D51, D59, D6, D62, D63, D67, D7, D71, D8, D87, D88: footprint (none) -> Package_DIP:DIP-14_W7.62mm
- D2, D21, D22, D23, D24, D25, D26, D27, D45, D64, D83, D84: footprint (none) -> Package_DIP:DIP-20_W7.62mm
- D35, D36, D46, D61, D89, D9: footprint (none) -> Package_DIP:DIP-16_W7.62mm
- E1, E2, E5, X6: footprint (none) -> Connector_PinHeader_2.54mm:PinHeader_1x02_P2.54mm_Vertical
- PS1, PS2: footprint (none) -> Connector_PinHeader_2.54mm:PinHeader_1x03_P2.54mm_Vertical
- V2: footprint (none) -> Diode_THT:D_DO-35_SOD27_P2.54mm_Vertical_AnodeUp
- W2, W3: footprint (none) -> Connector_PinHeader_2.54mm:PinHeader_1x01_P2.54mm_Vertical
- WD1, WD2, WD3: footprint (none) -> Resistor_THT:R_Axial_DIN0204_L3.6mm_D1.6mm_P7.62mm_Horizontal
Other:
- company: (none) -> Mario Gögel 2022
- title: (none) -> EC1834 Hauptplatine 201.

Commit message: Small corrections on Page 201.1
Parts:
- WD1, WD2, WD3: symbol Jumper:SolderJumper_2_Bridged -> Jumper:SolderJumper_2_Open
- X6: value Conn_02x01 -> RESET_BTN
Connections:
- net ~{NMIADRCS}: now also D71.8 (A3); no longer D71.9 (B3)
- net ~{XIOW}: now also D71.9 (B3); no longer D71.8 (A3)
- net ~{CS86L}: now reaches D23.9 (OE), D7.8 (Y3)
- net ~{F2}: now reaches D35.6, D40.9 (A3)
Other:
- moved on the sheet: D71C

Commit message: Updated footprint for EMR UC8821 Added footprint for PS5 PCB layout in progress small corrections in schematics
Parts:
- PS1: footprint Connector_PinHeader_2.54mm:PinHeader_1x03_P2.54mm_Vertical -> Connector_PinHeader_2.54mm:PinHeader_1x05_P2.54mm_Vertical
Changed lines of the file:
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@@
       (effects (font (size 1.27 1.27)) (justify right) hide)
     )
-    (property "Footprint" "Connector_PinHeader_2.54mm:PinHeader_1x03_P2.54mm_Vertical" (id 2) (at 416.56 255.27 0)
+    (property "Footprint" "Connector_PinHeader_2.54mm:PinHeader_1x05_P2.54mm_Vertical" (id 2) (at 416.56 255.27 0)
       (effects (font (size 1.27 1.27)) hide)
     )

Commit message: Updated footprints Updated PCB
Parts:
- C5: footprint Capacitor_THT:CP_Radial_D12.5mm_P5.00mm -> Capacitor_THT:CP_Axial_L18.0mm_D6.5mm_P25.00mm_Horizontal
- R1, R13, R19, R2, R20, R21, R3, R5, R50, R51, R6, R7, R8: footprint Resistor_THT:R_Axial_DIN0309_L9.0mm_D3.2mm_P12.70mm_Horizontal -> EC1834-Board:R_Axial_L9.0mm_D1.8mm_P12.70mm_Horizontal
Changed lines of the file:
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@@
       (effects (font (size 1.27 1.27)) (justify left))
     )
-    (property "Footprint" "Resistor_THT:R_Axial_DIN0309_L9.0mm_D3.2mm_P12.70mm_Horizontal" (id 2) (at 424.942 222.25 90)
+    (property "Footprint" "EC1834-Board:R_Axial_L9.0mm_D1.8mm_P12.70mm_Horizontal" (id 2) (at 424.942 222.25 90)
       (effects (font (size 1.27 1.27)) hide)
     )
@@
       (effects (font (size 1.27 1.27)) (justify left))
     )
-    (property "Footprint" "Resistor_THT:R_Axial_DIN0309_L9.0mm_D3.2mm_P12.70mm_Horizontal" (id 2) (at 424.942 229.87 90)
+    (property "Footprint" "EC1834-Board:R_Axial_L9.0mm_D1.8mm_P12.70mm_Horizontal" (id 2) (at 424.942 229.87 90)
       (effects (font (size 1.27 1.27)) hide)
     )
@@
     (property "Reference" "R7" (id 0) (at 426.72 215.9 90))
     (property "Value" "30" (id 1) (at 430.53 217.17 90))
-    (property "Footprint" "Resistor_THT:R_Axial_DIN0309_L9.0mm_D3.2mm_P12.70mm_Horizontal" (id 2) (at 426.72 214.122 90)
+    (property "Footprint" "EC1834-Board:R_Axial_L9.0mm_D1.8mm_P12.70mm_Horizontal" (id 2) (at 426.72 214.122 90)
       (effects (font (size 1.27 1.27)) hide)
     )
@@
     (property "Reference" "R3" (id 0) (at 426.72 208.28 90))
     (property "Value" "30" (id 1) (at 430.53 209.55 90))
-    (property "Footprint" "Resistor_THT:R_Axial_DIN0309_L9.0mm_D3.2mm_P12.70mm_Horizontal" (id 2) (at 426.72 206.502 90)
+    (property "Footprint" "EC1834-Board:R_Axial_L9.0mm_D1.8mm_P12.70mm_Horizontal" (id 2) (at 426.72 206.502 90)
       (effects (font (size 1.27 1.27)) hide)
     )
@@
       (effects (font (size 1.27 1.27)) (justify right))
     )
-    (property "Footprint" "Resistor_THT:R_Axial_DIN0309_L9.0mm_D3.2mm_P12.70mm_Horizontal" (id 2) (at 385.318 224.79 90)
+    (property "Footprint" "EC1834-Board:R_Axial_L9.0mm_D1.8mm_P12.70mm_Horizontal" (id 2) (at 385.318 224.79 90)
       (effects (font (size 1.27 1.27)) hide)
     )
@@
       (effects (font (size 1.27 1.27)) (justify right))
     )
-    (property "Footprint" "Resistor_THT:R_Axial_DIN0309_L9.0mm_D3.2mm_P12.70mm_Horizontal" (id 2) (at 367.538 224.79 90)
+    (property "Footprint" "EC1834-Board:R_Axial_L9.0mm_D1.8mm_P12.70mm_Horizontal" (id 2) (at 367.538 224.79 90)
       (effects (font (size 1.27 1.27)) hide)
     )
@@
       (effects (font (size 1.27 1.27)) (justify right))
     )
-    (property "Footprint" "Resistor_THT:R_Axial_DIN0309_L9.0mm_D3.2mm_P12.70mm_Horizontal" (id 2) (at 367.538 240.03 90)
+    (property "Footprint" "EC1834-Board:R_Axial_L9.0mm_D1.8mm_P12.70mm_Horizontal" (id 2) (at 367.538 240.03 90)
       (effects (font (size 1.27 1.27)) hide)
     )
@@
       (effects (font (size 1.27 1.27)) (justify left))
     )
-    (property "Footprint" "Resistor_THT:R_Axial_DIN0309_L9.0mm_D3.2mm_P12.70mm_Horizontal" (id 2) (at 464.312 246.38 90)
+    (property "Footprint" "EC1834-Board:R_Axial_L9.0mm_D1.8mm_P12.70mm_Horizontal" (id 2) (at 464.312 246.38 90)
       (effects (font (size 1.27 1.27)) hide)
     )
@@
     (property "Reference" "R2" (id 0) (at 468.63 252.5522 90))
     (property "Value" "4k7" (id 1) (at 468.63 254.8636 90))
-    (property "Footprint" "Resistor_THT:R_Axial_DIN0309_L9.0mm_D3.2mm_P12.70mm_Horizontal" (id 2) (at 468.63 256.032 90)
+    (property "Footprint" "EC1834-Board:R_Axial_L9.0mm_D1.8mm_P12.70mm_Horizontal" (id 2) (at 468.63 256.032 90)
       (effects (font (size 1.27 1.27)) hide)
     )
@@
     (property "Reference" "R51" (id 0) (at 368.3 201.93 90))
     (property "Value" "100" (id 1) (at 368.3 204.47 90))
-    (property "Footprint" "Resistor_THT:R_Axial_DIN0309_L9.0mm_D3.2mm_P12.70mm_Horizontal" (id 2) (at 368.3 206.248 90)
+    (property "Footprint" "EC1834-Board:R_Axial_L9.0mm_D1.8mm_P12.70mm_Horizontal" (id 2) (at 368.3 206.248 90)
       (effects (font (size 1.27 1.27)) hide)
     )
@@
     (property "Reference" "R50" (id 0) (at 368.3 196.85 90))
     (property "Value" "100" (id 1) (at 368.3 199.39 90))
-    (property "Footprint" "Resistor_THT:R_Axial_DIN0309_L9.0mm_D3.2mm_P12.70mm_Horizontal" (id 2) (at 368.3 201.168 90)
+    (property "Footprint" "EC1834-Board:R_Axial_L9.0mm_D1.8mm_P12.70mm_Horizontal" (id 2) (at 368.3 201.168 90)
       (effects (font (size 1.27 1.27)) hide)
     )
@@
     (property "Reference" "R8" (id 0) (at 400.05 271.6022 90))
     (property "Value" "30" (id 1) (at 400.05 273.9136 90))
-    (property "Footprint" "Resistor_THT:R_Axial_DIN0309_L9.0mm_D3.2mm_P12.70mm_Horizontal" (id 2) (at 400.05 275.082 90)
+    (property "Footprint" "EC1834-Board:R_Axial_L9.0mm_D1.8mm_P12.70mm_Horizontal" (id 2) (at 400.05 275.082 90)
       (effects (font (size 1.27 1.27)) hide)
     )
@@
       (effects (font (size 1.27 1.27)) (justify left))
     )
-    (property "Footprint" "Resistor_THT:R_Axial_DIN0309_L9.0mm_D3.2mm_P12.70mm_Horizontal" (id 2) (at 123.952 158.75 90)
+    (property "Footprint" "EC1834-Board:R_Axial_L9.0mm_D1.8mm_P12.70mm_Horizontal" (id 2) (at 123.952 158.75 90)
       (effects (font (size 1.27 1.27)) hide)
     )
@@
       (effects (font (size 1.27 1.27)) (justify right))
     )
-    (property "Footprint" "Capacitor_THT:CP_Radial_D12.5mm_P5.00mm" (id 2) (at 355.9048 236.22 0)
-      (effects (font (size 1.27 1.27)) hide)
-    )
+    (property "Footprint" "Capacitor_THT:CP_Axial_L18.0mm_D6.5mm_P25.00mm_Horizontal" (id 2) (at 355.9048 236.22 0)
+      (effects (font (size 1.27 1.27)) hide)
+    )
