File: EC1834_201.2.kicad_sch (KiCad schematic)
At the start: 77 parts

Commit message: Improved schematics and docs
Parts:
- added Br4: Br4, symbol Jumper:SolderJumper_2_Bridged
- added C10: 10pF, symbol Device:C
- added C5: 47µF, symbol Device:C
- added C6: 10nF, symbol Device:C
- added unit 1 of D11
- added unit 2 of D14
- added D34: DL008D, symbol robotron_ec1834:DL008D
- added D82: DL004D, symbol RFT_Digitalschaltkreise:DL004D
- added E1, E2, E5: SolderJumper_2_Bridged, symbol Jumper:SolderJumper_2_Bridged
- added PS1, PS2: Conn_01x03, symbol Connector_Generic:Conn_01x03
- added V1: 14745,6KHz, symbol Device:Crystal
- added V2: SAY30, symbol Device:D
- added W2, W3: Conn_01x01, symbol Connector_Generic:Conn_01x01
- added X6: Conn_02x01, symbol Connector_Generic:Conn_02x01
Connections:
- net D11 is gone; now on net D10: D21.16 (B3), D22.4 (A3)
- net D12 is gone; now on net D10: D21.15 (B4), D22.5 (A4)
- net D13 is gone; now on net D10: D21.14 (B5), D22.6 (A5)
- net D14 is gone; now on net D10: D21.13 (B6), D22.7 (A6)
- net D15 is gone; now on net D10: D21.12 (B7), D22.8 (A7)
- net D8 is gone; now on net D10: D21.19 (B0), D22.1 (A0)
- net D9 is gone; now on net D10: D21.18 (B1), D22.2 (A1)
- net CEN: now also D4.15 (CEN)
- net D10: now also D21.11 (T), D23.11 (T)
- net ~{CLK}: now also D15.11 (C)
- net ~{RESETDRV}: now reaches D12.10 (B3), R12.3 (R2.2)
- net ~{RESETDRV}: now also D12.2 (B1), D34.10 (Y5), D35.1 (R), D35.1 (R), D59.1 (A1)
- net +5V: now reaches D38.1 (R)
- net +5V: now also D13.4 (S), D15.1 (R), D15.10 (S), D15.13 (R), D15.4 (S)
- net GND: now reaches D38.2 (D)
- net GND: now also R5.1, R6.2
- net BS-/WAIT: now reaches D38.5
- net at D24.11 (C), D36.12 (D3), D36.7: now also D15.12 (D), D32.9 (A3)
- net ~{AEN}: now reaches D12.5 (B2)
- net ~{AEN}: now also D16.5 (B2), D67.12 (D)
- net ~{F4}: now reaches D39.10 (B3)
- net ~{F4}: now also D35.14
- net at D43.16 (X2): now also R5.2, V1.1
- net at D43.17 (X1): now also R6.1, C10.1
- net at D23.9 (OE): now also D7.8 (Y3)
- net AENI: now reaches D84.6 (A5)
- net AENI: now also D12.11 (Y4), D32.12 (A4)
- net RESETDRV: now reaches D59.2 (Y1)
- net at D8.1 (A1): now also R11.4 (R3.2)
- net at D35.2: now also D39.1 (A1)
- net at D35.4 (D1): now also D37.3 (Y1)
- net CLK: now reaches D35.9 (C)
- net CLK: now also D35.9 (C), D35.9 (C), D38.11 (C)
- net at D35.13 (D4): now also D35.10
- net at D35.11: now also D47.2 (B1), D67.13 (R)
- net at D35.12 (D3): now also D67.9
- net IOCHRDY: now reaches D67.10 (S)
- net IOCHRDY: now also R13.1
- net IORW: now reaches D67.11 (C)
- net IORW: now also D10.3 (Y1)
- net at D67.8: now also D47.1 (A1)
- net at D51.2 (D): now also D37.2 (B1), D38.9
- net PCLK: now reaches D51.3 (C)
- net at D51.4 (S): now also D51.5, D51.6
- net IED: now reaches D38.10 (S)
- net IED: now also D38.8
- net at D38.12 (D): now also D34.2 (Y1)
- net HRQDMA: now reaches D38.13 (R)
- net at D34.1 (A1): now also D3.8 (Y2)
- net ~{XIOR}: now reaches D10.1 (A1)
- net ~{XIOW}: now reaches D10.2 (B1)
- net at D39.2 (B1): now also D37.1 (A1)
- net ~{BHE}: now reaches D33.2 (A1)
- net VA0: now reaches D33.3 (B1)
- net ~{MEMADRSEL}: now reaches D88.10 (B3)
- net ~{MEMW}: now reaches D32.4 (A2)
- net ~{MEMCS16}: now reaches D32.5 (B2)
- net ~{MASTER}: now reaches D12.12 (A4)
- net ~{MASTER}: now also D47.13 (B4)
- net AENBRD: now reaches D12.13 (B4)
- net DT-/R: now reaches D16.4 (A2)
- net ~{XMEMW}: now reaches D32.13 (B4)
- net BHE: now reaches D47.12 (A4)
- net ~{MEMR}: now reaches D7.2 (B1)
- net ~{S1}: now reaches D3.10 (B2)
- net ~{S2}: now reaches D3.12 (C2)
- net ~{LOCK}: now reaches D3.13 (D2)
- net ~{S0}: now reaches D3.9 (A2)
- net at D7.6 (Y2): now also D21.9 (OE)
- net at D7.10 (B3): now also D7.11 (Y4)
- net A0: now reaches D40.13 (B4)
- new net: C10.2, V1.2
- no-connect marks 3 -> 4
Other:
- note added: "Bei der Verwend. d. K1810GF84 entfällt E1"
- moved on the sheet: D1, D10A, D11B, D126A, D12A, D12B, D12C, D12D, D13A, D14A, D14C, D15A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

Commit message: Improved schematics
Parts:
- removed D34: DL008D, symbol robotron_ec1834:DL008D
- added unit 4 of D34
- Br4: footprint (none) -> Resistor_THT:R_Axial_DIN0204_L3.6mm_D1.6mm_P5.08mm_Horizontal
- C10, C6: footprint (none) -> Capacitor_THT:C_Disc_D4.3mm_W1.9mm_P5.00mm
- C5: footprint (none) -> Capacitor_THT:CP_Radial_D12.5mm_P5.00mm
- E1, E2, E5: symbol Jumper:SolderJumper_2_Bridged -> Connector_Generic:Conn_02x01
- R1, R13, R19, R2, R20, R21, R3, R5, R50, R51, R6, R7, R8: footprint (none) -> Resistor_THT:R_Axial_DIN0309_L9.0mm_D3.2mm_P12.70mm_Horizontal
- V1: footprint (none) -> Crystal:Crystal_HC18-U_Horizontal
Connections:
- net HRQDMA: now also D50.10 (HRQ)
- net PCLK: now also D50.12 (CLK)
- net ~{XMEMW}: now also D50.4 (MEMW)
- net 1: now reaches D64.5 (A4)
- net 1: now also D50.37 (A4)
- net 2: now reaches D64.6 (A5)
- net 2: now also D50.38 (A5)
- net 3: now reaches D64.7 (A6)
- net 3: now also D50.39 (A6)
- net 4: now reaches D64.8 (A7)
- net 4: now also D50.40 (A7)
- net at D64.9 (OE): now also D45.9 (OE)
- net at D45.11 (STN): now also D50.8 (ADSTB)
- net at D47.10 (B3): now also D50.36 (TC)
- net TC: now reaches D47.8 (Y3)
- net at D48.17 (INT): now also Br4.2 (B), D49.20 (IR2)
- net at D48.19 (IR1): now also Br4.1 (A)
- net at D48.26 (INTA): now also D49.26 (INTA), R52.2 (R1.2)
- net ~{YIOR}: now reaches D50.1 (IOR)
- net ~{DMACS}: now reaches D50.11 (CS)
- net RESET: now reaches D50.13 (RESET)
- net DRQ3: now reaches D50.16 (DRQ3)
- net DRQ2: now reaches D50.17 (DRQ2)
- net DRQ1: now reaches D50.18 (DRQ1)
- net DRQ0: now reaches D50.19 (DRQ0)
- net ~{YIOW}: now reaches D50.2 (IOW)
- net ~{XMEMR}: now reaches D50.3 (MEMR)
- net TDYTODMA: now reaches D50.6 (RDY)
- net HOLDA: now reaches D50.7 (HLDA)
- net AENDMA: now reaches D50.9 (AEN)
- no-connect marks 4 -> 5
Other:
- note added: "D64A PIN Pos abweichend von Zeichnung 1.13.120030.0/04"
- moved on the sheet: D45A, D64A, D71C, R52A

Commit message: Almsot completed page 1
Connections:
- net DT-/R is gone; now on net D10: D16.4 (A2)
- net +5V: now also D1.40 (VCC), D126.1 (R), D20.40 (VCC), D28.06 (V), D29.06 (V), D42.1, D43.18 (VCC), D47.9 (A3), D51.10 (S), D6.06 (V), R1.1, R10.1 (R1.1), R19.2, R2.2, R52.1 (R1.1)
- net A0: now also D64.19 (B0)
- net AENBRD: now also D27.11 (T), D35.2, D35.5 (D2), D39.1 (A1), D83.9 (OE)
- net AENDMA: now also D39.3 (Y1)
- net BS-/WAIT: now also D14.2 (B1)
- net CLK: now also D35.9 (C), D84.13 (B6)
- net D10: now also D4.4 (DT/~{R})
- net DEN: now also D4.16 (DEN), D8.3 (A2)
- net GND: now also C5.1, C6.1, D1.1 (GND), D1.20 (GND), D20.1 (GND), D20.20 (GND), D20.33 (MAX), D28.01 (A0), D29.01 (A0), D4.1 (IOB), D43.6 (RDY2), D48.16 (SP), D6.01 (A0), D61.04 (DI0), D61.07 (DI1), D61.09 (DI2), D61.15 (DIEN), D84.9 (OE), D9.04 (E1), D9.05 (E2), R21.1, R50.1, R51.1, X6.1 (Pin_1)
- net HOLDA: now also D51.4 (S), D51.5, D51.6
- net IED: now also D40.10 (B3)
- net IOCHRDY: now also D14.1 (A1)
- net PCLK: now also R7.1
- net RESET: now also D43.10 (RESET)
- net TC: now also D51.11 (C)
- net VA0: now also D88.12 (A4)
- net ~{BHE}: now also D1.34 (BHE), D20.34 (BHE), D61.13 (DB3), D7.5 (B2)
- net ~{CLK}: now also D87.12 (Y6)
- net ~{MASTER}: now also D8.1 (A1), R11.4 (R3.2)
- net ~{MEMR}: now also R9.1 (R1.1)
- net ~{MEMW}: now also R9.3 (R2.1)
- net ~{RESETDRV}: now also D35.1 (R)
- net ~{S0}: now also D20.26 (S0), D4.19 (S0), PS1.1 (Pin_1)
- net ~{S1}: now also D20.27 (S1), D4.3 (S1), PS1.2 (Pin_2)
- net ~{S2}: now also D20.28 (S2), D4.18 (S2), PS1.3 (Pin_3)
- net ~{XIOR}: now also D27.15 (B4), D27.6 (A5), D48.3 (RD), D49.3 (RD), R10.6 (R5.2)
- net ~{XIOW}: now also D27.13 (B6), D27.8 (A7), D48.2 (WR), D49.2 (WR), D71.8 (A3), R10.8 (R7.2)
- net ~{XMEMR}: now also D27.2 (A1), R10.2 (R1.2)
- net ~{XMEMW}: now also D27.4 (A3), R10.4 (R3.2)
- net ~{YIOR}: now also D27.5 (A4), R12.6 (R5.2), R12.9 (R8.2)
- net ~{YIOW}: now also D27.7 (A6)
- net DACK0: now reaches D51.12 (D)
- net DACK0: now also D8.12 (Y6)
- net PB3: now reaches D51.13 (R)
- net IRQ8: now reaches D51.9
- net IRQ8: now also D48.18 (IR0)
- net at D89.07 (O7): now also W3.1 (Pin_1)
- net AD6: now reaches D1.10 (AD6)
- net AD6: now also D20.10 (AD6)
- net AD5: now reaches D1.11 (AD5)
- net AD5: now also D20.11 (AD5)
- net AD4: now reaches D1.12 (AD4)
- net AD4: now also D20.12 (AD4)
- net AD3: now reaches D1.13 (AD3)
- net AD3: now also D20.13 (AD3)
- net AD2: now reaches D1.14 (AD2)
- net AD2: now also D20.14 (AD2)
- net AD1: now reaches D1.15 (AD1)
- net AD1: now also D20.15 (AD1)
- net AD0: now reaches D1.16 (AD0)
- net AD0: now also D20.16 (AD0)
- net AD14: now reaches D1.2 (AD14)
- net AD14: now also D20.2 (AD14)
- net at D1.23 (BUSY): now also D20.23 (TEST), R2.1
- net AD13: now reaches D1.3 (AD13)
- net AD13: now also D20.3 (AD13)
- net 5PW1: now reaches D1.33 (~{GT1})
- net 5PW1: now also D20.31 (~{GT0}), D43.7 (AEN2), E1.1 (Pin_1)
- net AD19: now reaches D1.35 (A19)
- net AD19: now also D20.35 (A19)
- net AD18: now reaches D1.36 (A18)
- net AD18: now also D20.36 (A18)
- net AD17: now reaches D1.37 (A17)
- net AD17: now also D20.37 (A17)
- net AD16: now reaches D1.38 (A16)
- net AD16: now also D20.38 (A16)
- net AD15: now reaches D1.39 (AD15)
- net AD15: now also D20.39 (AD15)
- net AD12: now reaches D1.4 (AD12)
- net AD12: now also D20.4 (AD12)
- net AD11: now reaches D1.5 (AD11)
- net AD11: now also D20.5 (AD11)
- net AD10: now reaches D1.6 (AD10)
- net AD10: now also D20.6 (AD10)
- net AD9: now reaches D1.7 (AD9)
- net AD9: now also D20.7 (AD9)
- net AD8: now reaches D1.8 (AD8)
- net AD8: now also D20.8 (AD8)
- net AD7: now reaches D1.9 (AD7)
- net AD7: now also D20.9 (AD7)
- net at D20.30 (~{GT1}): now also R1.2
- net ~{CIOW}: now reaches D4.12 (AIOWC)
- net ~{CIOW}: now also D27.12 (B7), R10.9 (R8.2), R9.8 (R4.2)
- net ~{CIOR}: now reaches D4.13 (IORC)
- net ~{CIOR}: now also D27.14 (B5), R10.7 (R6.2), R9.6 (R3.2)
- net ~{INTA}: now reaches D4.14 (~{INTA})
- net ~{INTA}: now also D48.26 (INTA), D49.26 (INTA), D88.13 (B4), R52.2 (R1.2)
- net CLK86: now reaches D4.2 (CLK)
- net CLK86: now also D126.3 (C), D84.7 (A6), D87.13 (A6), R3.1
- net at D4.5 (ALE): now also R8.2
- net AENBRDW: now reaches D4.6 (AEN)
- net ~{CMEMR}: now reaches D4.7 (MRDC)
- net ~{CMEMR}: now also D27.18 (B1), R10.3 (R2.2), R9.2 (R1.2)
- net ~{CMEMW}: now reaches D4.8 (AMWC)
- net ~{CMEMW}: now also D27.16 (B3), R10.5 (R4.2), R9.4 (R2.2)
- net at D43.1 (CSYN): now also PS2.1 (Pin_1), R51.2
- net at D43.11 (RES): now also C6.2, D42.4, R19.1, X6.2 (Pin_2)
- net at D43.12 (OSC): now also E5.1 (Pin_1)
- net at D43.13 (F/C): now also E2.2 (Pin_2)
- net at D43.14 (EFI): now also PS2.3 (Pin_3), W2.1 (Pin_1)
- net at D43.15 (ASYN): now also E1.2 (Pin_2)
- net at D43.2 (PC): now also R7.2
- net at D43.3 (AEN1): now also D126.2 (D), D14.12 (Y1)
- net at D43.4 (RDY1): now also D126.6
- net READY: now reaches D43.5 (READY)
- net at D43.8 (CLK): now also R3.2
- net at D42.2: now also C5.2, R20.1, R21.2, V2.2 (A)
- net XD0: now reaches D6.02 (A1)
- net XD0: now also D28.02 (A1), D29.02 (A1), D45.1 (DI0), D48.11 (D0), D49.11 (D0), D50.30 (DB0)
- net XD1: now reaches D6.03 (A2)
- net XD1: now also D28.03 (A2), D29.03 (A2), D45.2 (DI1), D48.10 (D1), D49.10 (D1), D50.29 (DB1)
- net XD2: now reaches D6.04 (A3)
- net XD2: now also D28.04 (A3), D29.04 (A3), D45.3 (DI2), D48.9 (D2), D49.9 (D2), D50.28 (DB2)
- net XD3: now reaches D6.05 (A4)
- net XD3: now also D28.05 (A4), D29.05 (A4), D45.4 (DI3), D48.8 (D3), D49.8 (D3), D50.27 (DB3)
- net at D6.08 (CS): now also D33.4 (Y2)
- net at D6.09 (C): now also D8.6 (Y3)
- net A19: now reaches D6.10 (F3)
- net A19: now also D28.10 (F3), D29.10 (F3)
- net A18: now reaches D6.11 (F2)
- net A18: now also D28.11 (F2), D29.11 (F2)
- net A17: now reaches D6.12 (F1)
- net A17: now also D28.12 (F1), D29.12 (F1)
- net A16: now reaches D6.13 (F0)
- net A16: now also D28.13 (F0), D29.13 (F0)
- net at D28.08 (CS): now also D33.10 (Y3)
- net at D28.09 (C): now also D8.8 (Y4)
- net at D29.08 (CS): now also D33.13 (Y4)
- net at D29.09 (C): now also D8.10 (Y5)
- net A8: now reaches D84.1 (A0)
- net A8: now also D45.19 (DO0)
- net 5PW2: now reaches D84.11 (T)
- net 5PW2: now also D64.11 (T), D83.11 (T), D9.06 (E3)
- net ~{DACK0}: now reaches D84.12 (B7)
- net ~{DACK0}: now also D40.2 (B1)
- net AEN: now reaches D84.14 (B5)
- net XA12: now reaches D84.15 (B4)
- net XA11: now reaches D84.16 (B3)
- net XA10: now reaches D84.17 (B2)
- net XA9: now reaches D84.18 (B1)
- net XA8: now reaches D84.19 (B0)
- net A9: now reaches D84.2 (A1)
- net A9: now also D45.18 (DO1)
- net A10: now reaches D84.3 (A2)
- net A10: now also D45.17 (DO2)
- net A11: now reaches D84.4 (A3)
- net A11: now also D45.16 (DO3)
- net A12: now reaches D84.5 (A4)
- net A12: now also D45.15 (DO4)
- net ~{DACK0BRD}: now reaches D84.8 (A7)
- net ~{DACK0BRD}: now also D50.25 (DACK0), D8.13 (A6)
- net ~{DMAWAIT}: now reaches D126.4 (S)
- net ~{DMAWAIT}: now also D40.8 (Y3)
- net RDY-/WAIT: now reaches D14.13 (C1)
- net RDY-/WAIT: now also D47.3 (Y1)
- net A13: now reaches D83.1 (A0)
- net A13: now also D45.14 (DO5)
- net XA7: now reaches D83.12 (B7)
- net XA6: now reaches D83.13 (B6)
- net XA5: now reaches D83.14 (B5)
- net XA4: now reaches D83.15 (B4)
- net XA3: now reaches D83.16 (B3)
- net XA3: now also D64.4 (A3)
- net XA2: now reaches D83.17 (B2)
- net XA2: now also D64.3 (A2)
- net XA1: now reaches D83.18 (B1)
- net XA1: now also D64.2 (A1), D9.02 (A1)
- net XA13: now reaches D83.19 (B0)
- net A1: now reaches D83.2 (A1)
- net A1: now also D64.18 (B1)
- net A2: now reaches D83.3 (A2)
- net A2: now also D64.17 (B2)
- net A3: now reaches D83.4 (A3)
- net A3: now also D64.16 (B3)
- net A4: now reaches D83.5 (A4)
- net A4: now also D64.15 (B4)
- net A5: now reaches D83.6 (A5)
- net A5: now also D64.14 (B5)
- net A6: now reaches D83.7 (A6)
- net A6: now also D64.13 (B6)
- net A7: now reaches D83.8 (A7)
- net A7: now also D64.12 (B7)
- net at D33.5 (A2): now also D40.3 (Y1)
- net MASTER: now reaches D33.6 (B2)
- net MASTER: now also D27.9 (OE), D33.12 (B4), D33.9 (B3), D8.2 (Y1)
- net at D8.5 (A3): now also D9.07 (O7)
- net at D8.9 (A4): now also D9.10 (O5)
- net at D8.11 (A5): now also D9.09 (O6)
- net ~{DACK3}: now reaches D33.11 (A4)
- net ~{DACK3}: now also D50.15 (DACK3)
- net ~{DACK2}: now reaches D33.8 (A3)
- net ~{DACK2}: now also D50.14 (DACK2)
- net ~{DACK1}: now reaches D40.1 (A1)
- net ~{DACK1}: now also D50.24 (DACK1)
- net at D40.9 (A3): now also D35.6
- net XA0: now reaches D9.01 (A0)
- net XA0: now also D48.27 (A0), D49.27 (A0), D64.1 (A0)
- net WRTDMAPGREG: now reaches D9.03 (A2)
- net WRTDMAPGREG: now also D71.10 (Y3)
- net at D61.01 (CS): now also D45.9 (OE), D62.3 (Y1), D64.9 (OE)
- net ~{A0}: now reaches D61.12 (DI3)
- net A15: now reaches D45.12 (DO7)
- net A14: now reaches D45.13 (DO6)
- net XD4: now reaches D45.5 (DI4)
- net XD4: now also D48.7 (D4), D49.7 (D4), D50.26 (DB4)
- net XD5: now reaches D45.6 (DI5)
- net XD5: now also D48.6 (D5), D49.6 (D5), D50.23 (DB5)
- net XD6: now reaches D45.7 (DI6)
- net XD6: now also D48.5 (D6), D49.5 (D6), D50.22 (DB6)
- net XD7: now reaches D45.8 (DI7)
- net XD7: now also D48.4 (D7), D49.4 (D7), D50.21 (DB7)
- net RDYTODMA: now reaches D37.1 (A1), D39.2 (B1)
- net ~{NMIADRCS}: now reaches D71.9 (B3)
- net ~{DMAAEN}: now reaches D62.1 (A1)
- net ~{INTRCS2}: now reaches D48.1 (CS)
- net CAS0: now reaches D48.12 (CAS0)
- net CAS0: now also D49.12 (CAS0)
- net CAS1: now reaches D48.13 (CAS1)
- net CAS1: now also D49.13 (CAS1)
- net CAS2: now reaches D48.15 (CAS2)
- net CAS2: now also D49.15 (CAS2)
- net IRQ2: now reaches Br4.2 (B), D48.17 (INT), D49.20 (IR2)
- net IRQ2: now also Br4.1 (A), D48.19 (IR1)
- net IRQ10: now reaches D48.20 (IR2)
- net IRQ11: now reaches D48.21 (IR3)
- net IRQ12: now reaches D48.22 (IR4)
- net NPNPI: now reaches D48.23 (IR5)
- net IRQ14: now reaches D48.24 (IR6)
- net IRQ15: now reaches D48.25 (IR7)
- net ~{INTRCS1}: now reaches D49.1 (CS)
- net at D49.16 (SP): now also R12.10 (R9.2)
- net INT: now reaches D49.17 (INT)
- net IRQ0: now reaches D49.18 (IR0)
- net IRQ1: now reaches D49.19 (IR1)
- net IRQ3: now reaches D49.21 (IR3)
- net IRQ4: now reaches D49.22 (IR4)
- net IRQ5: now reaches D49.23 (IR5)
- net IRQ6: now reaches D49.24 (IR6)
- net IRQ7: now reaches D49.25 (IR7)
- net at D7.4 (A2): now also D7.9 (A3), D8.4 (Y2)
- net ~{CS86H}: now reaches D21.9 (OE), D7.6 (Y2)
- net at D7.12 (A4): now also D88.11 (Y4)
- net at D7.13 (B4): now also D15.9
- net ~{IOR}: now reaches R9.5 (R3.1)
- net ~{IOW}: now reaches R9.7 (R4.1)
- net +12V: now reaches R20.2
- net +12V: now also V2.1 (K)
- net at R50.2: now also E2.1 (Pin_1), PS2.2 (Pin_2)
- net ALE: now reaches R8.1
- net OSCI: now reaches E5.2 (Pin_2)
- no-connect marks 5 -> 29
Other:
- moved on the sheet: C10, C5, C6, D27A, D28A, D29A, D35B, D40A, D42, D4A, D62A, E1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

Commit message: Completed signal connections Work on bus signal names
Connections:
- net A0: now also D2.18 (DO1), D46.03 (DB0)
- net A1: now also D26.19 (DO0)
- net A10: now also D25.17 (DO2)
- net A11: now also D25.16 (DO3)
- net A12: now also D25.15 (DO4)
- net A13: now also D25.14 (DO5)
- net A14: now also D25.13 (DO6)
- net A15: now also D25.12 (DO7)
- net A16: now also D2.15 (DO4)
- net A17: now also D2.14 (DO5)
- net A18: now also D2.13 (DO6)
- net A19: now also D2.16 (DO3)
- net A2: now also D26.18 (DO1)
- net A3: now also D26.17 (DO2)
- net A4: now also D26.16 (DO3)
- net A5: now also D26.15 (DO4)
- net A6: now also D26.14 (DO5)
- net A7: now also D26.13 (DO6)
- net A8: now also D25.19 (DO0)
- net A9: now also D25.18 (DO1)
- net AD0: now also D2.2 (DI1), D23.8 (A7), D24.12 (Q4), D26.8 (DI7)
- net AD1: now also D23.7 (A6), D24.9 (Q3), D26.1 (DI0)
- net AD10: now also D21.3 (A2), D25.3 (DI2)
- net AD11: now also D21.4 (A3), D25.4 (DI3)
- net AD12: now also D21.5 (A4), D25.5 (DI4)
- net AD13: now also D21.6 (A5), D25.6 (DI5)
- net AD14: now also D21.7 (A6), D25.7 (DI6)
- net AD15: now also D21.8 (A7), D25.8 (DI7)
- net AD16: now also D2.5 (DI4)
- net AD17: now also D2.6 (DI5)
- net AD18: now also D2.7 (DI6)
- net AD19: now also D2.4 (DI3)
- net AD2: now also D23.6 (A5), D24.6 (Q2), D26.2 (DI1)
- net AD3: now also D23.5 (A4), D24.15 (Q5), D26.3 (DI2)
- net AD4: now also D23.4 (A3), D24.16 (Q6), D26.4 (DI3)
- net AD5: now also D23.3 (A2), D24.5 (Q1), D26.5 (DI4)
- net AD6: now also D23.2 (A1), D24.2 (Q0), D26.6 (DI5)
- net AD7: now also D23.1 (A0), D24.19 (Q7), D26.7 (DI6)
- net AD8: now also D21.1 (A0), D25.1 (DI0)
- net AD9: now also D21.2 (A1), D25.2 (DI1)
- net AENBRD: now also D46.01 (CS), WD1.2 (B)
- net AENBRDW: now also D2.9 (OE), D25.9 (OE), D26.9 (OE), R10.10 (R9.2), WD1.1 (A)
- net ALE: now also D2.11 (STN), D25.11 (STN), D26.11 (STN)
- net CLK86: now also D1.19 (CLK), D20.19 (CLK)
- net GND: now also D46.07 (DI1), D46.09 (DI2), D46.12 (DI3), D46.15 (DIEN)
- net INT: now also D20.18 (INTR)
- net NPNPI: now also D1.32 (INT)
- net READY: now also D1.22 (READY), D20.22 (READY)
- net RESET: now also D1.21 (RESET), D20.21 (RESET)
- net VA0: now also D26.12 (DO7)
- net XA0: now also D50.32 (A0)
- net XA1: now also D50.33 (A1)
- net XA2: now also D50.34 (A2)
- net XA3: now also D50.35 (A3)
- net XA5: now also D89.01 (A0)
- net XA6: now also D89.02 (A1)
- net XA7: now also D89.03 (A2)
- net XA8: now also D89.04 (E1)
- net XA9: now also D89.05 (E2)
- net ~{AEN}: now also D89.06 (E3)
- net ~{BHE}: now also D2.12 (DO7), D2.8 (DI7)
- net ~{DMACS}: now also D89.15 (O0)
- net ~{INTRCS1}: now also D89.14 (O1)
- net ~{INTRCS2}: now also D89.09 (O6)
- net ~{LOCK}: now also D20.29 (~{LOCK})
- net ~{NMIADRCS}: now also D89.11 (O4)
- net ~{S0}: now also D1.26 (S0)
- net ~{S1}: now also D1.27 (S1)
- net ~{S2}: now also D1.28 (S2)
- net ~{NMIREGCS}: now reaches D89.10 (O5)
- net ~{PPICS}: now reaches D89.12 (O3)
- net ~{TIMERCS}: now reaches D89.13 (O2)
- net QS1: now reaches D1.24 (QS1)
- net QS1: now also D20.24 (QS1)
- net QS0: now reaches D1.25 (QS0)
- net QS0: now also D20.25 (QS0)
- net ~{GT1}: now reaches D1.31 (~{GT0})
- net ~{GT1}: now also D20.30 (~{GT1}), R1.2
- net NMI: now reaches D20.17 (NMI)
- net at D46.04 (DI0): now also D7.10 (B3), D7.11 (Y4)
- no-connect marks 29 -> 40
Other:
- moved on the sheet: WD1

Commit message: Completed main bus signal label on CPU page
Connections:
- net AENDMA: now also D37.1 (A1), D39.2 (B1); no longer D39.3 (Y1)
- net D10: no longer D16.4 (A2), D21.11 (T), D21.12 (B7), D21.13 (B6), D21.14 (B5), D21.15 (B4), D21.16 (B3), D21.18 (B1), D21.19 (B0), D22.1 (A0), D22.2 (A1), D22.4 (A3), D22.5 (A4), D22.6 (A5), D22.7 (A6), D22.8 (A7), D23.11 (T), D4.4 (DT/~{R})
- net D5: no longer D24.4 (D1)
- net MASTER: now also D62.2 (B1)
- net RDY-/WAIT: now also D47.1 (A1), D67.8; no longer D47.3 (Y1)
- net RDYTODMA: now also D47.3 (Y1); no longer D37.1 (A1), D39.2 (B1)
- net RESET: now also D34.11 (A5)
- net ~{AEN}: now also D35.3
- net ~{DMAAEN}: now also D39.3 (Y1)
- net ~{RESETDRV}: now also D35.1 (R)
- new net D11: D21.16 (B3), D22.4 (A3)
- new net D12: D21.15 (B4), D22.5 (A4)
- new net D13: D21.14 (B5), D22.6 (A5)
- new net D14: D21.13 (B6), D22.7 (A6)
- new net D15: D21.12 (B7), D22.8 (A7)
- new net D8: D21.19 (B0), D22.1 (A0)
- new net D9: D21.18 (B1), D22.2 (A1)
- new net DT-/R: D16.4 (A2), D21.11 (T), D23.11 (T), D4.4 (DT/~{R})

Commit message: Corrected schema names added bus signals
Parts:
- removed Br4: Br4, Resistor_THT:R_Axial_DIN0204_L3.6mm_D1.6mm_P5.08mm_Horizontal, symbol Jumper:SolderJumper_2_Bridged
- removed C10: 10pF, Capacitor_THT:C_Disc_D4.3mm_W1.9mm_P5.00mm, symbol Device:C
- removed C5: 47µF, Capacitor_THT:CP_Radial_D12.5mm_P5.00mm, symbol Device:C
- removed C6: 10nF, Capacitor_THT:C_Disc_D4.3mm_W1.9mm_P5.00mm, symbol Device:C
- removed D1: K1810WM87, Package_DIP:DIP-40_W15.24mm, symbol robotron_ec1834:K1810WM87
- removed D10, D16, D32, D39: DL000D, symbol RFT_Digitalschaltkreise:DL000D
- removed D11, D3: DL020D, symbol RFT_Digitalschaltkreise:DL020D
- removed D12, D40, D47, D88: DL008D, symbol RFT_Digitalschaltkreise:DL008D
- removed D126, D13, D15, D38, D51, D67: DL074, symbol robotron_ec1834:DL074
- removed D14: DL010D, symbol RFT_Digitalschaltkreise:DL010D
- removed D2, D25, D26, D45: DS8282, symbol robotron_ec1834:DS8282
- removed D20: K1810WM86, Package_DIP:DIP-40_W15.24mm, symbol robotron_ec1834:K1810WM86
- removed D21: DS8286D-D111, symbol robotron_ec1834:DS8286D-D111
- removed D22, D83, D84: DS8286D, symbol robotron_ec1834:DS8286D
- removed D23, D64: DS8286D-D23, symbol robotron_ec1834:DS8286D-D23
- removed D24: DL374, symbol robotron_ec1834:DL374
- removed D27: DS8286D-D27, symbol robotron_ec1834:DS8286D-D27
- removed D28, D29, D6: DL295, symbol robotron_ec1834:DL295
- removed D33, D71: DL002D, symbol RFT_Digitalschaltkreise:DL002D
- removed D34, D59, D8, D82, D87: DL004D, symbol RFT_Digitalschaltkreise:DL004D
- removed D35, D36: DL175, symbol robotron_ec1834:DL175
- removed D37, D62, D7: DL032D, symbol RFT_Digitalschaltkreise:DL032D
- removed D4: KR1810WG88, Package_DIP:DIP-20_W7.62mm, symbol robotron_ec1834:KR1810WG88
- removed D42: A302D, Package_DIP:DIP-4_W7.62mm, symbol robotron_ec1834:A302D
- removed D43: 8284, Package_DIP:DIP-18_W7.62mm, symbol robotron_ec1834:8284
- removed D46, D61: DS8216, symbol robotron_ec1834:DS8216
- removed D48, D49: KR580WN59A, Package_DIP:DIP-28_W15.24mm, symbol robotron_ec1834:KR580WN59A
- removed D50: KR580IK57, Package_DIP:DIP-40_W15.24mm, symbol robotron_ec1834:KR580IK57
- removed D63: DL010D-D63, symbol robotron_ec1834:DL010D-D63
- removed D89, D9: DS8205, symbol robotron_ec1834:DS8205
- removed E1, E2, E5: SolderJumper_2_Bridged, symbol Connector_Generic:Conn_02x01
- removed PS1, PS2: Conn_01x03, symbol Connector_Generic:Conn_01x03
- removed R1, R2: 4k7, Resistor_THT:R_Axial_DIN0309_L9.0mm_D3.2mm_P12.70mm_Horizontal, symbol Device:R
- removed R10, R12: 4k7, Resistor_THT:R_Array_SIP10, symbol Device:R_Network09_Split
- removed R11: 1k, Resistor_THT:R_Array_SIP6, symbol Device:R_Network05_Split
- removed R13: 4,7k, Resistor_THT:R_Axial_DIN0309_L9.0mm_D3.2mm_P12.70mm_Horizontal, symbol Device:R
- removed R19: 18k, Resistor_THT:R_Axial_DIN0309_L9.0mm_D3.2mm_P12.70mm_Horizontal, symbol Device:R
- removed R20: 180k, Resistor_THT:R_Axial_DIN0309_L9.0mm_D3.2mm_P12.70mm_Horizontal, symbol Device:R
- removed R21: 100k, Resistor_THT:R_Axial_DIN0309_L9.0mm_D3.2mm_P12.70mm_Horizontal, symbol Device:R
- removed R3, R7, R8: 30, Resistor_THT:R_Axial_DIN0309_L9.0mm_D3.2mm_P12.70mm_Horizontal, symbol Device:R
- removed R5, R6: 511, Resistor_THT:R_Axial_DIN0309_L9.0mm_D3.2mm_P12.70mm_Horizontal, symbol Device:R
- removed R50, R51: 100, Resistor_THT:R_Axial_DIN0309_L9.0mm_D3.2mm_P12.70mm_Horizontal, symbol Device:R
- removed R52: 3k9, Resistor_THT:R_Array_SIP8, symbol Device:R_Network07_Split
- removed R9: 30, Resistor_THT:R_Array_SIP8, symbol Device:R_Pack04_SIP_Split
- removed V1: 14745,6KHz, Crystal:Crystal_HC18-U_Horizontal, symbol Device:Crystal
- removed V2: SAY30, symbol Device:D
- removed W2, W3: Conn_01x01, symbol Connector_Generic:Conn_01x01
- removed WD1: WD1, symbol Jumper:SolderJumper_2_Bridged
- removed WD2: WD2, symbol Jumper:SolderJumper_2_Bridged
- removed WD3: WD3, symbol Jumper:SolderJumper_2_Bridged
- removed X6: Conn_02x01, symbol Connector_Generic:Conn_02x01
- added C7, C8: 680pF, Capacitor_THT:C_Disc_D4.3mm_W1.9mm_P5.00mm, symbol Device:C
- added D10, D16, D39: DL000D, symbol RFT_Digitalschaltkreise:DL000D
- added D100, D101, D115, D116: U2764, symbol robotron_ec1834:U2764
- added D111, D112, D44: DS8286D-D111, symbol robotron_ec1834:DS8286D-D111
- added D13, D67: DL074, symbol robotron_ec1834:DL074
- added D30, D31: DL374, symbol robotron_ec1834:DL374
- added D34, D59, D82, D87: DL004D, symbol RFT_Digitalschaltkreise:DL004D
- added D37, D62: DL032D, symbol RFT_Digitalschaltkreise:DL032D
- added D47: DL008D, symbol robotron_ec1834:DL008D
- added D5: DL030D, symbol RFT_Digitalschaltkreise:DL030D
- added D52, D58, D60: 74HC74, symbol robotron_ec1834:74HC74
- added D53: KR580WI53, Package_DIP:DIP-24_W15.24mm, symbol robotron_ec1834:KR580WI53
- added D54: 8255A, Package_DIP:DIP-40_W15.24mm, symbol robotron_ec1834:8255A
- added D55: UC8821, EC1834-Board:EMR-64_W22.86mm, symbol robotron_ec1834:UC8821
- added D56: 2716, Package_DIP:DIP-24_W15.24mm, symbol robotron_ec1834:2716
- added D57, D69, D70, D72, D88: DL008D, symbol RFT_Digitalschaltkreise:DL008D
- added D63: DL010D-D63, symbol robotron_ec1834:DL010D-D63
- added D65, D66: DS8205, symbol robotron_ec1834:DS8205
- added D68: 74S51, symbol robotron_ec1834:74S51
- added D71: DL002D, symbol RFT_Digitalschaltkreise:DL002D
- added D85, D86: KR531KP11, symbol robotron_ec1834:KR531KP11
- added D90: KR531LI1, symbol robotron_ec1834:KR531LI1
- added R11: 1k, Resistor_THT:R_Array_SIP6, symbol Device:R_Network05_Split
- added R12: 4k7, Resistor_THT:R_Array_SIP10, symbol Device:R_Network09_Split
- added R14, R15, R16: 30, Resistor_THT:R_Array_SIP8, symbol Device:R_Pack04_SIP_Split
- added R17: 4k7, Resistor_THT:R_Axial_DIN0309_L9.0mm_D3.2mm_P12.70mm_Horizontal, symbol Device:R
- added R18: 30, Resistor_THT:R_Axial_DIN0309_L9.0mm_D3.2mm_P12.70mm_Horizontal, symbol Device:R
- added R23, R40, R41: 4k7, Resistor_THT:R_Array_SIP10, symbol Device:R_Network09
- added R24, R25: 1k, Resistor_THT:R_Axial_DIN0309_L9.0mm_D3.2mm_P12.70mm_Horizontal, symbol Device:R
- added R52: 3k9, Resistor_THT:R_Array_SIP8, symbol Device:R_Network07_Split
- added SW1: SW_DIP_x08, Button_Switch_THT:SW_DIP_SPSTx08_Slide_9.78x22.5mm_W7.62mm_P2.54mm, symbol Switch:SW_DIP_x08
Connections:
- net +5V: now also D56.21 (VPP), R11.1 (R1.1), R23.1 (common)
- net 1: now also D55.39 (D1), D56.10 (D1)
- net 2: now also D55.38 (D2), D56.11 (D2)
- net 3: now also D55.37 (D3), D56.13 (D3)
- net 4: now also D55.24 (D4), D56.14 (D4)
- net D0: now also D111.19 (B0)
- net D1: now also D111.18 (B1)
- net GND: now also D56.18 (CE), D56.20 (OE), SW1.1, SW1.2, SW1.3, SW1.4, SW1.5, SW1.6, SW1.7, SW1.8
- new net: D55.25 (A0), D56.08 (A0)
- new net: D55.26 (A1), D56.07 (A1)
- new net: D55.27 (A2), D56.06 (A2)
- new net: D55.28 (A3), D56.05 (A3)
- new net: D55.29 (A4), D56.04 (A4)
- new net: D55.30 (A5), D56.03 (A5)
- new net: D55.31 (A6), D56.02 (A6)
- new net: D55.32 (A7), D56.01 (A7)
- new net: D55.33 (A8), D56.23 (A8)
- new net: D55.34 (A9), D56.22 (A9)
- new net: D55.35 (A10), D56.19 (A10)
- new net: D55.45 (P07), R23.9 (R8), SW1.9
- new net: D55.46 (P06), R23.8 (R7), SW1.10
- new net: D55.47 (P05), R23.7 (R6), SW1.11
- new net: D55.49 (P04), R23.6 (R5), SW1.12
- new net: D55.50 (P03), R23.5 (R4), SW1.13
- new net: D55.51 (P02), R23.4 (R3), SW1.14
- new net: D55.52 (P01), R23.3 (R2), SW1.15
- new net: D55.53 (P00), R23.2 (R1), SW1.16
- new net: D55.55 (P35), D82.1 (A1)
- new net: D55.61 (P37), D82.3 (A2)
- new net 0: D55.40 (D0), D56.09 (D0)
- new net 5: D55.23 (D5), D56.15 (D5)
- new net 6: D55.22 (D6), D56.16 (D6)
- new net 7: D55.21 (D7), D56.17 (D7)
- no-connect marks 40 -> 5
Other:
- note removed: "Bei der Verwend. d. K1810GF84 entfällt E1"
- note removed: "D64A PIN Pos abweichend von Zeichnung 1.13.120030.0/04"
- title: (none) -> EC1834_201.2
