File: EC1834_201.2.kicad_sch (KiCad schematic)
At the start: 58 parts, among them SW1 SW_DIP_x08

Commit message: corrected page names progress on page 2 added 1834 bus symbol
Parts:
- added BR1, WD4, WD5: SolderJumper_2_Bridged, symbol Jumper:SolderJumper_2_Bridged
- added E4: SolderJumper_2_Bridged, symbol Connector_Generic:Conn_02x01
- added L1: L_Ferrite_Coupled_Small_15263748, symbol robotron_ec1834:L_Ferrite_Coupled_Small_15263748
- added R53, R54: 100, Resistor_THT:R_Axial_DIN0309_L9.0mm_D3.2mm_P12.70mm_Horizontal, symbol Device:R
- added X4: Lautsprecher, symbol Connector_Generic:Conn_01x02
- added X7: DB9_Female, symbol Connector:DB9_Female
Connections:
- net +5V: now also C7.1, D100.1 (VPP), D100.27 (~{PGM}), D101.1 (VPP), D101.27 (~{PGM}), D115.1 (VPP), D115.27 (~{PGM}), D116.1 (VPP), D116.27 (~{PGM}), D55.60 (P30), D55.63 (XTAL2), D82.4 (Y2), R24.1, R25.1, R25.2, R40.1 (common), R41.1 (common), E4.1 (Pin_1), L1.5, L1.7
- net GND: now also C7.2, C8.2, D55.48 (GND), L1.6, R53.2, X4.2 (Pin_2)
- net ~{CSROM1}: now reaches D101.22 (OE)
- net ~{CSROM1}: now also D116.22 (OE), D66.07 (O7)
- net ~{CSROM0}: now reaches D115.22 (OE)
- net ~{CSROM0}: now also D100.22 (OE), D66.10 (O5)
- net at D85.1 (WS): now also D58.9, D67.2 (D), D86.1 (WS)
- net at D85.12 (F3): now also R15.5 (R3.1)
- net at D85.15 (S): now also D86.15 (S), R53.1
- net at D85.4 (F0): now also R15.4 (R2.2)
- net at D85.7 (F1): now also R15.2 (R1.2)
- net at D85.9 (F2): now also R15.8 (R4.2)
- net at D86.12 (F3): now also R14.5 (R3.1)
- net at D86.14 (A3): now also D68.6
- net at D86.4 (F0): now also R14.3 (R2.1)
- net at D86.7 (F1): now also R14.1 (R1.1)
- net at D86.9 (F2): now also R14.8 (R4.2)
- net at D5.11 (G): now also R11.2 (R1.2)
- net at D5.8 (Y): now also D66.04 (E1)
- net at D111.11 (T): now also D112.11 (T)
- net D7: now reaches D111.12 (B7)
- net D6: now reaches D111.13 (B6)
- net D5: now reaches D111.14 (B5)
- net D4: now reaches D111.15 (B4)
- net D3: now reaches D111.16 (B3)
- net D2: now reaches D111.17 (B2)
- net at D111.9 (OE): now also D62.8 (Y3)
- net at D112.9 (OE): now also D62.11 (Y4)
- net at D59.8 (Y4): now also D37.9 (A3)
- net at D44.11 (T): now also D37.8 (Y3)
- net at D71.1 (Y1): now also D37.10 (B3)
- net at D71.2 (A1): now also D62.6 (Y2)
- net at D30.1 (OE): now also D16.8 (Y3)
- net at D30.11 (C): now also D10.5 (B2), D10.8 (Y3), D31.11 (C), D54.11 (PC6), D63.11 (C3)
- net at D31.1 (OE): now also D16.11 (Y4)
- net at D31.19 (Q7): now also D13.12 (D)
- net at D87.1 (A1): now also D37.6 (Y2)
- net at D87.2 (Y1): now also D16.10 (B3), D16.12 (A4)
- net PA3: now reaches D54.1 (PA3)
- net PA3: now also D55.17 (P13)
- net OUT2: now reaches D54.12 (PC5)
- net OUT2: now also D39.5 (B2), D53.17 (OUT2)
- net PC4: now reaches D54.13 (PC4)
- net PC4: now also D55.12 (P34)
- net GATE2: now reaches D54.18 (PB0)
- net GATE2: now also D53.16 (GATE2)
- net PB1: now reaches D54.19 (PB1)
- net PB1: now also D39.4 (A2)
- net PA2: now reaches D54.2 (PA2)
- net PA2: now also D55.18 (P12)
- net PB2: now reaches D54.20 (PB2)
- net PB2: now also D55.10 (P20)
- net at D54.24 (PB6): now also D55.54 (P32)
- net at D54.25 (PB7): now also D55.11 (P33)
- net PA1: now reaches D54.3 (PA1)
- net PA1: now also D55.19 (P11)
- net PA7: now reaches D54.37 (PA7)
- net PA7: now also D55.13 (P17)
- net PA6: now reaches D54.38 (PA6)
- net PA6: now also D55.14 (P16)
- net PA5: now reaches D54.39 (PA5)
- net PA5: now also D55.15 (P15)
- net PA0: now reaches D54.4 (PA0)
- net PA0: now also D55.20 (P10)
- net PA4: now reaches D54.40 (PA4)
- net PA4: now also D55.16 (P14)
- net at D53.13 (OUT1): now also D52.11 (C)
- net at D53.9 (CLK0): now also D52.5
- net at D55.02 (P31): now also C8.1, D82.2 (Y1), R24.2, L1.8
- net at D55.64 (Ucc): now also E4.2 (Pin_2)
- net at D13.11 (C): now also D59.12 (Y6)
- net at D13.9: now also D90.13 (B4)
- net at D59.13 (A6): now also D71.4 (Y2)
- net at D47.5 (B2): now also R12.4 (R3.2)
- net at D47.6 (Y2): now also D10.13 (B4)
- net at D10.11 (Y4): now also D63.9 (A3)
- net at D10.4 (A2): now also R11.3 (R2.2)
- net at D10.6 (Y2): now also D10.9 (A3)
- net at D10.10 (B3): now also D34.6 (Y3)
- net at D62.10 (B3): now also D62.12 (A4), R17.1, WD5.1 (A)
- net at D90.3 (Y1): now also WD5.2 (B)
- net at D63.8 (Y3): now also D90.12 (A4)
- net at D60.10 (S): now also R52.8 (R7.2)
- net at D60.11 (C): now also D57.10 (B3), D57.12 (A4), D57.13 (B4), D57.3 (Y1), D57.9 (A3), D67.3 (C)
- net at D60.9: now also D69.10 (B3), D88.5 (B2)
- net at D58.11 (C): now also D57.11 (Y4)
- net at D58.12 (D): now also D58.5
- net at D58.13 (R): now also D87.8 (Y4)
- net at D60.1 (R): now also D34.12 (Y6)
- net at D60.2 (D): now also D71.13 (Y4)
- net at D58.2 (D): now also D69.8 (Y3)
- net at D57.1 (A1): now also D57.2 (B1)
- net at D69.9 (A3): now also BR1.2 (B)
- net at D69.1 (A1): now also D67.5
- net at D69.2 (B1): now also D59.4 (Y2)
- net at D69.3 (Y1): now also D72.10 (B3)
- net at D67.1 (R): now also D70.1 (A1), D70.4 (A2)
- net at D72.8 (Y3): now also R16.5 (R3.1)
- net at D72.9 (A3): now also R52.4 (R3.2)
- net at D72.11 (Y4): now also R16.7 (R4.1)
- net at D72.12 (A4): now also D69.11 (Y4)
- net at D72.13 (B4): now also R52.3 (R2.2)
- net at D69.13 (B4): now also D59.6 (Y3)
- net at D88.4 (A2): now also R52.7 (R6.2)
- net at D88.6 (Y2): now also R18.2
- net at D70.2 (B1): now also D70.8 (Y3)
- net at D70.3 (Y1): now also D72.2 (B1)
- net at D70.5 (B2): now also D70.11 (Y4)
- net at D70.6 (Y2): now also D72.5 (B2)
- net at D72.1 (A1): now also R52.6 (R5.2)
- net at D72.3 (Y1): now also R16.1 (R1.1)
- net at D72.4 (A2): now also R52.5 (R4.2)
- net at D72.6 (Y2): now also R16.3 (R2.1)
- net at D88.1 (A1): now also D65.15 (O0), D70.12 (A4)
- net at D88.2 (B1): now also D65.14 (O1), D70.9 (A3)
- net at D88.3 (Y1): now also D87.9 (A4)
- net at D70.13 (B4): now also D70.10 (B3)
- net at D68.8: now also D71.12 (B4)
- net at D65.04 (E1): now also WD4.2 (B)
- net at D65.05 (E2): now also R54.1
- net at D52.2 (D): now also D52.6
- net at D52.10 (S): now also D52.12 (D)
- net at D39.6 (Y2): now also X4.1 (Pin_1)
- new net: L1.1, X7.1, X7.6
- new net: L1.2, X7.5, X7.9
- new net: R54.2, WD4.1 (A)
- new net KBCLK: L1.3, X7.4
- new net KBDATA: L1.4, X7.2
- no-connect marks 5 -> 39
Other:
- moved on the sheet: C7, C8, D100A, D10B, D10C, D10D, D115A, D13B, D16C, D16D, D34C, D34F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

Commit message: Schematics almost done, need to connect busses
Parts:
- added PS3: PS3, symbol Connector_Generic:Conn_01x09
- added PS4: PS4, symbol Connector_Generic:Conn_01x03
- renumbered SW1 to S1
Connections:
- net +5V: now also D13.10 (S), D47.4 (A2), D5.6 (F), D52.10 (S), D52.12 (D), D52.4 (S), R17.2
- net 0: now also R15.6 (R3.2)
- net 1: now also R15.1 (R1.1)
- net 2: now also R15.3 (R2.1)
- net 3: now also R15.7 (R4.1)
- net 4: now also R14.4 (R2.2)
- net 5: now also R14.7 (R4.1)
- net 6: now also R14.2 (R1.2)
- net 7: now also R14.6 (R3.2)
- net D0: now also D44.19 (B0)
- net D1: now also D44.18 (B1)
- net D2: now also D44.17 (B2)
- net D3: now also D44.16 (B3)
- net D4: now also D44.15 (B4)
- net D5: now also D44.14 (B5)
- net D6: now also D44.13 (B6)
- net D7: now also D44.12 (B7)
- net GND: now also D100.20 (CS), D101.20 (CS), D115.20 (CS), D116.20 (CS), D31.14 (D5), D31.17 (D6), D31.18 (D7), R54.2, WD4.1 (A)
- net PB3: now also D54.21 (PB3)
- net XA1: now reaches D101.10 (A0)
- net XA1: now also D100.10 (A0), D115.10 (A0), D116.10 (A0), D53.20 (A1), D54.8 (A1)
- net MD8: now reaches D101.11 (D0)
- net MD8: now also D100.11 (D0), D112.1 (A0), R41.2 (R1)
- net MD9: now reaches D101.12 (D1)
- net MD9: now also D100.12 (D1), D112.2 (A1), R41.3 (R2)
- net MD10: now reaches D101.13 (D2)
- net MD10: now also D100.13 (D2), D112.3 (A2), R41.4 (R3)
- net MD11: now reaches D101.15 (D3)
- net MD11: now also D100.15 (D3), D112.4 (A3), R41.5 (R4)
- net MD12: now reaches D101.16 (D4)
- net MD12: now also D100.16 (D4), D112.5 (A4), R41.6 (R5)
- net MD13: now reaches D101.17 (D5)
- net MD13: now also D100.17 (D5), D112.6 (A5), R41.7 (R6)
- net MD14: now reaches D101.18 (D6)
- net MD14: now also D100.18 (D6), D112.7 (A6), R41.8 (R7)
- net MD15: now reaches D101.19 (D7)
- net MD15: now also D100.19 (D7), D112.8 (A7), R41.9 (R8)
- net XA13: now reaches D101.2 (A12)
- net XA13: now also D100.2 (A12), D115.2 (A12), D116.2 (A12)
- net XA11: now reaches D101.21 (A10)
- net XA11: now also D100.21 (A10), D115.21 (A10), D116.21 (A10)
- net XA12: now reaches D101.23 (A11)
- net XA12: now also D100.23 (A11), D115.23 (A11), D116.23 (A11)
- net XA10: now reaches D101.24 (A9)
- net XA10: now also D100.24 (A9), D115.24 (A9), D116.24 (A9)
- net XA9: now reaches D101.25 (A8)
- net XA9: now also D100.25 (A8), D115.25 (A8), D116.25 (A8), D62.4 (A2), D62.5 (B2)
- net XA8: now reaches D101.3 (A7)
- net XA8: now also D100.3 (A7), D115.3 (A7), D116.3 (A7)
- net XA7: now reaches D101.4 (A6)
- net XA7: now also D100.4 (A6), D115.4 (A6), D116.4 (A6)
- net XA6: now reaches D101.5 (A5)
- net XA6: now also D100.5 (A5), D115.5 (A5), D116.5 (A5)
- net XA5: now reaches D101.6 (A4)
- net XA5: now also D100.6 (A4), D115.6 (A4), D116.6 (A4)
- net XA4: now reaches D101.7 (A3)
- net XA4: now also D100.7 (A3), D115.7 (A3), D116.7 (A3)
- net XA3: now reaches D101.8 (A2)
- net XA3: now also D100.8 (A2), D115.8 (A2), D116.8 (A2)
- net XA2: now reaches D101.9 (A1)
- net XA2: now also D100.9 (A1), D115.9 (A1), D116.9 (A1)
- net MD0: now reaches D116.11 (D0)
- net MD0: now also D111.1 (A0), D115.11 (D0), R40.2 (R1)
- net MD1: now reaches D116.12 (D1)
- net MD1: now also D111.2 (A1), D115.12 (D1), R40.3 (R2)
- net MD2: now reaches D116.13 (D2)
- net MD2: now also D111.3 (A2), D115.13 (D2), R40.4 (R3)
- net MD3: now reaches D116.15 (D3)
- net MD3: now also D111.4 (A3), D115.15 (D3), R40.5 (R4)
- net MD4: now reaches D116.16 (D4)
- net MD4: now also D111.5 (A4), D115.16 (D4), R40.6 (R5)
- net MD5: now reaches D116.17 (D5)
- net MD5: now also D111.6 (A5), D115.17 (D5), R40.7 (R6)
- net MD6: now reaches D116.18 (D6)
- net MD6: now also D111.7 (A6), D115.18 (D6), R40.8 (R7)
- net MD7: now reaches D116.19 (D7)
- net MD7: now also D111.8 (A7), D115.19 (D7), R40.9 (R8)
- net PS4:3: now reaches D85.15 (S), D86.15 (S), R53.1
- net PS4:3: now also PS4.3 (Pin_3)
- net A16: now reaches D5.1 (A)
- net PS1:4: now reaches D5.11 (G), R11.2 (R1.2)
- net ~{AEN}: now reaches D5.12 (H)
- net A17: now reaches D5.2 (B)
- net A17: now also D65.01 (A0)
- net A18: now reaches D5.3 (C)
- net A18: now also D65.02 (A1)
- net A19: now reaches D5.4 (D)
- net A19: now also D65.03 (A2)
- net A15: now reaches D5.5 (E)
- net ~{ROMADRSEL}: now reaches D5.8 (Y), D66.04 (E1)
- net ~{ROMADRSEL}: now also D90.2 (B1)
- net 5PW2: now reaches D66.01 (A0)
- net 5PW2: now also D53.11 (GATE0), D53.14 (GATE1), D66.03 (A2)
- net A14: now reaches D66.02 (A1)
- net ~{XMEMR}: now reaches D66.05 (E2)
- net ~{RESETDRV}: now reaches D66.06 (E3)
- net ~{RESETDRV}: now also D13.13 (R), D52.1 (R), D55.59 (RESET)
- net MEMR: now reaches D111.11 (T), D112.11 (T)
- net D15: now reaches D112.12 (B7)
- net D14: now reaches D112.13 (B6)
- net D13: now reaches D112.14 (B5)
- net D12: now reaches D112.15 (B4)
- net D11: now reaches D112.16 (B3)
- net D10: now reaches D112.17 (B2)
- net D9: now reaches D112.18 (B1)
- net D8: now reaches D112.19 (B0)
- net ~{INTA}: now reaches D59.9 (A4)
- net XD0: now reaches D44.1 (A0)
- net XD0: now also D30.2 (Q0), D31.2 (Q0), D53.8 (D0), D54.34 (D0)
- net XD1: now reaches D44.2 (A1)
- net XD1: now also D30.5 (Q1), D31.5 (Q1), D53.7 (D1), D54.33 (D1)
- net XD2: now reaches D44.3 (A2)
- net XD2: now also D30.6 (Q2), D31.6 (Q2), D53.6 (D2), D54.32 (D2)
- net XD3: now reaches D44.4 (A3)
- net XD3: now also D30.9 (Q3), D31.9 (Q3), D53.5 (D3), D54.31 (D3)
- net XD4: now reaches D44.5 (A4)
- net XD4: now also D30.12 (Q4), D31.12 (Q4), D53.4 (D4), D54.30 (D4)
- net XD5: now reaches D44.6 (A5)
- net XD5: now also D30.15 (Q5), D31.15 (Q5), D53.3 (D5), D54.29 (D5)
- net XD6: now reaches D44.7 (A6)
- net XD6: now also D30.16 (Q6), D31.16 (Q6), D53.2 (D6), D54.28 (D6)
- net XD7: now reaches D44.8 (A7)
- net XD7: now also D13.12 (D), D30.19 (Q7), D31.19 (Q7), D53.1 (D7), D54.27 (D7)
- net AENBRD: now reaches D44.9 (OE)
- net ~{XIOR}: now reaches D71.3 (B1)
- net ~{XIOR}: now also D37.5 (B2), D53.22 (~{RD}), D54.5 (RD)
- net ~{OCHCK}: now reaches D10.5 (B2), D10.8 (Y3), D30.11 (C), D31.11 (C), D54.11 (PC6), D63.11 (C3)
- net A4: now reaches D30.13 (D4)
- net A5: now reaches D30.14 (D5)
- net A6: now reaches D30.17 (D6)
- net A7: now reaches D30.18 (D7)
- net A0: now reaches D30.3 (D0)
- net A0: now also D59.3 (A2), D62.9 (A3), D68.2
- net A1: now reaches D30.4 (D1)
- net A2: now reaches D30.7 (D2)
- net A3: now reaches D30.8 (D3)
- net ~{IOW}: now reaches D31.13 (D4)
- net A8: now reaches D31.3 (D0)
- net A8: now also D68.4
- net A9: now reaches D31.4 (D1)
- net ~{BHE}: now reaches D31.7 (D2)
- net ~{BHE}: now also D59.5 (A3), D62.13 (B4)
- net ~{IOR}: now reaches D31.8 (D3)
- net PCK: now reaches D54.10 (PC7)
- net PCK: now also D60.5
- net ~{ENBRAMPCK}: now reaches D54.22 (PB4)
- net ~{ENBRAMPCK}: now also D34.13 (A6)
- net ~{ENIOCK}: now reaches D54.23 (PB5)
- net ~{ENIOCK}: now also D34.5 (A3)
- net PB6: now reaches D54.24 (PB6), D55.54 (P32)
- net PB7: now reaches D54.25 (PB7), D55.11 (P33)
- net RESET: now reaches D54.35 (RESET)
- net ~{XIOW}: now reaches D54.36 (WR)
- net ~{XIOW}: now also D71.6 (B2)
- net ~{PPICS}: now reaches D54.6 (CS)
- net XA0: now reaches D54.9 (A0)
- net XA0: now also D16.13 (B4), D53.19 (A0)
- net IRQ0: now reaches D53.10 (OUT0)
- net at D53.15 (CLK1): now also D52.5, D53.18 (CLK2), D53.9 (CLK0)
- net ~{TIMERCS}: now reaches D53.21 (~{CS})
- net ~{XOW}: now reaches D53.23 (~{WR})
- net IRQ1: now reaches D55.01 (P36)
- net NPINSTLSW: now reaches D55.46 (P06), R23.8 (R7), S1.10
- net NPINSTLSW: now also D10.12 (A4)
- net CLK86: now reaches D55.62 (XTAL1)
- net ~{A0}: now reaches D16.9 (A3)
- net ~{A0}: now also D59.4 (Y2), D68.10, D69.2 (B1)
- net ~{NMIREGCS}: now reaches D71.5 (A2)
- net NPNPI: now reaches D47.5 (B2), R12.4 (R3.2)
- net ~{IOCHCK}: now reaches D10.4 (A2), R11.3 (R2.2)
- net ~{MEMADRSEL}: now reaches D62.10 (B3), D62.12 (A4), R17.1, WD5.1 (A)
- net ~{RAMADRSEL}: now reaches D90.1 (A1)
- net ~{RAMADRSEL}: now also D71.11 (A4)
- net ~{PCK}: now reaches D63.10 (B3)
- net ~{PCK}: now also D60.4 (S), D60.6
- net NMI: now reaches D90.11 (Y4)
- net ~{MEMR}: now reaches D60.3 (C)
- net PS4:1: now reaches BR1.2 (B), D69.9 (A3)
- net PS4:1: now also PS4.1 (Pin_1)
- net PS3:5: now reaches D72.9 (A3), R52.4 (R3.2)
- net PS3:5: now also PS3.5 (Pin_5)
- net PS3:6: now reaches D72.13 (B4), R52.3 (R2.2)
- net PS3:6: now also PS3.6 (Pin_6)
- net BHE: now reaches D59.6 (Y3), D69.13 (B4)
- net BHE: now also D68.1
- net PS3:2: now reaches D88.4 (A2), R52.7 (R6.2)
- net PS3:2: now also PS3.2 (Pin_2)
- net PS3:3: now reaches D72.1 (A1), R52.6 (R5.2)
- net PS3:3: now also PS3.3 (Pin_3)
- net PS3:4: now reaches D72.4 (A2), R52.5 (R4.2)
- net PS3:4: now also PS3.4 (Pin_4)
- net DACK0: now reaches D68.3
- net ~{DACK0}: now reaches D68.5
- net ~{DACK0}: now also D70.10 (B3), D70.13 (B4)
- net MDPOE: now reaches D68.13
- net MDPEE: now reaches D68.9
- net at D65.04 (E1), WD4.2 (B): now also R12.5 (R4.2)
- net PS4:2: now reaches D65.05 (E2), R54.1
- net PS4:2: now also PS4.2 (Pin_2)
- net ~{DACK0BRD}: now reaches D65.06 (E3)
- net ~{DACK0BRD}: now also D52.13 (R)
- net ~{NMIADRCS}: now reaches D37.4 (A2)
- net PCLK: now reaches D52.3 (C)
- net DRQ0: now reaches D52.9
- net ~{RAS1}: now reaches R16.2 (R1.2)
- net ~{RAS0}: now reaches R16.4 (R2.2)
- net ~{CASL}: now reaches R16.6 (R3.2)
- net ~{CASH}: now reaches R16.8 (R4.2)
- net 8: now reaches R18.1
- new net PS3:1: PS3.1 (Pin_1)
- new net PS3:7: PS3.7 (Pin_7)
- no-connect marks 39 -> 44
Other:
- note added: "5P"
- moved on the sheet: D115A, E4, R40
