File: Power.kicad_sch (KiCad schematic)
At the start: 236 parts, among them K10 100n, K100 100n, K101 100, K102 100n, K103 100n, K104 100n, K105 100n, K106 100n, K107 100n, K108 100n, K109 100n, K11 100n, K110 100n, K111 100n, K112 100n, K113 100n, K114 100n, K115 100n, K116 100n, K117 100n, K118 100n, K12 100n, K120 100n, K121 100n, K122 100n, K123 100n, K124 100n, K125 100n, K126 100n, K13 100n, K14 100n, K15 100n, K16 100n, K199 100n, K2 100n, K21 100n, K22 100n, K23 100n, K24 100n, K25 100n, K26 100n, K27 100n, K28 100n, K29 100n, K3 100n, K30 100n, K31 100n, K32 100n, K33 100n, K34 100n, K35 100n, K36 100n, K37 100n, K38 100n, K39 100n, K4 100n, K40 100n, K43 100n, K44 100n, K45 100n, K46 100n, K47 100n, K48 100n, K49 100n, K5 100n, K50 100n, K51 100n, K52 100n, K53 100n, K54 100n, K56 100n, K57 100n, K58 100n, K59 100, K6 100n, K60 100n, K61 100n, K62 100n, K63 100n, K64 100n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

Commit message: Improved schematics
Parts:
- added C101, C102, C103, C104, C105, C106, C107, C108, C109, C110, C111, C112, C113, C114, C115, C116, C117, C118, C119, C120, C121, C122, C123, C2, C3, C4: 47µF, Capacitor_THT:CP_Radial_D12.5mm_P5.00mm, symbol Device:C
- added E6, E7, E8: Conn_01x02, symbol Connector_Generic:Conn_01x02
- added K1, K18, K19, K55: 100n, Capacitor_THT:C_Disc_D4.3mm_W1.9mm_P5.00mm, symbol Device:C
- added R12: 4k7, Resistor_THT:R_Array_SIP10, symbol Device:R_Network09_Split
- added R22: 130, Resistor_THT:R_Axial_DIN0309_L9.0mm_D3.2mm_P12.70mm_Horizontal, symbol Device:R
- added R30, R31: 30, Resistor_THT:R_Axial_DIN0309_L9.0mm_D3.2mm_P12.70mm_Horizontal, symbol Device:R
- added R32, R33, R4: 1k, Resistor_THT:R_Axial_DIN0309_L9.0mm_D3.2mm_P12.70mm_Horizontal, symbol Device:R
- added V3, V4, V5, V6: LED, symbol Device:LED
- K10, K100, K102, K103, K104, K105, K106, K107, K108, K109, K11, K110, K111, K112, K113, K114, K115, K116, K117, K118, K12, K120, K121, K122, K123, K124, K125, K126, K13, K14, K15, K16, K2, K21, K22, K23, K24, K25, K26, K27, K28, K29, K3, K30, K31, K32, K33, K34, K35, K36, K37, K38, K39, K4, K40, K43, K44, K45, K46, K47, K48, K49, K5, K50, K51, K52, K53, K54, K56, K57, K58, K6, K60, K61, K62, K63, K64, K65, K66, K67, K68, K69, K7, K70, K71, K72, K73, K74, K75, K76, K77, K78, K79, K8, K80, K81, K82, K83, K84, K85, K86, K87, K88, K89, K9, K90, K91, K92, K93, K94, K95, K96, K97, K99: footprint (none) -> Capacitor_THT:C_Disc_D4.3mm_W1.9mm_P5.00mm
- K101, K59, K98: value 100 -> 100n; footprint (none) -> Capacitor_THT:C_Disc_D4.3mm_W1.9mm_P5.00mm
- K119: renamed from K199; footprint (none) -> Capacitor_THT:C_Disc_D4.3mm_W1.9mm_P5.00mm
Connections:
- net +5P: no longer K56.2
- net GND: now also K1.2, K18.2, K19.2, K55.2; no longer K56.1
- new net +5V: K1.1, K18.1, K19.1, K55.1
- new net -5V: C3.2
Other:
- moved on the sheet: K56

Commit message: Corrected schema names added bus signals
Parts:
- added unit 1 of D11
- added unit 2 of D126
- added unit 2 of D14
- added unit 1 of D3
- added unit 4 of D34
- added unit 4 of D37
- added unit 1 of D63
- added unit 2 of D69
- added unit 3 of D82
- added unit 4 of D82
- added unit 5 of D82
- added unit 6 of D82
- added unit 5 of D87
- added unit 2 of D87
- added R11: 1k, Resistor_THT:R_Array_SIP6, symbol Device:R_Network05_Split
- added X2: Conn_01x06, symbol Connector_Generic:Conn_01x06
- added X3: Conn_01x08, symbol Connector_Generic:Conn_01x08
Connections:
- net +12V: now also C4.1, R32.1, X2.1 (Pin_1)
- net +5P: now also D37.12 (A4), D82.11 (A5), D82.13 (A6), D82.5 (A3), D82.9 (A4), D87.11 (A5)
- net +5V: now also C101.1, C102.1, C103.1, C104.1, C105.1, C106.1, C107.1, C108.1, C109.1, C110.1, C111.1, C112.1, C113.1, C114.1, C115.1, C116.1, C117.1, C118.1, C119.1, C120.1, C121.1, C122.1, C123.1, R12.1 (R1.1), R22.2, R30.1, R4.1, X3.5 (Pin_5), X3.6 (Pin_6), X3.7 (Pin_7), X3.8 (Pin_8)
- net -12V: now also C2.2, R33.2, X2.3 (Pin_3)
- net -5V: now also R31.2, X2.6 (Pin_6)
- net GND: now also C101.2, C102.2, C103.2, C104.2, C105.2, C106.2, C107.2, C108.2, C109.2, C110.2, C111.2, C112.2, C113.2, C114.2, C115.2, C116.2, C117.2, C118.2, C119.2, C120.2, C121.2, C122.2, C123.2, C2.1, C3.1, C4.2, E6.1 (Pin_1), E6.2 (Pin_2), E7.1 (Pin_1), E7.2 (Pin_2), E8.1 (Pin_1), E8.2 (Pin_2), V3.1 (K), V4.2 (A), V5.1 (K), V6.2 (A), D11.5 (D1), D126.10 (S), D14.5 (C2), D3.1 (A1), D34.9 (A4), D63.13 (C1), D69.5 (B2), D87.3 (A2), X2.2 (Pin_2), X2.4 (Pin_4), X2.5 (Pin_5), X3.1 (Pin_1), X3.2 (Pin_2), X3.3 (Pin_3), X3.4 (Pin_4)
- net at R32.2: now also V5.2 (A)
- net at V3.2 (A): now also R30.2
- net at V6.1 (K): now also R33.1
- net 5PW1: now reaches R4.2
- net at R31.1: now also V4.1 (K)
- net 5PW2: now reaches R12.2 (R1.2)
- no-connect marks 0 -> 30
Other:
- moved on the sheet: C2, C3, R12A, R31, R4, V4
