File: Power.kicad_sch (KiCad schematic)
At the start: 283 parts, among them K1 100n, K10 100n, K100 100n, K101 100n, K102 100n, K103 100n, K104 100n, K105 100n, K106 100n, K107 100n, K108 100n, K109 100n, K11 100n, K110 100n, K111 100n, K112 100n, K113 100n, K114 100n, K115 100n, K116 100n, K117 100n, K118 100n, K119 100n, K12 100n, K120 100n, K121 100n, K122 100n, K123 100n, K124 100n, K125 100n, K126 100n, K13 100n, K14 100n, K15 100n, K16 100n, K18 100n, K19 100n, K2 100n, K21 100n, K22 100n, K23 100n, K24 100n, K25 100n, K26 100n, K27 100n, K28 100n, K29 100n, K3 100n, K30 100n, K31 100n, K32 100n, K33 100n, K34 100n, K35 100n, K36 100n, K37 100n, K38 100n, K39 100n, K4 100n, K40 100n, K43 100n, K44 100n, K45 100n, K46 100n, K47 100n, K48 100n, K49 100n, K5 100n, K50 100n, K51 100n, K52 100n, K53 100n, K54 100n, K55 100n, K56 100n, K57 100n, K58 100n, K59 100n, K6 100n, K60 100n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

Commit message: Page 1 & 2 connected Hierarchival connections created and tested
Connections:
- net +5P: now also K56.2
- net GND: now also K56.1
- no-connect marks 30 -> 31
Other:
- moved on the sheet: K56
Changed lines of the file:
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@@
   (junction (at 180.34 96.52) (diameter 0) (color 0 0 0 0)
   )
+  (junction (at 52.07 88.9) (diameter 0) (color 0 0 0 0)
+  )
   (junction (at 74.93 156.21) (diameter 0) (color 0 0 0 0)
   )
@@
   (junction (at 140.97 261.62) (diameter 0) (color 0 0 0 0)
   )
+  (no_connect (at 528.32 226.06))
   (no_connect (at 538.48 113.03))
   (no_connect (at 528.32 140.97))
@@
     (stroke (width 0) (type default) (color 0 0 0 0))
   )
+  (wire (pts (xy 39.37 96.52) (xy 52.07 96.52))
+    (stroke (width 0) (type default) (color 0 0 0 0))
+  )
   (wire (pts (xy 200.66 285.75) (xy 210.82 285.75))
     (stroke (width 0) (type default) (color 0 0 0 0))
@@
     (stroke (width 0) (type default) (color 0 0 0 0))
   )
+  (wire (pts (xy 39.37 88.9) (xy 52.07 88.9))
+    (stroke (width 0) (type default) (color 0 0 0 0))
+  )
   (wire (pts (xy 257.81 135.89) (xy 265.43 135.89))
     (stroke (width 0) (type default) (color 0 0 0 0))
@@
     (pin "2")
   )
-  (symbol (lib_id "Device:C") (at 99.06 81.28 0) (unit 1)
+  (symbol (lib_id "Device:C") (at 39.37 92.71 0) (unit 1)
     (in_bom yes) (on_board yes)
-    (property "Reference" "K56" (id 0) (at 99.06 78.74 0)
+    (property "Reference" "K56" (id 0) (at 39.37 90.17 0)
       (effects (font (size 1.27 1.27)) (justify left))
     )
-    (property "Value" "100n" (id 1) (at 99.06 83.82 0)
+    (property "Value" "100n" (id 1) (at 39.37 95.25 0)
       (effects (font (size 1.27 1.27)) (justify left))
     )
-    (property "Footprint" "Capacitor_THT:C_Disc_D4.3mm_W1.9mm_P5.00mm" (id 2) (at 100.0252 85.09 0)
+    (property "Footprint" "Capacitor_THT:C_Disc_D4.3mm_W1.9mm_P5.00mm" (id 2) (at 40.3352 96.52 0)
       (effects (font (size 1.27 1.27)) hide)
     )
-    (property "Datasheet" "~" (id 3) (at 99.06 81.28 0)
+    (property "Datasheet" "~" (id 3) (at 39.37 92.71 0)
       (effects (font (size 1.27 1.27)) hide)
     )
@@
   (symbol (lib_id "power:GND") (at 518.16 144.78 270) (unit 1)
     (in_bom yes) (on_board yes)
-    (property "Reference" "#PWR?" (id 0) (at 511.81 144.78 0)
+    (property "Reference" "#PWR0194" (id 0) (at 511.81 144.78 0)
       (effects (font (size 1.27 1.27)) hide)
     )
@@
   (symbol (lib_id "power:GND") (at 539.75 240.03 270) (unit 1)
     (in_bom yes) (on_board yes)
-    (property "Reference" "#PWR?" (id 0) (at 533.4 240.03 0)
+    (property "Reference" "#PWR0193" (id 0) (at 533.4 240.03 0)
       (effects (font (size 1.27 1.27)) hide)
     )
@@
   (symbol (lib_id "power:+5P") (at 542.29 226.06 90) (unit 1)
     (in_bom yes) (on_board yes)
-    (property "Reference" "#PWR?" (id 0) (at 546.1 226.06 0)
+    (property "Reference" "#PWR0200" (id 0) (at 546.1 226.06 0)
       (effects (font (size 1.27 1.27)) hide)
     )
@@
   (symbol (lib_id "power:GND") (at 518.16 190.5 270) (unit 1)
     (in_bom yes) (on_board yes)
-    (property "Reference" "#PWR?" (id 0) (at 511.81 190.5 0)
+    (property "Reference" "#PWR0190" (id 0) (at 511.81 190.5 0)
       (effects (font (size 1.27 1.27)) hide)
     )
@@
   (symbol (lib_id "power:GND") (at 518.16 161.29 270) (unit 1)
     (in_bom yes) (on_board yes)
-    (property "Reference" "#PWR?" (id 0) (at 511.81 161.29 0)
+    (property "Reference" "#PWR0195" (id 0) (at 511.81 161.29 0)
       (effects (font (size 1.27 1.27)) hide)
     )
@@
   (symbol (lib_id "power:+5P") (at 542.29 168.91 90) (unit 1)
     (in_bom yes) (on_board yes)
-    (property "Reference" "#PWR?" (id 0) (at 546.1 168.91 0)
+    (property "Reference" "#PWR0189" (id 0) (at 546.1 168.91 0)
       (effects (font (size 1.27 1.27)) hide)
     )
@@
   (symbol (lib_id "power:GND") (at 542.29 135.89 270) (unit 1)
     (in_bom yes) (on_board yes)
-    (property "Reference" "#PWR?" (id 0) (at 535.94 135.89 0)
+    (property "Reference" "#PWR0188" (id 0) (at 535.94 135.89 0)
       (effects (font (size 1.27 1.27)) hide)
     )
@@
   (symbol (lib_id "power:+5P") (at 518.16 201.93 90) (unit 1)
     (in_bom yes) (on_board yes)
-    (property "Reference" "#PWR?" (id 0) (at 521.97 201.93 0)
+    (property "Reference" "#PWR0197" (id 0) (at 521.97 201.93 0)
       (effects (font (size 1.27 1.27)) hide)
     )
@@
   (symbol (lib_id "power:GND") (at 518.16 226.06 270) (unit 1)
     (in_bom yes) (on_board yes)
-    (property "Reference" "#PWR?" (id 0) (at 511.81 226.06 0)
+    (property "Reference" "#PWR0198" (id 0) (at 511.81 226.06 0)
       (effects (font (size 1.27 1.27)) hide)
     )
@@
   (symbol (lib_id "power:+5P") (at 542.29 201.93 90) (unit 1)
     (in_bom yes) (on_board yes)
-    (property "Reference" "#PWR?" (id 0) (at 546.1 201.93 0)
+    (property "Reference" "#PWR0191" (id 0) (at 546.1 201.93 0)
       (effects (font (size 1.27 1.27)) hide)
     )
@@
   (symbol (lib_id "power:GND") (at 542.29 189.23 270) (unit 1)
     (in_bom yes) (on_board yes)
-    (property "Reference" "#PWR?" (id 0) (at 535.94 189.23 0)
+    (property "Reference" "#PWR0192" (id 0) (at 535.94 189.23 0)
       (effects (font (size 1.27 1.27)) hide)
     )
@@
   (symbol (lib_id "power:+5P") (at 518.16 213.36 90) (unit 1)
     (in_bom yes) (on_board yes)
-    (property "Reference" "#PWR?" (id 0) (at 521.97 213.36 0)
+    (property "Reference" "#PWR0199" (id 0) (at 521.97 213.36 0)
       (effects (font (size 1.27 1.27)) hide)
     )
@@
   (symbol (lib_id "power:GND") (at 518.16 171.45 270) (unit 1)
     (in_bom yes) (on_board yes)
-    (property "Reference" "#PWR?" (id 0) (at 511.81 171.45 0)
+    (property "Reference" "#PWR0196" (id 0) (at 511.81 171.45 0)
       (effects (font (size 1.27 1.27)) hide)
     )
@@
   (symbol (lib_id "power:+5P") (at 542.29 213.36 90) (unit 1)
     (in_bom yes) (on_board yes)
-    (property "Reference" "#PWR?" (id 0) (at 546.1 213.36 0)
+    (property "Reference" "#PWR0201" (id 0) (at 546.1 213.36 0)
       (effects (font (size 1.27 1.27)) hide)
     )

Commit message: Completed BUS Final checks required
Parts:
- added X5: PowerLED, Connector_PinHeader_2.54mm:PinHeader_1x02_P2.54mm_Vertical, symbol Connector_Generic:Conn_01x02
- D10, D11, D113, D114, D12, D126, D13, D14, D15, D16, D28, D29, D3, D32, D33, D34, D37, D38, D39, D40, D47, D5, D51, D52, D57, D58, D59, D6, D60, D62, D63, D67, D68, D69, D7, D70, D71, D72, D8, D82, D87, D88, D90: footprint (none) -> Package_DIP:DIP-14_W7.62mm
- D100, D101, D115, D116: footprint (none) -> Package_DIP:DIP-28_W15.24mm
- D111, D112, D2, D21, D22, D23, D24, D25, D26, D27, D30, D31, D44, D45, D64, D83, D84: footprint (none) -> Package_DIP:DIP-20_W7.62mm
- D35, D36, D46, D61, D65, D66, D85, D86, D89, D9: footprint (none) -> Package_DIP:DIP-16_W7.62mm
- E6, E7, E8: footprint (none) -> Connector_PinHeader_2.54mm:PinHeader_1x02_P2.54mm_Vertical
- V3, V4, V5, V6: footprint (none) -> LED_THT:LED_D5.0mm
- X2: footprint (none) -> TerminalBlock_RND:TerminalBlock_RND_205-00236_1x06_P5.08mm_Horizontal
- X3: footprint (none) -> TerminalBlock_RND:TerminalBlock_RND_205-00238_1x08_P5.08mm_Horizontal
Connections:
- net GND: now also X5.2 (Pin_2)
- net at R22.1: now also X5.1 (Pin_1)
Other:
- company: (none) -> Mario Gögel 2022
- title: (none) -> EC1834 Hauptplatine 201.2-Power

Commit message: Updated footprints Updated PCB
Parts:
- R22, R30, R31, R32, R33, R4: footprint Resistor_THT:R_Axial_DIN0309_L9.0mm_D3.2mm_P12.70mm_Horizontal -> EC1834-Board:R_Axial_L9.0mm_D1.8mm_P12.70mm_Horizontal
Changed lines of the file:
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@@
     (property "Reference" "R32" (id 0) (at 102.87 261.62 90))
     (property "Value" "1k" (id 1) (at 100.33 261.62 90))
-    (property "Footprint" "Resistor_THT:R_Axial_DIN0309_L9.0mm_D3.2mm_P12.70mm_Horizontal" (id 2) (at 98.552 261.62 90)
+    (property "Footprint" "EC1834-Board:R_Axial_L9.0mm_D1.8mm_P12.70mm_Horizontal" (id 2) (at 98.552 261.62 90)
       (effects (font (size 1.27 1.27)) hide)
     )
@@
     (property "Reference" "R30" (id 0) (at 93.98 287.02 90))
     (property "Value" "30" (id 1) (at 91.44 287.02 90))
-    (property "Footprint" "Resistor_THT:R_Axial_DIN0309_L9.0mm_D3.2mm_P12.70mm_Horizontal" (id 2) (at 89.662 287.02 90)
+    (property "Footprint" "EC1834-Board:R_Axial_L9.0mm_D1.8mm_P12.70mm_Horizontal" (id 2) (at 89.662 287.02 90)
       (effects (font (size 1.27 1.27)) hide)
     )
@@
     (property "Reference" "R4" (id 0) (at 129.54 259.08 90))
     (property "Value" "1k" (id 1) (at 129.54 261.62 90))
-    (property "Footprint" "Resistor_THT:R_Axial_DIN0309_L9.0mm_D3.2mm_P12.70mm_Horizontal" (id 2) (at 129.54 263.398 90)
+    (property "Footprint" "EC1834-Board:R_Axial_L9.0mm_D1.8mm_P12.70mm_Horizontal" (id 2) (at 129.54 263.398 90)
       (effects (font (size 1.27 1.27)) hide)
     )
@@
     (property "Reference" "R33" (id 0) (at 116.84 330.2 90))
     (property "Value" "1k" (id 1) (at 114.3 330.2 90))
-    (property "Footprint" "Resistor_THT:R_Axial_DIN0309_L9.0mm_D3.2mm_P12.70mm_Horizontal" (id 2) (at 112.522 330.2 90)
+    (property "Footprint" "EC1834-Board:R_Axial_L9.0mm_D1.8mm_P12.70mm_Horizontal" (id 2) (at 112.522 330.2 90)
       (effects (font (size 1.27 1.27)) hide)
     )
@@
     (property "Reference" "R31" (id 0) (at 102.87 317.5 90))
     (property "Value" "30" (id 1) (at 100.33 317.5 90))
-    (property "Footprint" "Resistor_THT:R_Axial_DIN0309_L9.0mm_D3.2mm_P12.70mm_Horizontal" (id 2) (at 98.552 317.5 90)
+    (property "Footprint" "EC1834-Board:R_Axial_L9.0mm_D1.8mm_P12.70mm_Horizontal" (id 2) (at 98.552 317.5 90)
       (effects (font (size 1.27 1.27)) hide)
     )
@@
     (property "Reference" "R22" (id 0) (at 87.63 265.43 90))
     (property "Value" "130" (id 1) (at 87.63 267.97 90))
-    (property "Footprint" "Resistor_THT:R_Axial_DIN0309_L9.0mm_D3.2mm_P12.70mm_Horizontal" (id 2) (at 87.63 269.748 90)
-      (effects (font (size 1.27 1.27)) hide)
-    )
+    (property "Footprint" "EC1834-Board:R_Axial_L9.0mm_D1.8mm_P12.70mm_Horizontal" (id 2) (at 87.63 269.748 90)
+      (effects (font (size 1.27 1.27)) hide)
+    )

Commit message: Completed PCB layout Changed PS5
Parts:
- removed C122, C123: 47µF, Capacitor_THT:CP_Radial_D12.5mm_P5.00mm, symbol Device:C
- removed K114, K21, K26, K28, K29, K32, K35, K40, K43, K46, K47, K56, K67, K82, K85, K87: 100n, Capacitor_THT:C_Disc_D4.3mm_W1.9mm_P5.00mm, symbol Device:C
- added K20: 100n, Capacitor_THT:C_Disc_D4.3mm_W1.9mm_P5.00mm, symbol Device:C
- C101, C102, C103, C104, C105, C106, C107, C108, C109, C110, C111, C112, C113, C114, C115, C116, C117, C119, C120, C121, C2, C3, C4: footprint Capacitor_THT:CP_Radial_D12.5mm_P5.00mm -> Capacitor_THT:CP_Radial_D5.0mm_P2.50mm
- C127: renamed from C118; footprint Capacitor_THT:CP_Radial_D12.5mm_P5.00mm -> Capacitor_THT:CP_Radial_D5.0mm_P2.50mm
- V3, V4, V5, V6: footprint LED_THT:LED_D5.0mm -> LED_THT:LED_D3.0mm
Connections:
- net +5V: now also K20.1
- net GND: now also K20.2
