File: Power.kicad_sch (KiCad schematic)
At the start: 267 parts, among them K1 100n, K10 100n, K100 100n, K101 100n, K102 100n, K103 100n, K104 100n, K105 100n, K106 100n, K107 100n, K108 100n, K109 100n, K11 100n, K110 100n, K111 100n, K112 100n, K113 100n, K115 100n, K116 100n, K117 100n, K118 100n, K119 100n, K12 100n, K120 100n, K121 100n, K122 100n, K123 100n, K124 100n, K125 100n, K126 100n, K13 100n, K14 100n, K15 100n, K16 100n, K18 100n, K19 100n, K2 100n, K20 100n, K22 100n, K23 100n, K24 100n, K25 100n, K27 100n, K3 100n, K30 100n, K31 100n, K33 100n, K34 100n, K36 100n, K37 100n, K38 100n, K39 100n, K4 100n, K44 100n, K45 100n, K48 100n, K49 100n, K5 100n, K50 100n, K51 100n, K52 100n, K53 100n, K54 100n, K55 100n, K57 100n, K58 100n, K59 100n, K6 100n, K60 100n, K61 100n, K62 100n, K63 100n, K64 100n, K65 100n, K66 100n, K68 100n, K69 100n, K7 100n, K70 100n, K71 100n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

Commit message: Replaced/corrected D70 from DL008 with DL000 Updated schematics
Parts:
- D70: value DL008D -> DL000D; symbol robotron_ec1834:DL008D -> robotron_ec1834:DL000D
Changed lines of the file:
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@@
     (pin "7")
   )
-  (symbol (lib_id "robotron_ec1834:DL008D") (at 294.64 59.69 0) (unit 5)
+  (symbol (lib_id "robotron_ec1834:DL000D") (at 294.64 59.69 0) (unit 5)
     (in_bom yes) (on_board yes)
     (property "Reference" "D70" (id 0) (at 292.1 71.12 0)
       (effects (font (size 1.27 1.27)) (justify left))
     )
-    (property "Value" "DL008D" (id 1) (at 297.18 63.5 90)
+    (property "Value" "DL000D" (id 1) (at 297.18 63.5 90)
       (effects (font (size 1.27 1.27)) (justify left))
     )
@@
       (effects (font (size 1.27 1.27)) hide)
     )
-    (property "Datasheet" "https://www-user.tu-chemnitz.de/~heha/basteln/Konsumg%C3%BCter/DDR-Halbleiter/dl008.gif" (id 3) (at 294.64 59.69 0)
+    (property "Datasheet" "https://www-user.tu-chemnitz.de/~heha/basteln/Konsumg%C3%BCter/DDR-Halbleiter/dl000.gif" (id 3) (at 294.64 67.31 0)
       (effects (font (size 1.27 1.27)) hide)
     )

Commit message: Fixed wrong symbol (some DL008 are 74S00)
Parts:
- D10, D32, D39, D70: value DL000D -> 74S00
- D16: value DL000D -> DL000
- D57, D69: value DL008D -> 74S00; symbol robotron_ec1834:DL008D -> robotron_ec1834:DL000D
Changed lines of the file:
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@@
     (pin "7")
   )
-  (symbol (lib_id "robotron_ec1834:DL008D") (at 279.4 59.69 0) (unit 5)
+  (symbol (lib_id "robotron_ec1834:DL000D") (at 279.4 59.69 0) (unit 5)
     (in_bom yes) (on_board yes)
     (property "Reference" "D57" (id 0) (at 276.86 71.12 0)
       (effects (font (size 1.27 1.27)) (justify left))
     )
-    (property "Value" "DL008D" (id 1) (at 281.94 63.5 90)
+    (property "Value" "74S00" (id 1) (at 281.94 63.5 90)
       (effects (font (size 1.27 1.27)) (justify left))
     )
@@
       (effects (font (size 1.27 1.27)) hide)
     )
-    (property "Datasheet" "https://www-user.tu-chemnitz.de/~heha/basteln/Konsumg%C3%BCter/DDR-Halbleiter/dl008.gif" (id 3) (at 279.4 59.69 0)
+    (property "Datasheet" "https://www-user.tu-chemnitz.de/~heha/basteln/Konsumg%C3%BCter/DDR-Halbleiter/dl000.gif" (id 3) (at 279.4 67.31 0)
       (effects (font (size 1.27 1.27)) hide)
     )
@@
     (pin "7")
   )
-  (symbol (lib_id "robotron_ec1834:DL008D") (at 287.02 59.69 0) (unit 5)
+  (symbol (lib_id "robotron_ec1834:DL000D") (at 287.02 59.69 0) (unit 5)
     (in_bom yes) (on_board yes)
     (property "Reference" "D69" (id 0) (at 284.48 71.12 0)
       (effects (font (size 1.27 1.27)) (justify left))
     )
-    (property "Value" "DL008D" (id 1) (at 289.56 63.5 90)
+    (property "Value" "74S00" (id 1) (at 289.56 63.5 90)
       (effects (font (size 1.27 1.27)) (justify left))
     )
@@
       (effects (font (size 1.27 1.27)) hide)
     )
-    (property "Datasheet" "https://www-user.tu-chemnitz.de/~heha/basteln/Konsumg%C3%BCter/DDR-Halbleiter/dl008.gif" (id 3) (at 287.02 59.69 0)
+    (property "Datasheet" "https://www-user.tu-chemnitz.de/~heha/basteln/Konsumg%C3%BCter/DDR-Halbleiter/dl000.gif" (id 3) (at 287.02 67.31 0)
       (effects (font (size 1.27 1.27)) hide)
     )
@@
       (effects (font (size 1.27 1.27)) (justify left))
     )
-    (property "Value" "DL000D" (id 1) (at 297.18 63.5 90)
+    (property "Value" "74S00" (id 1) (at 297.18 63.5 90)
       (effects (font (size 1.27 1.27)) (justify left))
     )
@@
       (effects (font (size 1.27 1.27)) (justify left))
     )
-    (property "Value" "DL000D" (id 1) (at 231.14 62.23 90)
+    (property "Value" "74S00" (id 1) (at 231.14 62.23 90)
       (effects (font (size 1.27 1.27)) (justify left))
     )
@@
       (effects (font (size 1.27 1.27)) (justify left))
     )
-    (property "Value" "DL000D" (id 1) (at 237.49 62.23 90)
+    (property "Value" "DL000" (id 1) (at 237.49 62.23 90)
       (effects (font (size 1.27 1.27)) (justify left))
     )
@@
       (effects (font (size 1.27 1.27)) (justify left))
     )
-    (property "Value" "DL000D" (id 1) (at 243.84 62.23 90)
+    (property "Value" "74S00" (id 1) (at 243.84 62.23 90)
       (effects (font (size 1.27 1.27)) (justify left))
     )
@@
       (effects (font (size 1.27 1.27)) (justify left))
     )
-    (property "Value" "DL000D" (id 1) (at 250.19 62.23 90)
+    (property "Value" "74S00" (id 1) (at 250.19 62.23 90)
       (effects (font (size 1.27 1.27)) (justify left))
     )
@@
     (pin "10")
   )
-  (symbol (lib_id "robotron_ec1834:DL008D") (at 547.37 186.69 0) (unit 2)
+  (symbol (lib_id "robotron_ec1834:DL000D") (at 547.37 186.69 0) (unit 2)
     (in_bom yes) (on_board yes)
     (property "Reference" "D69" (id 0) (at 544.83 179.07 0)
       (effects (font (size 1.27 1.27)) (justify left))
     )
-    (property "Value" "DL008D" (id 1) (at 543.56 181.61 0)
+    (property "Value" "74S00" (id 1) (at 543.56 181.61 0)
       (effects (font (size 1.27 1.27)) (justify left))
     )
@@
       (effects (font (size 1.27 1.27)) hide)
     )
-    (property "Datasheet" "https://www-user.tu-chemnitz.de/~heha/basteln/Konsumg%C3%BCter/DDR-Halbleiter/dl008.gif" (id 3) (at 547.37 186.69 0)
+    (property "Datasheet" "https://www-user.tu-chemnitz.de/~heha/basteln/Konsumg%C3%BCter/DDR-Halbleiter/dl000.gif" (id 3) (at 547.37 194.31 0)
       (effects (font (size 1.27 1.27)) hide)
     )

Commit message: Modifications to pass most ERC checks modified symbols for ERC check Added some notes
Parts:
- D5: symbol RFT_Digitalschaltkreise:DL030D -> robotron_ec1834:DL030D
- X3: symbol Connector_Generic:Conn_01x08 -> robotron_ec1834:Power_X3
