File: EC1834-Board.kicad_sch (KiCad schematic)
At the start: 0 parts

Commit message: Completed BUS Final checks required
Other:
- sheet Bus ports: added D[0..15], {A[0..19] VA0 ~{BHE}}, {~{DACK0} ~{DACK1} ~{DACK2} ~{DACK3} ALE RESETDRV CLK ~{IOR} ~{IOW} ~{MEMR} ~{MEMW} AEN IOCHRDY ~{IOCHCK} ~{MASTER} ~{MEMCS16} DRQ0 DRQ1 DRQ2 DRQ3 TC IRQ3 IRQ4 IRQ5 IRQ6 IRQ7 IRQ2 IRQ10 IRQ11 IRQ14 IRQ15 OSC}; removed none
- sheet EC1834 201.2 ports: added {A[0..19] VA0 ~{BHE}}; removed A[0..19]
- note added: "Seite 4 Stromversorgung"
- note added: "Seite 5 - BUS"
- company: (none) -> Mario Gögel 2022
- title: (none) -> EC1834 Hauptplatine

Commit message: Small improvements
Other:
- sheet EC1834 201.2 ports: added {AENBRD ~{AEN} MEMR PB3 ~{IOCHCK} BHE DRQ0 ~{DACK0BRD} DACK0 ~{DACK0} ~{INTA} ~{IOR} ~{IOW} ~{XIOR} ~{XIOW} ~{XMEMR} ~{MEMR} ~{MEMW} ~{NMIADRCS} ~{TIMERCS} ~{PPICS} ~{NIMREGCS} IRQ0 IRQ1 OSC OSC1 PCLK CLK86 ~{MEMADRSEL} NMI NPNPI RESET ~{RESETDRV} MDPEE MDPOE}; removed {AENBRD ~{AEN} MEMR PB3 ~{IOCHCK} BHE DRQ0 ~{DACK0BRD} DACK0 ~{DACK0} ~{INTA} ~{IOR} ~{IOW} ~{XIOR} ~{XIOW} ~{XMEMR} ~{MEMR} ~{MEMW} ~{NMIADRCS} ~{TIMERCS} ~{PPICS} ~{NIMREGCS} IRQ0 IRQ1 OSC OSC1 PCLK CLK86 ~{MEMADRSEL} NMI NPNPI RESET ~{RESETDRV}}
Changed lines of the file:
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@@
       (effects (font (size 1.27 1.27)) (justify left top))
     )
-    (pin "{AENBRD ~{AEN} MEMR PB3 ~{IOCHCK} BHE DRQ0 ~{DACK0BRD} DACK0 ~{DACK0} ~{INTA} ~{IOR} ~{IOW} ~{XIOR} ~{XIOW} ~{XMEMR} ~{MEMR} ~{MEMW} ~{NMIADRCS} ~{TIMERCS} ~{PPICS} ~{NIMREGCS} IRQ0 IRQ1 OSC OSC1 PCLK CLK86 ~{MEMADRSEL} NMI NPNPI RESET ~{RESETDRV}}" input (at 289.56 381 0)
+    (pin "{AENBRD ~{AEN} MEMR PB3 ~{IOCHCK} BHE DRQ0 ~{DACK0BRD} DACK0 ~{DACK0} ~{INTA} ~{IOR} ~{IOW} ~{XIOR} ~{XIOW} ~{XMEMR} ~{MEMR} ~{MEMW} ~{NMIADRCS} ~{TIMERCS} ~{PPICS} ~{NIMREGCS} IRQ0 IRQ1 OSC OSC1 PCLK CLK86 ~{MEMADRSEL} NMI NPNPI RESET ~{RESETDRV} MDPEE MDPOE}" input (at 289.56 381 0)
       (effects (font (size 1.27 1.27)) (justify right))
     )
