File: EC1834-Board.kicad_sch (KiCad schematic)
At the start: 0 parts

Commit message: Modifications to pass most ERC checks modified symbols for ERC check Added some notes
Other:
- sheet Bus ports: added {~{A0} AEN AENBRD AENBRDW AENDMA ALE BHE BS-/WAIT CLK CLK86 DACK0 DEN DT-/R DRQ0 DRQ1 DRQ2 DRQ3 HOLDA HRQDMA IED INT IOCHRDY IORW IRQ0 IRQ1 IRQ2 IRQ3 IRQ4 IRQ5 IRQ6 IRQ7 IRQ8 IRQ10 IRQ11 IRQ12 IRQ14 IRQ15 MASTER MDPEE MDPOE MEMR NPNPI NMI PB3 PCLK OSC OSC1 QS0 QS1 RDY-/WAIT READY RDYTODMA RESET RESETDRV TC VA0 XA0 ~{AEN} ~{BHE} ~{CLK} ~{DACK0BRD} ~{DACK0} ~{DACK1} ~{DACK2} ~{DACK3} ~{DMACS} ~{DMAAEN} ~{INTA} ~{INTRCS1} ~{INTRCS2} ~{IOR} ~{IOW} ~{GT1} ~{LOCK} ~{MASTER} ~{MEMADRSEL} ~{MEMCS16} ~{MEMR} ~{MEMW} ~{NMIADRCS} ~{NMIREGCS} ~{PPICS} ~{RESETDRV} ~{S0} ~{S1} ~{S2} ~{TIMERCS} ~{XIOR} ~{XIOW} ~{XMEMR} ~{XMEMW} ~{YIOR} ~{YIOW}}; removed {~{DACK0} ~{DACK1} ~{DACK2} ~{DACK3} ALE RESETDRV CLK ~{IOR} ~{IOW} ~{MEMR} ~{MEMW} AEN IOCHRDY ~{IOCHCK} ~{MASTER} ~{MEMCS16} DRQ0 DRQ1 DRQ2 DRQ3 TC IRQ3 IRQ4 IRQ5 IRQ6 IRQ7 IRQ2 IRQ10 IRQ11 IRQ14 IRQ15 OSC}
- sheet EC1834 201.1 ports: added {~{A0} AEN AENBRD AENBRDW AENDMA ALE BHE BS-/WAIT CLK CLK86 DACK0 DEN DT-/R DRQ0 DRQ1 DRQ2 DRQ3 HOLDA HRQDMA IED INT IOCHRDY IORW IRQ0 IRQ1 IRQ2 IRQ3 IRQ4 IRQ5 IRQ6 IRQ7 IRQ8 IRQ10 IRQ11 IRQ12 IRQ14 IRQ15 MASTER MDPEE MDPOE MEMR NPNPI NMI PB3 PCLK OSC OSC1 QS0 QS1 RDY-/WAIT READY RDYTODMA RESET RESETDRV TC VA0 XA0 ~{AEN} ~{BHE} ~{CLK} ~{DACK0BRD} ~{DACK0} ~{DACK1} ~{DACK2} ~{DACK3} ~{DMACS} ~{DMAAEN} ~{INTA} ~{INTRCS1} ~{INTRCS2} ~{IOR} ~{IOW} ~{GT1} ~{LOCK} ~{MASTER} ~{MEMADRSEL} ~{MEMCS16} ~{MEMR} ~{MEMW} ~{NMIADRCS} ~{NMIREGCS} ~{PPICS} ~{RESETDRV} ~{S0} ~{S1} ~{S2} ~{TIMERCS} ~{XIOR} ~{XIOW} ~{XMEMR} ~{XMEMW} ~{YIOR} ~{YIOW}}; removed {AENBRD ~{AEN} MEMR PB3 ~{IOCHCK} BHE DRQ0 ~{DACK0BRD} DACK0 ~{DACK0} ~{INTA} ~{IOR} ~{IOW} ~{XIOR} ~{XIOW} ~{XMEMR} ~{MEMR} ~{MEMW} ~{NMIADRCS} ~{TIMERCS} ~{PPICS} ~{NIMREGCS} IRQ0 IRQ1 OSC OSC1 PCLK CLK86 ~{MEMADRSEL} NMI NPNPI RESET ~{RESETDRV}}
- sheet EC1834 201.2 ports: added {~{A0} AEN AENBRD AENBRDW AENDMA ALE BHE BS-/WAIT CLK CLK86 DACK0 DEN DT-/R DRQ0 DRQ1 DRQ2 DRQ3 HOLDA HRQDMA IED INT IOCHRDY IORW IRQ0 IRQ1 IRQ2 IRQ3 IRQ4 IRQ5 IRQ6 IRQ7 IRQ8 IRQ10 IRQ11 IRQ12 IRQ14 IRQ15 MASTER MDPEE MDPOE MEMR NPNPI NMI PB3 PCLK OSC OSC1 QS0 QS1 RDY-/WAIT READY RDYTODMA RESET RESETDRV TC VA0 XA0 ~{AEN} ~{BHE} ~{CLK} ~{DACK0BRD} ~{DACK0} ~{DACK1} ~{DACK2} ~{DACK3} ~{DMACS} ~{DMAAEN} ~{INTA} ~{INTRCS1} ~{INTRCS2} ~{IOR} ~{IOW} ~{GT1} ~{LOCK} ~{MASTER} ~{MEMADRSEL} ~{MEMCS16} ~{MEMR} ~{MEMW} ~{NMIADRCS} ~{NMIREGCS} ~{PPICS} ~{RESETDRV} ~{S0} ~{S1} ~{S2} ~{TIMERCS} ~{XIOR} ~{XIOW} ~{XMEMR} ~{XMEMW} ~{YIOR} ~{YIOW}}; removed {AENBRD ~{AEN} MEMR PB3 ~{IOCHCK} BHE DRQ0 ~{DACK0BRD} DACK0 ~{DACK0} ~{INTA} ~{IOR} ~{IOW} ~{XIOR} ~{XIOW} ~{XMEMR} ~{MEMR} ~{MEMW} ~{NMIADRCS} ~{TIMERCS} ~{PPICS} ~{NIMREGCS} IRQ0 IRQ1 OSC OSC1 PCLK CLK86 ~{MEMADRSEL} NMI NPNPI RESET ~{RESETDRV} MDPEE MDPOE}
Changed lines of the file:
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@@
       (effects (font (size 1.27 1.27)) (justify left top))
     )
-    (pin "D[0..15]" input (at 271.78 287.02 270)
-      (effects (font (size 1.27 1.27)) (justify left))
-    )
-    (pin "{A[0..19] VA0 ~{BHE}}" input (at 256.54 287.02 270)
-      (effects (font (size 1.27 1.27)) (justify left))
-    )
-    (pin "XA[0..19]" input (at 278.13 287.02 270)
-      (effects (font (size 1.27 1.27)) (justify left))
-    )
-    (pin "XD[0..15]" input (at 250.19 287.02 270)
+    (pin "D[0..15]" bidirectional (at 271.78 287.02 270)
+      (effects (font (size 1.27 1.27)) (justify left))
+    )
+    (pin "{A[0..19] VA0 ~{BHE}}" bidirectional (at 256.54 287.02 270)
+      (effects (font (size 1.27 1.27)) (justify left))
+    )
+    (pin "XA[0..19]" bidirectional (at 278.13 287.02 270)
+      (effects (font (size 1.27 1.27)) (justify left))
+    )
+    (pin "XD[0..15]" bidirectional (at 250.19 287.02 270)
       (effects (font (size 1.27 1.27)) (justify left))
     )
@@
       (effects (font (size 1.27 1.27)) (justify left))
     )
-    (pin "{AENBRD ~{AEN} MEMR PB3 ~{IOCHCK} BHE DRQ0 ~{DACK0BRD} DACK0 ~{DACK0} ~{INTA} ~{IOR} ~{IOW} ~{XIOR} ~{XIOW} ~{XMEMR} ~{MEMR} ~{MEMW} ~{NMIADRCS} ~{TIMERCS} ~{PPICS} ~{NIMREGCS} IRQ0 IRQ1 OSC OSC1 PCLK CLK86 ~{MEMADRSEL} NMI NPNPI RESET ~{RESETDRV}}" input (at 284.48 248.92 0)
+    (pin "{~{A0} AEN AENBRD AENBRDW AENDMA ALE BHE BS-{slash}WAIT CLK CLK86 DACK0 DEN DT-{slash}R DRQ0 DRQ1 DRQ2 DRQ3 HOLDA HRQDMA IED INT IOCHRDY IORW IRQ0 IRQ1 IRQ2 IRQ3 IRQ4 IRQ5 IRQ6 IRQ7 IRQ8 IRQ10 IRQ11 IRQ12 IRQ14 IRQ15 MASTER MDPEE MDPOE MEMR NPNPI NMI PB3 PCLK OSC OSC1 QS0 QS1 RDY-{slash}WAIT READY RDYTODMA RESET RESETDRV TC VA0 XA0 ~{AEN} ~{BHE} ~{CLK} ~{DACK0BRD} ~{DACK0} ~{DACK1} ~{DACK2} ~{DACK3} ~{DMACS} ~{DMAAEN} ~{INTA} ~{INTRCS1} ~{INTRCS2} ~{IOR} ~{IOW} ~{GT1} ~{LOCK} ~{MASTER} ~{MEMADRSEL} ~{MEMCS16} ~{MEMR} ~{MEMW} ~{NMIADRCS} ~{NMIREGCS} ~{PPICS} ~{RESETDRV} ~{S0} ~{S1} ~{S2} ~{TIMERCS} ~{XIOR} ~{XIOW} ~{XMEMR} ~{XMEMW} ~{YIOR} ~{YIOW}}" input (at 284.48 248.92 0)
       (effects (font (size 1.27 1.27)) (justify right))
     )
@@
       (effects (font (size 1.27 1.27)) (justify left top))
     )
-    (pin "{AENBRD ~{AEN} MEMR PB3 ~{IOCHCK} BHE DRQ0 ~{DACK0BRD} DACK0 ~{DACK0} ~{INTA} ~{IOR} ~{IOW} ~{XIOR} ~{XIOW} ~{XMEMR} ~{MEMR} ~{MEMW} ~{NMIADRCS} ~{TIMERCS} ~{PPICS} ~{NIMREGCS} IRQ0 IRQ1 OSC OSC1 PCLK CLK86 ~{MEMADRSEL} NMI NPNPI RESET ~{RESETDRV} MDPEE MDPOE}" input (at 289.56 381 0)
-      (effects (font (size 1.27 1.27)) (justify right))
-    )
-    (pin "XA[0..19]" input (at 278.13 312.42 90)
-      (effects (font (size 1.27 1.27)) (justify right))
-    )
-    (pin "D[0..15]" input (at 271.78 312.42 90)
-      (effects (font (size 1.27 1.27)) (justify right))
-    )
-    (pin "{A[0..19] VA0 ~{BHE}}" input (at 256.54 312.42 90)
-      (effects (font (size 1.27 1.27)) (justify right))
-    )
-    (pin "XD[0..15]" input (at 250.19 312.42 90)
+    (pin "{~{A0} AEN AENBRD AENBRDW AENDMA ALE BHE BS-{slash}WAIT CLK CLK86 DACK0 DEN DT-{slash}R DRQ0 DRQ1 DRQ2 DRQ3 HOLDA HRQDMA IED INT IOCHRDY IORW IRQ0 IRQ1 IRQ2 IRQ3 IRQ4 IRQ5 IRQ6 IRQ7 IRQ8 IRQ10 IRQ11 IRQ12 IRQ14 IRQ15 MASTER MDPEE MDPOE MEMR NPNPI NMI PB3 PCLK OSC OSC1 QS0 QS1 RDY-{slash}WAIT READY RDYTODMA RESET RESETDRV TC VA0 XA0 ~{AEN} ~{BHE} ~{CLK} ~{DACK0BRD} ~{DACK0} ~{DACK1} ~{DACK2} ~{DACK3} ~{DMACS} ~{DMAAEN} ~{INTA} ~{INTRCS1} ~{INTRCS2} ~{IOR} ~{IOW} ~{GT1} ~{LOCK} ~{MASTER} ~{MEMADRSEL} ~{MEMCS16} ~{MEMR} ~{MEMW} ~{NMIADRCS} ~{NMIREGCS} ~{PPICS} ~{RESETDRV} ~{S0} ~{S1} ~{S2} ~{TIMERCS} ~{XIOR} ~{XIOW} ~{XMEMR} ~{XMEMW} ~{YIOR} ~{YIOW}}" bidirectional (at 289.56 381 0)
+      (effects (font (size 1.27 1.27)) (justify right))
+    )
+    (pin "XA[0..19]" bidirectional (at 278.13 312.42 90)
+      (effects (font (size 1.27 1.27)) (justify right))
+    )
+    (pin "D[0..15]" bidirectional (at 271.78 312.42 90)
+      (effects (font (size 1.27 1.27)) (justify right))
+    )
+    (pin "{A[0..19] VA0 ~{BHE}}" bidirectional (at 256.54 312.42 90)
+      (effects (font (size 1.27 1.27)) (justify right))
+    )
+    (pin "XD[0..15]" bidirectional (at 250.19 312.42 90)
       (effects (font (size 1.27 1.27)) (justify right))
     )
@@
       (effects (font (size 1.27 1.27)) (justify right))
     )
-    (pin "MD[0..15]" input (at 289.56 384.81 0)
-      (effects (font (size 1.27 1.27)) (justify right))
-    )
-    (pin "{MEM[0..8] ~{RAS0} ~{RAS1} ~{CASL} ~{CASH} ~{WE}}" input (at 289.56 388.62 0)
+    (pin "MD[0..15]" bidirectional (at 289.56 384.81 0)
+      (effects (font (size 1.27 1.27)) (justify right))
+    )
+    (pin "{MEM[0..8] ~{RAS0} ~{RAS1} ~{CASL} ~{CASH} ~{WE}}" bidirectional (at 289.56 388.62 0)
       (effects (font (size 1.27 1.27)) (justify right))
     )
@@
       (effects (font (size 1.27 1.27)) (justify left top))
     )
-    (pin "{MEM[0..7] ~{WE} ~{RAS0} ~{RAS1} ~{CASL} ~{CASH}}" input (at 314.96 199.39 180)
-      (effects (font (size 1.27 1.27)) (justify left))
-    )
-    (pin "MD[0..15]" input (at 314.96 196.85 180)
-      (effects (font (size 1.27 1.27)) (justify left))
-    )
-    (pin "{~{MEMR} MEMR MDPOE MDPEE}" input (at 314.96 193.04 180)
+    (pin "{MEM[0..7] ~{WE} ~{RAS0} ~{RAS1} ~{CASL} ~{CASH}}" bidirectional (at 314.96 199.39 180)
+      (effects (font (size 1.27 1.27)) (justify left))
+    )
+    (pin "MD[0..15]" bidirectional (at 314.96 196.85 180)
+      (effects (font (size 1.27 1.27)) (justify left))
+    )
+    (pin "{~{MEMR} MEMR MDPOE MDPEE}" bidirectional (at 314.96 193.04 180)
       (effects (font (size 1.27 1.27)) (justify left))
     )
@@
       (effects (font (size 1.27 1.27)) (justify left top))
     )
-    (pin "D[0..15]" input (at 547.37 312.42 90)
-      (effects (font (size 1.27 1.27)) (justify right))
-    )
-    (pin "{A[0..19] VA0 ~{BHE}}" input (at 534.67 353.06 180)
-      (effects (font (size 1.27 1.27)) (justify left))
-    )
-    (pin "{~{DACK0} ~{DACK1} ~{DACK2} ~{DACK3} ALE RESETDRV CLK ~{IOR} ~{IOW} ~{MEMR} ~{MEMW} AEN IOCHRDY ~{IOCHCK} ~{MASTER} ~{MEMCS16} DRQ0 DRQ1 DRQ2 DRQ3 TC IRQ3 IRQ4 IRQ5 IRQ6 IRQ7 IRQ2 IRQ10 IRQ11 IRQ14 IRQ15 OSC}" input (at 534.67 341.63 180)
+    (pin "D[0..15]" bidirectional (at 547.37 312.42 90)
+      (effects (font (size 1.27 1.27)) (justify right))
+    )
+    (pin "{A[0..19] VA0 ~{BHE}}" bidirectional (at 534.67 353.06 180)
+      (effects (font (size 1.27 1.27)) (justify left))
+    )
+    (pin "{~{A0} AEN AENBRD AENBRDW AENDMA ALE BHE BS-{slash}WAIT CLK CLK86 DACK0 DEN DT-{slash}R DRQ0 DRQ1 DRQ2 DRQ3 HOLDA HRQDMA IED INT IOCHRDY IORW IRQ0 IRQ1 IRQ2 IRQ3 IRQ4 IRQ5 IRQ6 IRQ7 IRQ8 IRQ10 IRQ11 IRQ12 IRQ14 IRQ15 MASTER MDPEE MDPOE MEMR NPNPI NMI PB3 PCLK OSC OSC1 QS0 QS1 RDY-{slash}WAIT READY RDYTODMA RESET RESETDRV TC VA0 XA0 ~{AEN} ~{BHE} ~{CLK} ~{DACK0BRD} ~{DACK0} ~{DACK1} ~{DACK2} ~{DACK3} ~{DMACS} ~{DMAAEN} ~{INTA} ~{INTRCS1} ~{INTRCS2} ~{IOR} ~{IOW} ~{GT1} ~{LOCK} ~{MASTER} ~{MEMADRSEL} ~{MEMCS16} ~{MEMR} ~{MEMW} ~{NMIADRCS} ~{NMIREGCS} ~{PPICS} ~{RESETDRV} ~{S0} ~{S1} ~{S2} ~{TIMERCS} ~{XIOR} ~{XIOW} ~{XMEMR} ~{XMEMW} ~{YIOR} ~{YIOW}}" bidirectional (at 534.67 341.63 180)
       (effects (font (size 1.27 1.27)) (justify left))
     )
@@
       (reference "#PWR0207") (unit 1) (value "GND") (footprint "")
     )
+    (path "/00000000-0000-0000-0000-0000631598da/b73faecb-e92e-48a0-8dcc-2908ddccf9d7"
+      (reference "#PWR0209") (unit 1) (value "GND") (footprint "")
+    )
     (path "/00000000-0000-0000-0000-00006315bff5/1447c0b1-b561-4dcf-8efc-79f3985ecbf0"
