File: EC1834-Board.kicad_pcb (KiCad board)
At the start: 6 copper layers, 360 x 240 mm, 345 parts, among them K1 100n, K10 100n, K100 100n, K101 100n, K102 100n, K103 100n, K104 100n, K105 100n, K106 100n, K107 100n, K108 100n, K109 100n, K11 100n, K110 100n, K111 100n, K112 100n, K113 100n, K115 100n, K116 100n, K117 100n, K118 100n, K119 100n, K12 100n, K120 100n, K121 100n, K122 100n, K123 100n, K124 100n, K125 100n, K126 100n, K13 100n, K14 100n, K15 100n, K16 100n, K18 100n, K19 100n, K2 100n, K20 100n, K22 100n, K23 100n, K24 100n, K25 100n, K27 100n, K3 100n, K30 100n, K31 100n, K33 100n, K34 100n, K36 100n, K37 100n, K38 100n, K39 100n, K4 100n, K44 100n, K45 100n, K48 100n, K49 100n, K5 100n, K50 100n, K51 100n, K52 100n, K53 100n, K54 100n, K55 100n, K57 100n, K58 100n, K59 100n, K6 100n, K60 100n, K61 100n, K62 100n, K63 100n, K64 100n, K65 100n, K66 100n, K68 100n, K69 100n, K7 100n, K70 100n, K71 100n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

Commit message: Replaced/corrected D70 from DL008 with DL000 Updated schematics
Parts:
- D70: value DL008D -> DL000D
Connections:
- D50 pad 6: /EC1834 201.1/TDYTODMA -> /EC1834 201.1/RDYTODMA
- D72 pad 11: Net-(D72-Pad11) -> /EC1834_201.3 RAM/~{CASH}
- D72 pad 3: Net-(D72-Pad3) -> /EC1834_201.3 RAM/~{RAS1}
- D72 pad 6: Net-(D72-Pad6) -> /EC1834_201.3 RAM/~{RAS0}
- D72 pad 8: Net-(D72-Pad8) -> /EC1834_201.3 RAM/~{CASL}
- D85 pad 12: Net-(D85-Pad12) -> /EC1834 201.2/MEM0
- D85 pad 4: Net-(D85-Pad4) -> /EC1834 201.2/MEM2
- D85 pad 7: Net-(D85-Pad7) -> /EC1834 201.2/MEM1
- D85 pad 9: Net-(D85-Pad9) -> /EC1834 201.2/MEM3
- D86 pad 12: Net-(D86-Pad12) -> /EC1834 201.2/MEM7
- D86 pad 4: Net-(D86-Pad4) -> /EC1834 201.2/MEM4
- D86 pad 7: Net-(D86-Pad7) -> /EC1834 201.2/MEM6
- D86 pad 9: Net-(D86-Pad9) -> /EC1834 201.2/MEM5
- D88 pad 6: Net-(D88-Pad6) -> /EC1834_201.3 RAM/~{WE}
- R14 pad 1: Net-(D86-Pad7) -> /EC1834 201.2/MEM6
- R14 pad 3: Net-(D86-Pad4) -> /EC1834 201.2/MEM4
- R14 pad 5: Net-(D86-Pad12) -> /EC1834 201.2/MEM7
- R14 pad 8: Net-(D86-Pad9) -> /EC1834 201.2/MEM5
- R15 pad 2: Net-(D85-Pad7) -> /EC1834 201.2/MEM1
- R15 pad 4: Net-(D85-Pad4) -> /EC1834 201.2/MEM2
- R15 pad 5: Net-(D85-Pad12) -> /EC1834 201.2/MEM0
- R15 pad 8: Net-(D85-Pad9) -> /EC1834 201.2/MEM3
- R16 pad 1: Net-(D72-Pad3) -> /EC1834_201.3 RAM/~{RAS1}
- R16 pad 3: Net-(D72-Pad6) -> /EC1834_201.3 RAM/~{RAS0}
- R16 pad 5: Net-(D72-Pad8) -> /EC1834_201.3 RAM/~{CASL}
- R16 pad 7: Net-(D72-Pad11) -> /EC1834_201.3 RAM/~{CASH}
- R18 pad 2: Net-(D88-Pad6) -> /EC1834_201.3 RAM/~{WE}

Commit message: Fixed wrong symbol (some DL008 are 74S00)
Parts:
- D10, D32, D39, D70: value DL000D -> 74S00
- D16: value DL000D -> DL000
- D57, D69: value DL008D -> 74S00
Changed lines of the file:
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@@
       (effects (font (size 1 1) (thickness 0.15)))
     )
-    (fp_text value "DL000D" (at 3.81 17.57) (layer "F.Fab")
+    (fp_text value "DL000" (at 3.81 17.57) (layer "F.Fab")
       (effects (font (size 1 1) (thickness 0.15)))
     )
@@
       (effects (font (size 1 1) (thickness 0.15)))
     )
-    (fp_text value "DL008D" (at 3.81 12.065 90) (layer "F.Fab")
+    (fp_text value "74S00" (at 3.81 12.065 90) (layer "F.Fab")
       (effects (font (size 1 1) (thickness 0.15)))
     )
@@
       (effects (font (size 1 1) (thickness 0.15)))
     )
-    (fp_text value "DL000D" (at 3.81 17.57) (layer "F.Fab")
+    (fp_text value "74S00" (at 3.81 17.57) (layer "F.Fab")
       (effects (font (size 1 1) (thickness 0.15)))
     )
@@
       (effects (font (size 1 1) (thickness 0.15)))
     )
-    (fp_text value "DL000D" (at 3.81 17.57) (layer "F.Fab")
+    (fp_text value "74S00" (at 3.81 17.57) (layer "F.Fab")
       (effects (font (size 1 1) (thickness 0.15)))
     )
@@
       (effects (font (size 1 1) (thickness 0.15)))
     )
-    (fp_text value "DL000D" (at 3.81 17.57) (layer "F.Fab")
+    (fp_text value "74S00" (at 3.81 17.57) (layer "F.Fab")
       (effects (font (size 1 1) (thickness 0.15)))
     )
@@
       (effects (font (size 1 1) (thickness 0.15)))
     )
-    (fp_text value "DL008D" (at 3.81 17.57) (layer "F.Fab")
+    (fp_text value "74S00" (at 3.81 17.57) (layer "F.Fab")
       (effects (font (size 1 1) (thickness 0.15)))
     )
@@
       (effects (font (size 1 1) (thickness 0.15)))
     )
-    (fp_text value "DL000D" (at 3.81 17.57) (layer "F.Fab")
+    (fp_text value "74S00" (at 3.81 17.57) (layer "F.Fab")
       (effects (font (size 1 1) (thickness 0.15)))
     )

Commit message: Updated ec1834 symbols Fixed missing D8-D15 on bus connector Updated PDFs
Connections:
- Br2 pad 1: /EC1834_201.3 RAM/MDPEE -> /EC1834 201.1/MDPEE
- Br2 pad 2: /EC1834_201.3 RAM/MDPEE -> /EC1834 201.1/MDPEE
- Br3 pad 1: /EC1834_201.3 RAM/MDPOE -> /EC1834 201.1/MDPOE
- Br3 pad 2: /EC1834_201.3 RAM/MDPOE -> /EC1834 201.1/MDPOE
- D102 pad 2: /EC1834_201.3 RAM/MDPEE -> /EC1834 201.1/MDPEE
- D113 pad 5: /EC1834_201.3 RAM/MDPEE -> /EC1834 201.1/MDPEE
- D114 pad 5: /EC1834_201.3 RAM/MDPOE -> /EC1834 201.1/MDPOE
- D117 pad 2: /EC1834_201.3 RAM/MDPEE -> /EC1834 201.1/MDPEE
- D16 pad 9: /EC1834 201.2/~{A0} -> /EC1834 201.1/~{A0}
- D53 pad 23: /EC1834 201.2/~{XOW} -> /EC1834 201.1/~{XIOW}
- D57 pad 8: /EC1834 201.2/OSC -> /EC1834 201.1/OSC
- D59 pad 4: /EC1834 201.2/~{A0} -> /EC1834 201.1/~{A0}
- D68 pad 10: /EC1834 201.2/~{A0} -> /EC1834 201.1/~{A0}
- D68 pad 13: /EC1834 201.2/MDPOE -> /EC1834 201.1/MDPOE
- D68 pad 9: /EC1834 201.2/MDPEE -> /EC1834 201.1/MDPEE
- D69 pad 2: /EC1834 201.2/~{A0} -> /EC1834 201.1/~{A0}
- D71 pad 5: /EC1834 201.2/~{NMIREGCS} -> /EC1834 201.1/~{NMIREGCS}
- D73 pad 2: /EC1834_201.3 RAM/MDPOE -> /EC1834 201.1/MDPOE
- D91 pad 2: /EC1834_201.3 RAM/MDPOE -> /EC1834 201.1/MDPOE
- PS5 pad 10: /EC1834_201.3 RAM/MDPEE -> /EC1834 201.1/MDPEE
- PS5 pad 26: /EC1834_201.3 RAM/MDPOE -> /EC1834 201.1/MDPOE
- X1.1 pad a2: /Bus/RESET -> /EC1834 201.1/RESET
- X1.1 pad a30: /Bus/OSC -> /EC1834 201.1/OSC
- X1.1 pad b2: (no net) -> /EC1834 201.1/D8
- X1.1 pad b23: /Bus/IRQ12 -> /EC1834 201.1/IRQ12
- X1.1 pad b3: (no net) -> /EC1834 201.1/D9
- X1.1 pad b4: (no net) -> /EC1834 201.1/D10
- X1.1 pad b5: (no net) -> /EC1834 201.1/D11
- X1.1 pad b6: (no net) -> /EC1834 201.1/D12
- X1.1 pad b7: (no net) -> /EC1834 201.1/D13
- X1.1 pad b8: (no net) -> /EC1834 201.1/D14
- X1.1 pad b9: (no net) -> /EC1834 201.1/D15
- X1.2 pad a2: /Bus/RESET -> /EC1834 201.1/RESET
- X1.2 pad a30: /Bus/OSC -> /EC1834 201.1/OSC
- X1.2 pad b2: (no net) -> /EC1834 201.1/D8
- X1.2 pad b23: /Bus/IRQ12 -> /EC1834 201.1/IRQ12
- X1.2 pad b3: (no net) -> /EC1834 201.1/D9
- X1.2 pad b4: (no net) -> /EC1834 201.1/D10
- X1.2 pad b5: (no net) -> /EC1834 201.1/D11
- X1.2 pad b6: (no net) -> /EC1834 201.1/D12
- X1.2 pad b7: (no net) -> /EC1834 201.1/D13
- X1.2 pad b8: (no net) -> /EC1834 201.1/D14
- X1.2 pad b9: (no net) -> /EC1834 201.1/D15
- X1.3 pad a2: /Bus/RESET -> /EC1834 201.1/RESET
- X1.3 pad a30: /Bus/OSC -> /EC1834 201.1/OSC
- X1.3 pad b2: (no net) -> /EC1834 201.1/D8
- X1.3 pad b23: /Bus/IRQ12 -> /EC1834 201.1/IRQ12
- X1.3 pad b3: (no net) -> /EC1834 201.1/D9
- X1.3 pad b4: (no net) -> /EC1834 201.1/D10
- X1.3 pad b5: (no net) -> /EC1834 201.1/D11
- X1.3 pad b6: (no net) -> /EC1834 201.1/D12
- X1.3 pad b7: (no net) -> /EC1834 201.1/D13
- X1.3 pad b8: (no net) -> /EC1834 201.1/D14
- X1.3 pad b9: (no net) -> /EC1834 201.1/D15
- X1.3 pad c12: unconnected-(X1.3-Padc12) -> /EC1834 201.1/A19
- X1.3 pad c13: unconnected-(X1.3-Padc13) -> /EC1834 201.1/A18
- X1.3 pad c14: unconnected-(X1.3-Padc14) -> /EC1834 201.1/A17
- X1.3 pad c15: unconnected-(X1.3-Padc15) -> /EC1834 201.1/A16
- X1.3 pad c16: unconnected-(X1.3-Padc16) -> /EC1834 201.1/A15
- X1.3 pad c17: unconnected-(X1.3-Padc17) -> /EC1834 201.1/A14
- X1.3 pad c18: unconnected-(X1.3-Padc18) -> /EC1834 201.1/A13
- X1.3 pad c19: unconnected-(X1.3-Padc19) -> /EC1834 201.1/A12
- X1.3 pad c20: unconnected-(X1.3-Padc20) -> /EC1834 201.1/A11
- X1.3 pad c21: unconnected-(X1.3-Padc21) -> /EC1834 201.1/A10
- X1.3 pad c22: unconnected-(X1.3-Padc22) -> /EC1834 201.1/A9
- X1.3 pad c23: unconnected-(X1.3-Padc23) -> /EC1834 201.1/A8
- X1.3 pad c24: unconnected-(X1.3-Padc24) -> /EC1834 201.1/A7
- X1.3 pad c25: unconnected-(X1.3-Padc25) -> /EC1834 201.1/A6
- X1.3 pad c26: unconnected-(X1.3-Padc26) -> /EC1834 201.1/A5
- X1.3 pad c27: unconnected-(X1.3-Padc27) -> /EC1834 201.1/A4
- X1.3 pad c28: unconnected-(X1.3-Padc28) -> /EC1834 201.1/A3
- X1.3 pad c29: unconnected-(X1.3-Padc29) -> /EC1834 201.1/A2
- X1.3 pad c30: unconnected-(X1.3-Padc30) -> /EC1834 201.1/A1
- X1.3 pad c31: unconnected-(X1.3-Padc31) -> /EC1834 201.1/A0
- X1.4 pad a2: /Bus/RESET -> /EC1834 201.1/RESET
- X1.4 pad a30: /Bus/OSC -> /EC1834 201.1/OSC
- X1.4 pad b2: (no net) -> /EC1834 201.1/D8
- X1.4 pad b23: /Bus/IRQ12 -> /EC1834 201.1/IRQ12
- X1.4 pad b3: (no net) -> /EC1834 201.1/D9
- X1.4 pad b4: (no net) -> /EC1834 201.1/D10
- X1.4 pad b5: (no net) -> /EC1834 201.1/D11
- X1.4 pad b6: (no net) -> /EC1834 201.1/D12
- X1.4 pad b7: (no net) -> /EC1834 201.1/D13
- X1.4 pad b8: (no net) -> /EC1834 201.1/D14
- X1.4 pad b9: (no net) -> /EC1834 201.1/D15
- X1.5 pad a2: /Bus/RESET -> /EC1834 201.1/RESET
- X1.5 pad a30: /Bus/OSC -> /EC1834 201.1/OSC
- X1.5 pad b2: (no net) -> /EC1834 201.1/D8
- X1.5 pad b23: /Bus/IRQ12 -> /EC1834 201.1/IRQ12
- X1.5 pad b3: (no net) -> /EC1834 201.1/D9
- X1.5 pad b4: (no net) -> /EC1834 201.1/D10
- X1.5 pad b5: (no net) -> /EC1834 201.1/D11
- X1.5 pad b6: (no net) -> /EC1834 201.1/D12
- X1.5 pad b7: (no net) -> /EC1834 201.1/D13
- X1.5 pad b8: (no net) -> /EC1834 201.1/D14
- X1.5 pad b9: (no net) -> /EC1834 201.1/D15
- X1.6 pad a2: /Bus/RESET -> /EC1834 201.1/RESET
- X1.6 pad a30: /Bus/OSC -> /EC1834 201.1/OSC
- X1.6 pad b2: (no net) -> /EC1834 201.1/D8
- X1.6 pad b23: /Bus/IRQ12 -> /EC1834 201.1/IRQ12
- X1.6 pad b3: (no net) -> /EC1834 201.1/D9
- X1.6 pad b4: (no net) -> /EC1834 201.1/D10
- X1.6 pad b5: (no net) -> /EC1834 201.1/D11
- X1.6 pad b6: (no net) -> /EC1834 201.1/D12
- X1.6 pad b7: (no net) -> /EC1834 201.1/D13
- X1.6 pad b8: (no net) -> /EC1834 201.1/D14
- X1.6 pad b9: (no net) -> /EC1834 201.1/D15
- X1.6 pad c2: unconnected-(X1.6-Padc2) -> /EC1834 201.1/D7
- X1.6 pad c3: unconnected-(X1.6-Padc3) -> /EC1834 201.1/D6
- X1.6 pad c4: unconnected-(X1.6-Padc4) -> /EC1834 201.1/D5
- X1.7 pad a2: /Bus/RESET -> /EC1834 201.1/RESET
- X1.7 pad a30: /Bus/OSC -> /EC1834 201.1/OSC
- X1.7 pad b2: (no net) -> /EC1834 201.1/D8
- X1.7 pad b23: /Bus/IRQ12 -> /EC1834 201.1/IRQ12
- X1.7 pad b3: (no net) -> /EC1834 201.1/D9
- X1.7 pad b4: (no net) -> /EC1834 201.1/D10
- X1.7 pad b5: (no net) -> /EC1834 201.1/D11
- X1.7 pad b6: (no net) -> /EC1834 201.1/D12
- X1.7 pad b7: (no net) -> /EC1834 201.1/D13
- X1.7 pad b8: (no net) -> /EC1834 201.1/D14
- X1.7 pad b9: (no net) -> /EC1834 201.1/D15
- X1.8 pad a2: /Bus/RESET -> /EC1834 201.1/RESET
- X1.8 pad a30: /Bus/OSC -> /EC1834 201.1/OSC
- X1.8 pad b2: (no net) -> /EC1834 201.1/D8
- X1.8 pad b23: /Bus/IRQ12 -> /EC1834 201.1/IRQ12
- X1.8 pad b3: (no net) -> /EC1834 201.1/D9
- X1.8 pad b4: (no net) -> /EC1834 201.1/D10
- X1.8 pad b5: (no net) -> /EC1834 201.1/D11
- X1.8 pad b6: (no net) -> /EC1834 201.1/D12
- X1.8 pad b7: (no net) -> /EC1834 201.1/D13
- X1.8 pad b8: (no net) -> /EC1834 201.1/D14
- X1.8 pad b9: (no net) -> /EC1834 201.1/D15
